File: hardware/power_supply_module/rev_a/power_supply_module.sch (EAGLE design)
At the start: 1 part, among them J1 MODULE_POWER

Commit message: Started Power Module
Parts:
- added U$1, U$2: PCA9544A, signpost:PCA9544A
- added U$3, U$4: AOZ1037PI, signpost:AOZ1037PI
- added U1, U2, U3, U4, U5, U6, U7, U8: LTC2941-1, signpost:LTC2941-1
Changed lines of the file:
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@@
 <part name="FRAME1" library="lab11-frames" deviceset="LETTER_L_BLANK" device=""/>
 <part name="J1" library="signpost" deviceset="MODULE_POWER" device=""/>
+<part name="U1" library="signpost" deviceset="LTC2941-1" device=""/>
+<part name="U2" library="signpost" deviceset="LTC2941-1" device=""/>
+<part name="U3" library="signpost" deviceset="LTC2941-1" device=""/>
+<part name="U4" library="signpost" deviceset="LTC2941-1" device=""/>
+<part name="U5" library="signpost" deviceset="LTC2941-1" device=""/>
+<part name="U6" library="signpost" deviceset="LTC2941-1" device=""/>
+<part name="U7" library="signpost" deviceset="LTC2941-1" device=""/>
+<part name="U8" library="signpost" deviceset="LTC2941-1" device=""/>
+<part name="U$1" library="signpost" deviceset="PCA9544A" device=""/>
+<part name="U$2" library="signpost" deviceset="PCA9544A" device=""/>
+<part name="U$3" library="signpost" deviceset="AOZ1037PI" device=""/>
+<part name="U$4" library="signpost" deviceset="AOZ1037PI" device=""/>
 </parts>
 <sheets>
@@
 <instance part="FRAME1" gate="G$2" x="147.32" y="0"/>
 <instance part="J1" gate="G$1" x="109.22" y="139.7"/>
+<instance part="U1" gate="G$1" x="172.72" y="149.86"/>
+<instance part="U2" gate="G$1" x="172.72" y="119.38"/>
+<instance part="U3" gate="G$1" x="172.72" y="88.9"/>
+<instance part="U4" gate="G$1" x="172.72" y="58.42"/>
+<instance part="U5" gate="G$1" x="208.28" y="149.86"/>
+<instance part="U6" gate="G$1" x="208.28" y="119.38"/>
+<instance part="U7" gate="G$1" x="208.28" y="88.9"/>
+<instance part="U8" gate="G$1" x="208.28" y="58.42"/>
+<instance part="U$1" gate="G$1" x="101.6" y="78.74"/>
+<instance part="U$2" gate="G$1" x="101.6" y="40.64"/>
+<instance part="U$3" gate="G$1" x="45.72" y="132.08"/>
+<instance part="U$4" gate="G$1" x="45.72" y="111.76"/>
 </instances>
 <busses>

Commit message: Started 5v rails
Parts:
- removed U$3, U$4: AOZ1037PI, signpost:AOZ1037PI
- added C1, C6: EEEFK1A471P, signpost:EEEFK1A471P
- added C10, C4, C5, C9: 220p, passives:CAPACITOR0402_CAP
- added C2, C7: 1u, passives:CAPACITOR0402_CAP
- added C3, C8: 14n, passives:CAPACITOR0402_CAP
- added D1, D2: B340A, signpost:B340A
- added L1, L2: VLP8040, signpost:VLP8040
- added R1, R4: 10k, passives:RESISTOR0402_RES
- added R2, R5: 5k, passives:RESISTOR0402_RES
- added R3, R6: 30.9k, passives:RESISTOR0402_RES
- added U10, U9: TPS54233, signpost:TPS54233
Connections:
- new net 5V_1: C1.CATHODE, L1.1, R1.2
- new net 5V_2: C6.CATHODE, L2.1, R4.2
- new net GND: C3.2, C4.2, C8.2, C9.2, J1.GND, J1.VBATT-, R2.1, R3.1, R5.1, R6.1, U10.GND, U9.GND
- new net N$1: C2.1, D1.CATHODE, L1.2, U9.PH
- new net N$10: C6.ANODE, D2.ANODE
- new net N$11: R4.1, R5.2, U10.VSENSE
- new net N$12: C10.1, C9.1, U10.COMP
- new net N$13: C10.2, R6.2
- new net N$14: C8.1, U10.SS
- new net N$2: C2.2, U9.BOOT
- new net N$3: C7.1, D2.CATHODE, L2.2, U10.PH
- new net N$4: C1.ANODE, D1.ANODE
- new net N$5: R1.1, R2.2, U9.VSENSE
- new net N$6: C4.1, C5.1, U9.COMP
- new net N$7: C5.2, R3.2
- new net N$8: C7.2, U10.BOOT
- new net N$9: C3.1, U9.SS
- new net VBATT: J1.VBATT+, U10.VIN, U9.VIN
Other:
- note added: "5v Rail 1"
- note added: "5v Rail 2"

Commit message: Switched to TPS54331, finished 5v rails
Parts:
- removed U$1, U$2: PCA9544A, signpost:PCA9544A
- added C11, C12, C13, C14, C19, C20, C21: (no value), passives:CAPACITOR0402_CAP
- added C15, C22, C23: 47u, passives:CAPACITOR1210_CAP
- added C16, C17, C24, C25: 4.7u, passives:CAPACITOR0402_CAP
- added C18, C26: 0.01u, passives:CAPACITOR0402_CAP
- added R10, R8: 68.1k, passives:RESISTOR0402_RES
- added R7, R9: 332k, passives:RESISTOR0402_RES
- added SJ1, SJ2, SJ3, SJ4, SJ5, SJ6: SOLDERJUMPERNC, SparkFun-Passives:SOLDERJUMPERNC
- added U11, U12: LTC2941-1, signpost:LTC2941-1
- C1: value EEEFK1A471P -> 47u; device signpost:EEEFK1A471P -> passives:CAPACITOR1210_CAP
- C10: value 220p -> (none)
- C3: value 14n -> 0.01u
- C4: value 220p -> 47p
- C5, C9: value 220p -> 1000p
- C6: value EEEFK1A471P -> 1u; device signpost:EEEFK1A471P -> passives:CAPACITOR0402_CAP
- C7: value 1u -> 0.01u
- C8: value 14n -> 47p
- L1, L2: value VLP8040 -> NR8040T6R8N; device signpost:VLP8040 -> signpost:NR8040T6R8N
- R2, R5: value 5k -> 4.99k
- R3, R6: value 30.9k -> 29.4k
- U1, U7: value LTC2941-1 -> PCA9544A; device signpost:LTC2941-1 -> signpost:PCA9544A
- U10: value TPS54233 -> LTC2941-1; device signpost:TPS54233 -> signpost:LTC2941-1
- U6: value LTC2941-1 -> TPS54233; device signpost:LTC2941-1 -> signpost:TPS54233
Connections:
- new net !INT: J1.!SMBALERT, U1.!INT, U7.!INT
- new net 3V3: U12.SENSE+
- new net N$15: U1.SD0, U2.SDA
- new net N$16: U1.SC0, U2.SCL
- new net N$17: U1.!INT0, U2.!ALERT
- new net N$18: U7.!INT0, U8.!ALERT
- new net N$19: U1.SD1, U3.SDA
- new net N$20: U1.SC1, U3.SCL
- new net N$21: U1.!INT1, U3.!ALERT
- new net N$22: U1.SD2, U4.SDA
- new net N$23: U1.SC2, U4.SCL
- new net N$24: U1.!INT2, U4.!ALERT
- new net N$25: U1.SD3, U5.SDA
- new net N$26: U1.SC3, U5.SCL
- new net N$27: U1.!INT3, U5.!ALERT
- new net N$31: U10.SDA, U7.SD1
- new net N$32: R7.1, R8.2, U9.EN
- new net N$33: U10.SCL, U7.SC1
- new net N$34: U10.!ALERT, U7.!INT1
- new net N$35: U11.SDA, U7.SD2
- new net N$36: U11.SCL, U7.SC2
- new net N$37: U11.!ALERT, U7.!INT2
- new net N$38: U12.SDA, U7.SD3
- new net N$39: U12.SCL, U7.SC3
- new net N$40: U12.!ALERT, U7.!INT3
- new net N$44: C8.1, C9.1, U6.COMP
- new net N$45: C7.1, U6.SS
- new net N$46: R10.2, R9.1, U6.EN
- new net SCL: J1.SMBCLK, U1.SCL, U7.SCL
- new net SDA: J1.SMBDATA, U1.SDA, U7.SDA
- new net VCC_BACKPLANE: C21.1, J1.VCC_BACKPLANE, J1.VCC_CONTROLLER, U1.VCC, U12.SENSE-, U7.VCC
- new net VCC_LINUX: C11.1, J1.VCC_LINUX, U2.SENSE-
- new net VCC_MOD0: C12.1, J1.VCC_MOD0, U3.SENSE-
- new net VCC_MOD1: C13.1, J1.VCC_MOD1, U4.SENSE-
- new net VCC_MOD2: C14.1, J1.VCC_MOD2, U5.SENSE-
- new net VCC_MOD5: C10.1, J1.VCC_MOD5, U8.SENSE-
- new net VCC_MOD6: C19.1, J1.VCC_MOD6, U10.SENSE-
- new net VCC_MOD7: C20.1, J1.VCC_MOD7, U11.SENSE-
- net 5V_1: now also C1.1, C15.1, SJ1.2, SJ2.2, SJ3.2, U2.SENSE+, U3.SENSE+, U4.SENSE+, U5.SENSE+; no longer C1.CATHODE
- net 5V_2: now also C22.1, C23.1, SJ4.2, SJ5.2, SJ6.2, U10.SENSE+, U11.SENSE+, U7.A0, U8.SENSE+; no longer C6.CATHODE
- net GND: now also C10.2, C11.2, C12.2, C13.2, C14.2, C16.2, C17.2, C18.2, C19.2, C20.2, C21.2, C24.2, C25.2, C26.2, C7.2, R10.1, R8.1, SJ1.1, SJ2.1, SJ3.1, SJ4.1, SJ5.1, SJ6.1, U1.A0, U1.A1, U1.A2, U1.GND, U11.GND, U12.GND, U2.GND, U3.GND, U4.GND, U5.GND, U6.GND, U7.A1, U7.A2, U7.GND, U8.GND; no longer C9.2
- net N$10: now also C22.2, C23.2; no longer C6.ANODE
- net N$11: now also U6.VSENSE; no longer U10.VSENSE
- net N$12: now also C9.2, R6.2; no longer C10.1, C9.1, U10.COMP
- net N$13: now also U7.SD0, U8.SDA; no longer C10.2, R6.2
- net N$14: now also U7.SC0, U8.SCL; no longer C8.1, U10.SS
- net N$3: now also C6.1, U6.PH; no longer C7.1, U10.PH
- net N$4: now also C1.2, C15.2; no longer C1.ANODE
- net N$8: now also C6.2, U6.BOOT; no longer C7.2, U10.BOOT
- net VBATT: now also C16.1, C17.1, C18.1, C24.1, C25.1, C26.1, R7.2, R9.2, U6.VIN; no longer U10.VIN
Other:
- note added: "5v Rail 1, Coulomb Counters"
- note added: "For: Linux, MOD0, MOD1, MOD2"
- note removed: "5v Rail 1"
- note removed: "5v Rail 2"
- moved on the sheet: C10, C2, C3, C4, C5, C7, C8, C9, D1, D2, L1, L2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

Commit message: Added 3v3 rail
Parts:
- added C27: 1u, passives:CAPACITOR0402_CAP
- added C28, C39: 0.01u, passives:CAPACITOR0402_CAP
- added C29: 47p, passives:CAPACITOR0402_CAP
- added C30: 1000p, passives:CAPACITOR0402_CAP
- added C35, C36: 47u, passives:CAPACITOR1210_CAP
- added C37, C38: 4.7u, passives:CAPACITOR0402_CAP
- added D3: B340A, signpost:B340A
- added L3: NR8040T6R8N, signpost:NR8040T6R8N
- added R11: 10.2k, passives:RESISTOR0402_RES
- added R12: 3.24k, passives:RESISTOR0402_RES
- added R13: 29.4k, passives:RESISTOR0402_RES
- added R14: 332k, passives:RESISTOR0402_RES
- added R15: 68.1k, passives:RESISTOR0402_RES
- added U13: TPS54233, signpost:TPS54233
Connections:
- new net N$28: C27.1, D3.CATHODE, L3.2, U13.PH
- new net N$29: C27.2, U13.BOOT
- new net N$30: C35.2, C36.2, D3.ANODE
- new net N$41: R11.1, R12.2, U13.VSENSE
- new net N$42: C30.2, R13.2
- new net N$58: C29.1, C30.1, U13.COMP
- new net N$59: C28.1, U13.SS
- new net N$60: R14.1, R15.2, U13.EN
- net 3V3: now also C35.1, C36.1, L3.1, R11.2
- net GND: now also C28.2, C29.2, C37.2, C38.2, C39.2, R12.1, R13.1, R15.1, U13.GND
- net VBATT: now also C37.1, C38.1, C39.1, R14.2, U13.VIN
Other:
- note added: "3v3 Rail"
- note added: "5v Rail 2, Coulomb Counters"
- note added: "For: MOD5, MOD6, MOD7, Backplane/Controller"

Commit message: Added additional 5v rails isolated linux switched to ltc2941 with external sense resistor for higher current
Parts:
- removed SJ1, SJ2, SJ3, SJ4, SJ5, SJ6: SOLDERJUMPERNC, SparkFun-Passives:SOLDERJUMPERNC
- added C31, C32, C33, C34, C40, C54, C55, C56: 0.1u, passives:CAPACITOR0402_CAP
- added C44, C46, C53: 0.01u, passives:CAPACITOR0402_CAP
- added C45: 1u, passives:CAPACITOR0402_CAP
- added C47: 47p, passives:CAPACITOR0402_CAP
- added C48: 1000p, passives:CAPACITOR0402_CAP
- added C49, C50: 47u, passives:CAPACITOR1210_CAP
- added C51, C52: 4.7u, passives:CAPACITOR0402_CAP
- added D4, D5: B340A, signpost:B340A
- added L4, L5: NR8040T6R8N, signpost:NR8040T6R8N
- added R16, R22: 10.2k, passives:RESISTOR0402_RES
- added R17, R24: 1.91k, passives:RESISTOR0402_RES
- added R18, R23, R28, R29, R30, R31, R32, R33: 0.017, passives:RESISTOR
- added R19, R25: 29.4k, passives:RESISTOR0402_RES
- added R20, R26: 332k, passives:RESISTOR0402_RES
- added R21, R27: 68.1k, passives:RESISTOR0402_RES
- added U14: PCA9544A, signpost:PCA9544A
- added U15: LTC2941, signpost:LTC2941
- C10, C11: value (none) -> 47u; device passives:CAPACITOR0402_CAP -> passives:CAPACITOR1210_CAP
- C12, C13: value (none) -> 4.7u
- C14, C20: value (none) -> 0.01u
- C19: value (none) -> 1u
- C21: value (none) -> 47p
- C22: value 47u -> 1000p; device passives:CAPACITOR1210_CAP -> passives:CAPACITOR0402_CAP
- C24: value 4.7u -> 47u; device passives:CAPACITOR0402_CAP -> passives:CAPACITOR1210_CAP
- C26: value 0.01u -> 4.7u
- R1, R4: value 10k -> 10.2k
- R2, R5: value 4.99k -> 1.91k
- U1, U7: value PCA9544A -> TPS54231; device signpost:PCA9544A -> signpost:TPS54231
- U10, U11, U12, U3, U4, U5, U8: value LTC2941-1 -> LTC2941; device signpost:LTC2941-1 -> signpost:LTC2941
- U13, U6, U9: value TPS54233 -> TPS54231; device signpost:TPS54233 -> signpost:TPS54231
- U2: value LTC2941-1 -> PCA9544A; device signpost:LTC2941-1 -> signpost:PCA9544A
Connections:
- new net 5V_3: C23.1, C24.1, L4.1, R16.2, R23.2, R31.2, U10.SENSE+, U11.SENSE+
- new net 5V_4: C49.1, C50.1, L5.1, R22.2, R32.2, U12.SENSE+
- new net N$43: U14.SD0, U3.SDA
- new net N$47: U14.SC0, U3.SCL
- new net N$48: U10.!ALERT, U2.!INT0
- new net N$49: U11.SDA, U2.SD1
- new net N$50: U11.SCL, U2.SC1
- new net N$51: U11.!ALERT, U2.!INT1
- new net N$52: U14.SD2, U5.SDA
- new net N$53: U14.SC2, U5.SCL
- new net N$54: U14.!INT2, U5.!ALERT
- new net N$55: U14.SD3, U8.SDA
- new net N$56: U14.SC3, U8.SCL
- new net N$57: U14.!INT3, U8.!ALERT
- new net N$67: U14.!INT0, U3.!ALERT
- new net N$68: U14.SD1, U4.SDA
- new net N$70: U14.SC1, U4.SCL
- new net N$71: U14.!INT1, U4.!ALERT
- net !INT: now also U14.!INT, U2.!INT; no longer U1.!INT, U7.!INT
- net 3V3: now also R33.2, U15.SENSE+; no longer U12.SENSE+
- net 5V_1: now also R18.2, R28.2; no longer SJ1.2, SJ2.2, SJ3.2, U2.SENSE+, U5.SENSE+
- net 5V_2: now also C10.1, C11.1, R29.2, R30.2, U5.SENSE+; no longer C22.1, C23.1, SJ4.2, SJ5.2, SJ6.2, U10.SENSE+, U11.SENSE+, U7.A0
- net GND: now also C31.2, C32.2, C33.2, C34.2, C40.2, C44.2, C46.2, C47.2, C51.2, C52.2, C53.2, C54.2, C55.2, C56.2, R17.1, R19.1, R21.1, R24.1, R25.1, R27.1, U14.A0, U14.A1, U14.A2, U14.GND, U15.GND, U2.A1, U2.A2; no longer C10.2, C11.2, C19.2, C24.2, SJ1.1, SJ2.1, SJ3.1, SJ4.1, SJ5.1, SJ6.1, U1.A0, U1.A1, U1.A2, U7.A1, U7.A2
- net N$10: now also C10.2, C11.2; no longer C22.2, C23.2
- net N$11: now also U1.VSENSE; no longer U6.VSENSE
- net N$13: now also C8.1, C9.1, U1.COMP; no longer U7.SD0, U8.SDA
- net N$14: now also C7.1, U1.SS; no longer U7.SC0, U8.SCL
- net N$15: now also R10.2, R9.1, U1.EN; no longer U1.SD0, U2.SDA
- net N$16: now also C19.1, D4.CATHODE, L4.2, U6.PH; no longer U1.SC0, U2.SCL
- net N$17: now also C19.2, U6.BOOT; no longer U1.!INT0, U2.!ALERT
- net N$18: now also C23.2, C24.2, D4.ANODE; no longer U7.!INT0, U8.!ALERT
- net N$19: now also R16.1, R17.2, U6.VSENSE; no longer U1.SD1, U3.SDA
- net N$20: now also C22.2, R19.2; no longer U1.SC1, U3.SCL
- net N$21: now also U10.SDA, U2.SD0; no longer U1.!INT1, U3.!ALERT
- net N$22: now also U10.SCL, U2.SC0; no longer U1.SD2, U4.SDA
- net N$23: now also U12.SDA, U2.SD2; no longer U1.SC2, U4.SCL
- net N$24: now also U12.SCL, U2.SC2; no longer U1.!INT2, U4.!ALERT
- net N$25: now also U12.!ALERT, U2.!INT2; no longer U1.SD3, U5.SDA
- net N$26: now also U15.SDA, U2.SD3; no longer U1.SC3, U5.SCL
- net N$27: now also U15.SCL, U2.SC3; no longer U1.!INT3, U5.!ALERT
- net N$3: now also U1.PH; no longer U6.PH
- net N$31: now also C21.1, C22.1, U6.COMP; no longer U10.SDA, U7.SD1
- net N$33: now also C20.1, U6.SS; no longer U10.SCL, U7.SC1
- net N$34: now also R20.1, R21.2, U6.EN; no longer U10.!ALERT, U7.!INT1
- net N$35: now also C45.1, D5.CATHODE, L5.2, U7.PH; no longer U11.SDA, U7.SD2
- net N$36: now also C45.2, U7.BOOT; no longer U11.SCL, U7.SC2
- net N$37: now also C49.2, C50.2, D5.ANODE; no longer U11.!ALERT, U7.!INT2
- net N$38: now also R22.1, R24.2, U7.VSENSE; no longer U12.SDA, U7.SD3
- net N$39: now also C48.2, R25.2; no longer U12.SCL, U7.SC3
- net N$40: now also C47.1, C48.1, U7.COMP; no longer U12.!ALERT, U7.!INT3
- net N$44: now also C46.1, U7.SS; no longer C8.1, C9.1, U6.COMP
- net N$45: now also R26.1, R27.2, U7.EN; no longer C7.1, U6.SS
- net N$46: now also U15.!ALERT, U2.!INT3; no longer R10.2, R9.1, U6.EN
- net N$8: now also U1.BOOT; no longer U6.BOOT
- net SCL: now also U14.SCL, U2.SCL; no longer U1.SCL, U7.SCL
- net SDA: now also U14.SDA, U2.SDA; no longer U1.SDA, U7.SDA
- net VBATT: now also C12.1, C13.1, C14.1, C44.1, C51.1, C52.1, C53.1, R20.2, R26.2, U1.VIN, U7.VIN; no longer C24.1
- net VCC_BACKPLANE: now also C40.1, R33.1, U14.VCC, U15.SENSE-, U2.A0, U2.VCC; no longer C21.1, U1.VCC, U12.SENSE-, U7.VCC
- net VCC_LINUX: now also C34.1, R32.1, U12.SENSE-; no longer C11.1, U2.SENSE-
- net VCC_MOD0: now also C31.1, R18.1; no longer C12.1
- net VCC_MOD1: now also C54.1, R28.1; no longer C13.1
- net VCC_MOD2: now also C55.1, R29.1; no longer C14.1
- net VCC_MOD5: now also C56.1, R30.1; no longer C10.1
- net VCC_MOD6: now also C32.1, R23.1; no longer C19.1
- net VCC_MOD7: now also C33.1, R31.1; no longer C20.1
Other:
- note added: "5v Rail 1"
- note added: "5v Rail 2"
- note added: "5v Rail 3"
- note added: "5v Rail 4"
- note added: "Coulomb Counters"
- note added: "For MOD0, MOD1, MOD2, MOD5"
- note added: "For MOD6-7, LINUX, BACKPLANE/CONTROLLER"
- note added: "Power Module Header"
- note removed: "5v Rail 1, Coulomb Counters"
- note removed: "5v Rail 2, Coulomb Counters"
- note removed: "For: Linux, MOD0, MOD1, MOD2"
- note removed: "For: MOD5, MOD6, MOD7, Backplane/Controller"

Commit message: Switched regulator yet again
Parts:
- removed C17, C25, C26, C37, C38, C51, C52: 4.7u, passives:CAPACITOR0402_CAP
- removed C18, C20, C28, C39, C44, C46, C53: 0.01u, passives:CAPACITOR0402_CAP
- removed C19, C27, C45: 1u, passives:CAPACITOR0402_CAP
- removed C21, C29, C47: 47p, passives:CAPACITOR0402_CAP
- removed C22, C30, C48: 1000p, passives:CAPACITOR0402_CAP
- removed C23, C24, C35, C36, C49, C50: 47u, passives:CAPACITOR1210_CAP
- removed D1, D2, D3, D4, D5: B340A, signpost:B340A
- removed L5: NR8040T6R8N, signpost:NR8040T6R8N
- removed R13, R19, R25: 29.4k, passives:RESISTOR0402_RES
- removed R14, R20, R26: 332k, passives:RESISTOR0402_RES
- removed R15, R21, R27: 68.1k, passives:RESISTOR0402_RES
- removed R16, R22: 10.2k, passives:RESISTOR0402_RES
- removed R17, R24: 1.91k, passives:RESISTOR0402_RES
- added C41: 10uF, passives:CAPACITOR0402_CAP
- added C42: 0.1uF, passives:CAPACITOR0402_CAP
- added C43: 3.3nF, passives:CAPACITOR0402_CAP
- added C57: 22uF, passives:CAPACITOR0402_CAP
- added L6: 2.2uH, passives:INDUCTORIHL
- added R34: 750k, passives:RESISTOR0402_RES
- added R35: 240k, passives:RESISTOR0402_RES
- added R36: 100K, passives:RESISTOR0402_RES
- C1: value 47u -> 10uF; device passives:CAPACITOR1210_CAP -> passives:CAPACITOR0402_CAP
- C10: value 47u -> 0.1uF; device passives:CAPACITOR1210_CAP -> passives:CAPACITOR0402_CAP
- C11, C15: value 47u -> 3.3nF; device passives:CAPACITOR1210_CAP -> passives:CAPACITOR0402_CAP
- C12, C16: value 4.7u -> 22uF
- C13: value 4.7u -> 10uF
- C14: value 0.01u -> 0.1uF
- C2, C6: value 1u -> 0.1uF
- C3, C7: value 0.01u -> 3.3nF
- C4, C8: value 47p -> 22uF
- C5, C9: value 1000p -> 10uF
- L1, L2, L3, L4: value NR8040T6R8N -> 2.2uH; device signpost:NR8040T6R8N -> passives:INDUCTORIHL
- R1, R4: value 10.2k -> 750k
- R10: value 68.1k -> 750k
- R11: value 10.2k -> 143k
- R12: value 3.24k -> 100K
- R18, R23, R28, R29, R30, R31, R32, R33: device passives:RESISTOR -> passives:RESISTOR0805_RES
- R2, R5: value 1.91k -> 143k
- R3, R6: value 29.4k -> 100K
- R7: value 332k -> 750k
- R8: value 68.1k -> 143k
- R9: value 332k -> 100K
- U1, U13, U6, U7, U9: value TPS54231 -> TLV62130; device signpost:TPS54231 -> chips:TLV62130
Connections:
- removed net N$17: C19.2, U6.BOOT
- removed net N$18: C23.2, C24.2, D4.ANODE
- removed net N$19: R16.1, R17.2, U6.VSENSE
- removed net N$20: C22.2, R19.2
- removed net N$28: C27.1, D3.CATHODE, L3.2, U13.PH
- removed net N$29: C27.2, U13.BOOT
- removed net N$30: C35.2, C36.2, D3.ANODE
- removed net N$31: C21.1, C22.1, U6.COMP
- removed net N$32: R7.1, R8.2, U9.EN
- removed net N$33: C20.1, U6.SS
- removed net N$34: R20.1, R21.2, U6.EN
- removed net N$35: C45.1, D5.CATHODE, L5.2, U7.PH
- removed net N$36: C45.2, U7.BOOT
- removed net N$37: C49.2, C50.2, D5.ANODE
- removed net N$38: R22.1, R24.2, U7.VSENSE
- removed net N$39: C48.2, R25.2
- removed net N$40: C47.1, C48.1, U7.COMP
- removed net N$41: R11.1, R12.2, U13.VSENSE
- removed net N$42: C30.2, R13.2
- removed net N$44: C46.1, U7.SS
- removed net N$45: R26.1, R27.2, U7.EN
- removed net N$58: C29.1, C30.1, U13.COMP
- removed net N$59: C28.1, U13.SS
- removed net N$60: R14.1, R15.2, U13.EN
- new net N$61: C43.2, U6.SS/TR
- new net N$62: L6.1, U6.SW
- new net N$63: R36.1, U6.PG
- new net N$64: R34.1, R35.2, U6.FB
- net 3V3: now also C57.2, L6.2, R34.2, R36.2, U6.VOS; no longer C35.1, C36.1, L3.1, R11.2
- net 5V_1: now also C4.2, L1.2, R3.2, U1.VOS; no longer C1.1, C15.1, L1.1
- net 5V_2: now also C8.2, L2.2, R6.2, U7.VOS; no longer C10.1, C11.1, L2.1
- net 5V_3: now also C12.2, L3.2, R7.2, R9.2, U9.VOS; no longer C23.1, C24.1, L4.1, R16.2
- net 5V_4: now also C16.2, L4.2, R10.2, R12.2, U13.VOS; no longer C49.1, C50.1, L5.1, R22.2
- net GND: now also C1.2, C10.2, C11.1, C12.1, C15.1, C16.1, C2.2, C3.1, C4.1, C41.2, C42.2, C43.1, C5.2, C57.1, C6.2, C7.1, C8.1, C9.2, R11.1, R35.1, U1.AGND, U1.DEF, U1.FSW, U1.PGND, U13.AGND, U13.DEF, U13.FSW, U13.PGND, U6.AGND, U6.DEF, U6.FSW, U6.PGND, U7.AGND, U7.DEF, U7.FSW, U7.PGND, U9.AGND, U9.DEF, U9.FSW, U9.PGND; no longer C12.2, C16.2, C17.2, C18.2, C20.2, C21.2, C25.2, C26.2, C28.2, C29.2, C3.2, C37.2, C38.2, C39.2, C4.2, C44.2, C46.2, C47.2, C51.2, C52.2, C53.2, C7.2, C8.2, R10.1, R12.1, R13.1, R15.1, R17.1, R19.1, R21.1, R24.1, R25.1, R27.1, R3.1, R6.1, U1.GND, U13.GND, U6.GND, U7.GND, U9.GND
- net N$1: now also C7.2, U7.SS/TR; no longer C2.1, D1.CATHODE, L1.2, U9.PH
- net N$10: now also L3.1, U9.SW; no longer C10.2, C11.2, D2.ANODE
- net N$11: now also R9.1, U9.PG; no longer R4.1, R5.2, U1.VSENSE
- net N$12: now also R7.1, R8.2, U9.FB; no longer C9.2, R6.2
- net N$13: now also C15.2, U13.SS/TR; no longer C8.1, C9.1, U1.COMP
- net N$14: now also L4.1, U13.SW; no longer C7.1, U1.SS
- net N$15: now also R12.1, U13.PG; no longer R10.2, R9.1, U1.EN
- net N$16: now also R10.1, R11.2, U13.FB; no longer C19.1, D4.CATHODE, L4.2, U6.PH
- net N$2: now also L2.1, U7.SW; no longer C2.2, U9.BOOT
- net N$3: now also R6.1, U7.PG; no longer C6.1, D2.CATHODE, L2.2, U1.PH
- net N$4: now also R4.1, R5.2, U7.FB; no longer C1.2, C15.2, D1.ANODE
- net N$5: now also C3.2, U1.SS/TR; no longer R1.1, R2.2, U9.VSENSE
- net N$6: now also L1.1, U1.SW; no longer C3.1, U9.SS
- net N$7: now also R3.1, U1.PG; no longer C5.2, R3.2
- net N$8: now also C11.2, U9.SS/TR; no longer C6.2, U1.BOOT
- net N$9: now also R1.1, R2.2, U1.FB; no longer C4.1, C5.1, U9.COMP
- net VBATT: now also C1.1, C10.1, C2.1, C41.1, C42.1, C5.1, C6.1, C9.1, U1.AVIN, U1.EN, U1.PVIN, U13.AVIN, U13.EN, U13.PVIN, U6.AVIN, U6.EN, U6.PVIN, U7.AVIN, U7.EN, U7.PVIN, U9.AVIN, U9.EN, U9.PVIN; no longer C12.1, C16.1, C17.1, C18.1, C25.1, C26.1, C37.1, C38.1, C39.1, C44.1, C51.1, C52.1, C53.1, R14.2, R20.2, R26.2, R7.2, R9.2, U1.VIN, U13.VIN, U6.VIN, U7.VIN, U9.VIN
