File: hardware/controller/rev_a/controller.sch (EAGLE design)
At the start: 85 parts, among them J1 MODULE_CONTROLLER, J2 DM3AT-SF-PEJM5, J3 U.FL-R-SMT, J4 MICRO_USB_B_HIROSE_ZX62-B-5PA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, J5 MICRO_USB_B_HIROSE_ZX62-B-5PA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, J6 TC2030-JLINK-L, J7 TC2030-JLINK-L, Q1 MOSFET-NCHANNELSMD, Q2 NX3008PBK, U1 SAM4LC8AA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

Commit message: Controller fully routed!!!!
Parts:
- added J8: JUMPER-3PTH, umich:JUMPER-3PTH
- added JP1, JP2: (no value), umich:JUMPER-2PTH
- added JP3: (no value), pinhead:PINHD-2X10
- added SJ1: (no value), SparkFun-Passives:SOLDERJUMPER_2WAYPASTE2&3
- added SJ2: SOLDERJUMPERTRACE, SparkFun-Passives:SOLDERJUMPERTRACE
- added U6: PTS810SJ, switches:PTS810SJ
Connections:
- net N$27 renamed MODULES_SDA_1V8
- net N$42 renamed MODULES_SCL_1V8
- removed net !FRAM_CS/CONTROLLER_LED: R21.2, U1.PA25, U4.!CS
- removed net CONTROLLER_SWDIO/!STORAGE_CS: J7.SWDIO, R16.1, U1.PA03, U2.PA09
- removed net N$23: E_1_SPI.GP111_SPI_2_FS1, U8.A4
- removed net N$39: E_1_SPI.GP109_SPI_2_CLK, U8.A3
- removed net N$40: E_1_SPI.GP115_SPI_2_TXD, U8.A2
- removed net N$41: E_1_SPI.GP114_SPI_2_RXD, U8.A1
- new net !CONTROLLER_LED: JP2.2, R21.2
- new net !EDISON_SPI_CS_1V8: JP3.13, SJ1.2, U8.A4
- new net !FRAM_CS: JP2.1, JP3.9, U1.PA25, U4.!CS
- new net !STORAGE_CS: JP1.2, JP3.8, U2.PA09
- new net CONTROLLER_SWDIO: J7.SWDIO, JP1.1, R16.1, U1.PA03
- new net EDISON_SPI_MISO_1V8: E_1_SPI.GP109_SPI_2_CLK, JP3.12, U8.A3
- new net EDISON_SPI_MOSI_1V8: E_1_SPI.GP115_SPI_2_TXD, JP3.11, U8.A2
- new net EDISON_SPI_SCLK_1V8: E_1_SPI.GP114_SPI_2_RXD, JP3.10, U8.A1
- new net N$13: E_1_SPI.GP111_SPI_2_FS1, SJ1.3
- new net N$15: D1.CATHODE, SJ2.2
- new net N$16: J8.1, R3.2, R4.1
- net !BACKPLANE_RESET: now also U6.P$1
- net !SD_CS: now also JP3.4
- net GND: now also JP3.19, U6.P$2
- net GPS_IN_RX: now also JP3.15
- net GPS_OUT_TX: now also JP3.16
- net MEMORY_MISO: now also JP3.7
- net MEMORY_MOSI: now also JP3.5
- net MEMORY_SCLK: now also JP3.6
- net N$11: now also SJ1.1
- net SD_MISO: now also JP3.2
- net SD_MOSI: now also JP3.1
- net SD_SCLK: now also JP3.3
- net USB_ATTACHED_3V3: now also J8.2; no longer R3.2, R4.1
- net VCC_CONTROLLER: now also JP3.20
- net VCC_LINUX: now also JP3.17, SJ2.1; no longer D1.CATHODE
- net VCC_LINUX_1V8: now also JP3.14
- net VCC_LINUX_3V3: now also J8.3, JP3.18
Other:
- note added: "XXX Test points * GPS UART & PPS * Storage SPI * SD SPI * Edison SPI * Voltages"
- note removed: "Check VCCA vs VCCB"
- note removed: "XXX Button"
- note removed: "XXX Jumper me"
- note removed: "XXX Test points ? Modules I2C * GPS UART & PPS * Storage SPI * SD SPI * Edison SPI ? SMBUS & ALERT * Voltages"
- moved on the sheet: C23, C24, D1, E_1_SPI, FB2, J3, R3, R4, U3, U4

Commit message: Revised value prefix format
Parts:
- FB1: value 600 ohm -> 600 Ω
- FB2: value 300 ohm -> 300 Ω
- FB3, FB4: value 1.5 k -> 1.5 kΩ
- R1, R2: value 27 -> 27 Ω
- R10, R18, R22, R23, R24, R25: value 10 k -> 10 kΩ
- R11, R12, R13: value 1 k -> 1 kΩ
- R14, R15, R16, R17, R26: value 100 k -> 100 kΩ
- R19, R20, R21: value 1k -> 1 kΩ
- R3: value 665 k -> 665 kΩ
- R4: value 332 k -> 332 kΩ
- R5, R6: value 100 -> 100 Ω
- R9: value 1 M -> 1 MΩ
Changed lines of the file:
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@@
 </part>
 <part name="J2" library="connector" deviceset="DM3AT-SF-PEJM5" device=""/>
-<part name="FB2" library="passives" deviceset="FERRITE_BEAD" device="0402" value="300 ohm">
+<part name="FB2" library="passives" deviceset="FERRITE_BEAD" device="0402" value="300 Ω">
 <attribute name="DIGIKEY" value="ACML-0402-301-TCT-ND"/>
 </part>
@@
 <attribute name="DIGIKEY" value="490-6241-1-ND"/>
 </part>
-<part name="R1" library="passives" deviceset="RESISTOR" device="0402_RES" value="27">
+<part name="R1" library="passives" deviceset="RESISTOR" device="0402_RES" value="27 Ω">
 <attribute name="DIGIKEY" value="1276-3907-1-ND"/>
 </part>
-<part name="R2" library="passives" deviceset="RESISTOR" device="0402_RES" value="27">
+<part name="R2" library="passives" deviceset="RESISTOR" device="0402_RES" value="27 Ω">
 <attribute name="DIGIKEY" value="1276-3907-1-ND"/>
 </part>
 <part name="GND12" library="supply1" deviceset="GND" device=""/>
 <part name="GND13" library="supply1" deviceset="GND" device=""/>
-<part name="R5" library="passives" deviceset="RESISTOR" device="0402_RES" value="100">
+<part name="R5" library="passives" deviceset="RESISTOR" device="0402_RES" value="100 Ω">
 <attribute name="DIGIKEY" value="1276-3429-1-ND"/>
 </part>
-<part name="R6" library="passives" deviceset="RESISTOR" device="0402_RES" value="100">
+<part name="R6" library="passives" deviceset="RESISTOR" device="0402_RES" value="100 Ω">
 <attribute name="DIGIKEY" value="1276-3429-1-ND"/>
 </part>
-<part name="R3" library="passives" deviceset="RESISTOR" device="0402_RES" value="665 k">
+<part name="R3" library="passives" deviceset="RESISTOR" device="0402_RES" value="665 kΩ">
 <attribute name="DIGIKEY" value="1276-4275-1-ND"/>
 </part>
-<part name="R4" library="passives" deviceset="RESISTOR" device="0402_RES" value="332 k">
+<part name="R4" library="passives" deviceset="RESISTOR" device="0402_RES" value="332 kΩ">
 <attribute name="DIGIKEY" value="1276-4245-1-ND"/>
 </part>
@@
 <part name="S1" library="signpost" deviceset="SIP3240X" device=""/>
 <part name="GND18" library="umich" deviceset="GND" device=""/>
-<part name="R9" library="passives" deviceset="RESISTOR" device="0402_RES" value="1 M">
+<part name="R9" library="passives" deviceset="RESISTOR" device="0402_RES" value="1 MΩ">
 <attribute name="DIGIKEY" value="1276-3433-1-ND"/>
 </part>
@@
 <part name="D3" library="leds" deviceset="SML-LX0404SIUPGUSB" device=""/>
 <part name="U$13" library="signpost" deviceset="VCC_LINUX_3V3" device=""/>
-<part name="R11" library="passives" deviceset="RESISTOR" device="0402_RES" value="1 k">
-<attribute name="DIGIKEY" value="1276-3430-1-ND"/>
-</part>
-<part name="R12" library="passives" deviceset="RESISTOR" device="0402_RES" value="1 k">
-<attribute name="DIGIKEY" value="1276-3430-1-ND"/>
-</part>
-<part name="R13" library="passives" deviceset="RESISTOR" device="0402_RES" value="1 k">
+<part name="R11" library="passives" deviceset="RESISTOR" device="0402_RES" value="1 kΩ">
+<attribute name="DIGIKEY" value="1276-3430-1-ND"/>
+</part>
+<part name="R12" library="passives" deviceset="RESISTOR" device="0402_RES" value="1 kΩ">
+<attribute name="DIGIKEY" value="1276-3430-1-ND"/>
+</part>
+<part name="R13" library="passives" deviceset="RESISTOR" device="0402_RES" value="1 kΩ">
 <attribute name="DIGIKEY" value="1276-3430-1-ND"/>
 </part>
@@
 <attribute name="DIGIKEY" value="490-10777-1-ND"/>
 </part>
-<part name="FB3" library="passives" deviceset="FERRITE_BEAD" device="0402" value="1.5 k">
+<part name="FB3" library="passives" deviceset="FERRITE_BEAD" device="0402" value="1.5 kΩ">
 <attribute name="DIGIKEY" value="490-5216-1-ND"/>
 </part>
@@
 </part>
 <part name="U$18" library="signpost" deviceset="VCC_CONTROLLER" device=""/>
-<part name="R10" library="passives" deviceset="RESISTOR" device="0402_RES" value="10 k">
+<part name="R10" library="passives" deviceset="RESISTOR" device="0402_RES" value="10 kΩ">
 <attribute name="DIGIKEY" value="1276-3431-1-ND"/>
 </part>
@@
 <part name="X1" library="crystals" deviceset="FH1600015" device="" value="16 MHz"/>
 <part name="GND26" library="umich" deviceset="GND" device=""/>
-<part name="R14" library="passives" deviceset="RESISTOR" device="0402_RES" value="100 k">
-<attribute name="DIGIKEY" value="1276-3432-1-ND"/>
-</part>
-<part name="R15" library="passives" deviceset="RESISTOR" device="0402_RES" value="100 k">
+<part name="R14" library="passives" deviceset="RESISTOR" device="0402_RES" value="100 kΩ">
+<attribute name="DIGIKEY" value="1276-3432-1-ND"/>
+</part>
+<part name="R15" library="passives" deviceset="RESISTOR" device="0402_RES" value="100 kΩ">
 <attribute name="DIGIKEY" value="1276-3432-1-ND"/>
 </part>
@@
 <part name="U$9" library="signpost" deviceset="VCC_CONTROLLER" device=""/>
 <part name="GND19" library="umich" deviceset="GND" device=""/>
-<part name="R16" library="passives" deviceset="RESISTOR" device="0402_RES" value="100 k">
-<attribute name="DIGIKEY" value="1276-3432-1-ND"/>
-</part>
-<part name="R17" library="passives" deviceset="RESISTOR" device="0402_RES" value="100 k">
+<part name="R16" library="passives" deviceset="RESISTOR" device="0402_RES" value="100 kΩ">
+<attribute name="DIGIKEY" value="1276-3432-1-ND"/>
+</part>
+<part name="R17" library="passives" deviceset="RESISTOR" device="0402_RES" value="100 kΩ">
 <attribute name="DIGIKEY" value="1276-3432-1-ND"/>
 </part>
@@
 <part name="X2" library="crystals" deviceset="FH1600015" device="" value="16 MHz"/>
 <part name="GND20" library="umich" deviceset="GND" device=""/>
-<part name="R18" library="passives" deviceset="RESISTOR" device="0402_RES" value="10 k">
+<part name="R18" library="passives" deviceset="RESISTOR" device="0402_RES" value="10 kΩ">
 <attribute name="DIGIKEY" value="1276-3431-1-ND"/>
 </part>
@@
 <attribute name="DIGIKEY" value="490-10777-1-ND"/>
 </part>
-<part name="FB4" library="passives" deviceset="FERRITE_BEAD" device="0402" value="1.5 k">
+<part name="FB4" library="passives" deviceset="FERRITE_BEAD" device="0402" value="1.5 kΩ">
 <attribute name="DIGIKEY" value="490-5216-1-ND"/>
 </part>
@@
 <part name="U$22" library="signpost" deviceset="VCC_CONTROLLER" device=""/>
 <part name="D2" library="leds" deviceset="SML-LX0404SIUPGUSB" device=""/>
-<part name="R19" library="passives" deviceset="RESISTOR" device="0402_RES" value="1k">
-<attribute name="DIGIKEY" value="1276-3430-1-ND"/>
-</part>
-<part name="R20" library="passives" deviceset="RESISTOR" device="0402_RES" value="1k">
-<attribute name="DIGIKEY" value="1276-3430-1-ND"/>
-</part>
-<part name="R21" library="passives" deviceset="RESISTOR" device="0402_RES" value="1k">
+<part name="R19" library="passives" deviceset="RESISTOR" device="0402_RES" value="1 kΩ">
+<attribute name="DIGIKEY" value="1276-3430-1-ND"/>
+</part>
+<part name="R20" library="passives" deviceset="RESISTOR" device="0402_RES" value="1 kΩ">
+<attribute name="DIGIKEY" value="1276-3430-1-ND"/>
+</part>
+<part name="R21" library="passives" deviceset="RESISTOR" device="0402_RES" value="1 kΩ">
 <attribute name="DIGIKEY" value="1276-3430-1-ND"/>
 </part>
@@
 <part name="U$24" library="signpost" deviceset="VCC_CONTROLLER" device=""/>
 <part name="Q2" library="fets" deviceset="NX3008PBK" device=""/>
-<part name="R22" library="passives" deviceset="RESISTOR" device="0402_RES" value="10 k">
-<attribute name="DIGIKEY" value="1276-3431-1-ND"/>
-</part>
-<part name="R23" library="passives" deviceset="RESISTOR" device="0402_RES" value="10 k">
-<attribute name="DIGIKEY" value="1276-3431-1-ND"/>
-</part>
-<part name="R24" library="passives" deviceset="RESISTOR" device="0402_RES" value="10 k">
-<attribute name="DIGIKEY" value="1276-3431-1-ND"/>
-</part>
-<part name="R25" library="passives" deviceset="RESISTOR" device="0402_RES" value="10 k">
-<attribute name="DIGIKEY" value="1276-3431-1-ND"/>
-</part>
-<part name="R26" library="passives" deviceset="RESISTOR" device="0402_RES" value="100 k">
+<part name="R22" library="passives" deviceset="RESISTOR" device="0402_RES" value="10 kΩ">
+<attribute name="DIGIKEY" value="1276-3431-1-ND"/>
+</part>
+<part name="R23" library="passives" deviceset="RESISTOR" device="0402_RES" value="10 kΩ">
+<attribute name="DIGIKEY" value="1276-3431-1-ND"/>
+</part>
+<part name="R24" library="passives" deviceset="RESISTOR" device="0402_RES" value="10 kΩ">
+<attribute name="DIGIKEY" value="1276-3431-1-ND"/>
+</part>
+<part name="R25" library="passives" deviceset="RESISTOR" device="0402_RES" value="10 kΩ">
+<attribute name="DIGIKEY" value="1276-3431-1-ND"/>
+</part>
+<part name="R26" library="passives" deviceset="RESISTOR" device="0402_RES" value="100 kΩ">
 <attribute name="DIGIKEY" value="1276-3432-1-ND"/>
 </part>
@@
 </part>
 <part name="GND33" library="umich" deviceset="GND" device=""/>
-<part name="FB1" library="passives" deviceset="FERRITE_BEAD" device="0805" value="600 ohm">
+<part name="FB1" library="passives" deviceset="FERRITE_BEAD" device="0805" value="600 Ω">
 <attribute name="DIGIKEY" value="240-2390-1-ND"/>
 </part>

Commit message: Remove space between numbers and units
Also added more descriptions to schematic
Parts:
- C1, C2: value 47 pF -> 47pF
- C10, C16, C17, C18, C19, C20, C23, C24, C25, C26, C27, C28, C30, C6, C7, C8, C9: value 100 nF -> 100nF
- C11, C21, C22: value 4.7 uF -> 4.7uF
- C12, C13, C14, C15: value 8 pF -> 8pF
- C29: value 10 nF -> 10nF
- C3, C5: value 10 uF -> 10uF
- C4: value 22 uF -> 22uF
- FB1: value 600 Ω -> 600Ω
- FB2: value 300 Ω -> 300Ω
- FB3, FB4: value 1.5 kΩ -> 1.5kΩ
- L2: value 0.47 uH -> 0.47uH
- L4, L6: value 22 uH -> 22uH
- R1, R2: value 27 Ω -> 27Ω
- R10, R18, R22, R23, R24, R25: value 10 kΩ -> 10kΩ
- R11, R12, R13, R19, R20, R21: value 1 kΩ -> 1kΩ
- R14, R15, R16, R17, R26: value 100 kΩ -> 100kΩ
- R3: value 665 kΩ -> 665kΩ
- R4: value 332 kΩ -> 332kΩ
- R5, R6: value 100 Ω -> 100Ω
- R9: value 1 MΩ -> 1MΩ
- X1, X2: value 16 MHz -> 16MHz
Other:
- note added: "Backplane Reset Button"
- note added: "Controller & Storage Master LED"
- note added: "FRAM Storage"
- note added: "GPS"
- note added: "JLINK Programming Header"
- note added: "SD Card Adapter"
- note added: "Signpost Headers"
- note added: "Test Points"
- note removed: "XXX SAM4L Thermal pad vias"
- note removed: "XXX Test points * GPS UART & PPS * Storage SPI * SD SPI * Edison SPI * Voltages"

Commit message: Schematic part numbers updated! BOM generated
Parts:
- removed L4: 22uH, signpost:LHQ3NP
- removed R25: 10kΩ, passives:RESISTOR0402_RES
- removed R26: 100kΩ, passives:RESISTOR0402_RES
- added L1: 0.47uH, passives:INDUCTORDFE322512C
- added LOGO1: UMICH_SOLID_MEDIUM, logos:UMICH_SOLID_MEDIUM
- added R7, R8: 1kΩ, passives:RESISTOR0402_RES
- C1, C2: value 47pF -> 8pF; DIGIKEY 490-6241-1-ND -> 490-8230-1-ND
- C11, C21, C22: value 4.7uF -> 100nF; DIGIKEY 490-13252-1-ND -> 490-10777-1-ND
- C12, C13, C14, C15: value 8pF -> 100nF; DIGIKEY 490-8230-1-ND -> 490-10777-1-ND
- C25, C26, C27: value 100nF -> 4.7uF; DIGIKEY 490-10777-1-ND -> 490-13252-1-ND
- C28: value 100nF -> 10uF; device passives:CAPACITOR0402_CAP -> passives:CAPACITOR0805_CAP; DIGIKEY 490-10777-1-ND -> 490-8316-1-ND
- C29: value 10nF -> 10uF; DIGIKEY 490-6296-1-ND -> 490-13811-1-ND
- C3: value 10uF -> 8pF; device passives:CAPACITOR0805_CAP -> passives:CAPACITOR0402_CAP; DIGIKEY 490-8316-1-ND -> 490-8230-1-ND
- C30: value 100nF -> 22uF; device passives:CAPACITOR0402_CAP -> passives:CAPACITOR0805_CAP; DIGIKEY 490-10777-1-ND -> 490-1719-1-ND
- C4: value 22uF -> 8pF; device passives:CAPACITOR0805_CAP -> passives:CAPACITOR0402_CAP; DIGIKEY 490-1719-1-ND -> 490-8230-1-ND
- C5: value 10uF -> 47pF; DIGIKEY 490-13811-1-ND -> 490-6241-1-ND
- C6: value 100nF -> 47pF; DIGIKEY 490-10777-1-ND -> 490-6241-1-ND
- C7: value 100nF -> 10nF; DIGIKEY 490-10777-1-ND -> 490-6296-1-ND
- FB1: value 600Ω -> 300Ω; device passives:FERRITE_BEAD0805 -> passives:FERRITE_BEAD0402; DIGIKEY 240-2390-1-ND -> ACML-0402-301-TCT-ND
- FB2: value 300Ω -> 600Ω; device passives:FERRITE_BEAD0402 -> passives:FERRITE_BEAD0805; DIGIKEY ACML-0402-301-TCT-ND -> 240-2390-1-ND
- L2: value 0.47uH -> 22uH; device passives:INDUCTORDFE322512C -> signpost:LHQ3NP; MOUSER 81-1277AS-H-R47MP2 -> (none)
- R10: value 10kΩ -> 1kΩ; DIGIKEY 1276-3431-1-ND -> 1276-3430-1-ND
- R11, R12, R13: value 1kΩ -> 10kΩ; DIGIKEY 1276-3430-1-ND -> 1276-3431-1-ND
- R14, R15, R16: value 100kΩ -> 10kΩ; DIGIKEY 1276-3432-1-ND -> 1276-3431-1-ND
- R18: value 10kΩ -> 100kΩ; DIGIKEY 1276-3431-1-ND -> 1276-3432-1-ND
- R19, R20, R21: value 1kΩ -> 100kΩ; DIGIKEY 1276-3430-1-ND -> 1276-3432-1-ND
- R22: value 10kΩ -> 332kΩ; DIGIKEY 1276-3431-1-ND -> 1276-4245-1-ND
- R23: value 10kΩ -> 665kΩ; DIGIKEY 1276-3431-1-ND -> 1276-4275-1-ND
- R24: value 10kΩ -> 1MΩ; DIGIKEY 1276-3431-1-ND -> 1276-3433-1-ND
- R3: value 665kΩ -> 100Ω; DIGIKEY 1276-4275-1-ND -> 1276-3429-1-ND
- R4: value 332kΩ -> 100Ω; DIGIKEY 1276-4245-1-ND -> 1276-3429-1-ND
- R5, R6: value 100Ω -> 1kΩ; DIGIKEY 1276-3429-1-ND -> 1276-3430-1-ND
- R9: value 1MΩ -> 1kΩ; DIGIKEY 1276-3433-1-ND -> 1276-3430-1-ND
- renumbered L6 to L3, S1 to SW2, U6 to SW1
Connections:
- net !CONTROLLER_LED: now also R10.2; no longer R21.2
- net !SD_CS: now also R15.1; no longer R24.1
- net !STORAGE_LED: now also R9.2; no longer R20.2
- net CONTROLLER_BUCK/LDO_N: now also R12.1; no longer R18.1
- net CONTROLLER_SWDCLK: now also R20.1; no longer R17.1
- net CONTROLLER_SWDIO: now also R19.1; no longer R16.1
- net CONTROLLER_XIN: now also C3.1; no longer C14.1
- net CONTROLLER_XOUT: now also C4.1; no longer C15.1
- net D+: now also C6.1; no longer C2.1
- net D-: now also C5.1; no longer C1.1
- net EDISON_UART_RX: now also R3.2; no longer R5.2
- net EDISON_UART_TX: now also R4.2; no longer R6.2
- net GND: now also C21.1, C24.1, C26.2, C30.2, R13.1, R23.1, R5.2, R8.2; no longer C21.2, C24.2, C26.1, C30.1, R11.2, R19.2, R22.1, R3.1
- net LINUX_5V_IN: now also C28.1; no longer C3.1
- net LINUX_ENABLE_POWER: now also R24.1; no longer R9.1
- net N$1: now also FB1.P$1; no longer FB2.P$1
- net N$10: now also FB2.P$2; no longer FB1.P$2
- net N$12: now also R7.2; no longer R13.2
- net N$14: now also L1.1; no longer L2.1
- net N$16: now also R22.1, R23.2; no longer R3.2, R4.1
- net N$17: now also C27.1, R14.2, R15.2, R16.2, R21.2; no longer C22.1, R23.2, R24.2, R25.2, R26.2
- net N$24: now also R3.1; no longer R5.1
- net N$25: now also R4.1; no longer R6.1
- net N$28: now also C7.1, FB2.P$1; no longer C29.1, FB1.P$1
- net N$29: now also C8.1; no longer C6.1
- net N$3: now also FB1.P$2; no longer FB2.P$2
- net N$32: now also C13.1; no longer C16.1
- net N$34: now also R5.1; no longer R11.1
- net N$37: now also R6.1; no longer R12.1
- net N$38: now also R7.1; no longer R13.1
- net N$44: now also C17.1, C26.1; no longer C20.1, C21.1
- net N$45: now also C12.1, C25.1, L2.1; no longer C10.1, C11.1, L4.1
- net N$46: now also L2.2; no longer L4.2
- net N$50: now also R6.2; no longer R12.2
- net N$7: now also R8.1; no longer R19.1
- net N$8: now also R9.1; no longer R20.1
- net N$9: now also R10.1; no longer R21.1
- net SD_DETECT: now also R21.1; no longer R26.1
- net SD_ENABLE: now also R13.2; no longer R22.2
- net SD_MISO: now also R16.1; no longer R25.1
- net SD_MOSI: now also R14.1; no longer R23.1
- net STORAGE_BUCK/LDO_N: now also R11.1; no longer R10.1
- net STORAGE_SWDCLK: now also R18.1; no longer R15.1
- net STORAGE_SWDIO: now also R17.1; no longer R14.1
- net STORAGE_XIN: now also C1.1; no longer C12.1
- net STORAGE_XOUT: now also C2.1; no longer C13.1
- net USB_VBUS: now also R22.2; no longer R4.2
- net VCC_CONTROLLER: now also C10.1, C11.1, C14.1, C15.1, C16.1, C29.1, R11.2, R12.2, R19.2, R20.2; no longer C17.1, C23.1, C24.1, C5.1, C7.1, C8.1, R10.2, R14.2, R15.2, R16.2
- net VCC_LINUX: now also R24.2; no longer R9.2
- net VCC_LINUX_1V8: now also C23.1, C24.2; no longer C28.1, C30.2
- net VCC_LINUX_3V3: now also C20.1, C21.2, C22.1, C30.1, L1.2; no longer C25.1, C26.2, C27.1, C4.1, L2.2
Other:
- moved on the sheet: C10, C11, C12, C14, C15, C16, C17, C18, C19, C30, C8, C9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

Commit message: Controller module, candidate for fab
Also added all the gerbers to the gitignore
Parts:
- added JP4, JP5: (no value), pinhead:PINHD-1X2
Connections:
- net GND: now also JP4.1, JP4.2, JP5.1, JP5.2
Other:
- moved on the sheet: JP3, SW1
