File: hardware/radio_module/rev_a/radio_module.sch (EAGLE design)
At the start: 119 parts, among them J1 MODULE_GENERIC, J2 TC2030-JLINK-NL, J4 NANO_SIM, J5 TC2030-JLINK-L, P1 MOLEX_73251-135X, P2 MOLEX_73251-135X, Q1 MOSFET-NCHANNELXFDN-3, Q2 MOSFET-NCHANNELXFDN-3, Q3 MOSFET-NCHANNELXFDN-3, Q4 MOSFET-NCHANNELXFDN-3, Q5 SI223DDS, Q6 SI223DDS, Q7 SI223DDS, U1 NUCLEUM, U10 TXB0106, U11 SAM4LC8BA, U12 UBLOX_SARA_G350, U2 TLV62130, U4 LTC2941, U5 LTC2941, U6 IM880_MODULE, U7 PCA9544AQFN-N20, U8 TLV62130, U9 LTC2941, X2 16 MHz

Commit message: added tps for internal i2c bus
Parts:
- added TP13, TP4, TP5: TPB1,27, testpad:TPB1,27
Connections:
- net N$9: now also TP13.TP
- net SCL_INTERNAL: now also TP5.TP
- net SDA_INTERNAL: now also TP4.TP
Other:
- note added: "Rsense = 0.05V/Imax = 0.05V/118mA"
- note added: "Rsense = 0.05V/Imax = 0.05V/15mA"
- note removed: "Rsense = 0.05V/Imax = 0.05V/118ma"
- note removed: "Rsense = 0.05V/Imax = 0.05V/15ma"
Changed lines of the file:
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@@
 <part name="GND29" library="umich" deviceset="GND" device=""/>
 <part name="GND30" library="umich" deviceset="GND" device=""/>
+<part name="TP4" library="testpad" deviceset="TP" device="B1,27"/>
+<part name="TP5" library="testpad" deviceset="TP" device="B1,27"/>
+<part name="TP13" library="testpad" deviceset="TP" device="B1,27"/>
 </parts>
 <sheets>
@@
 </instance>
 <instance part="U$1" gate="G$1" x="238.76" y="177.8"/>
+<instance part="TP4" gate="G$1" x="88.9" y="63.5" smashed="yes" rot="R90">
+<attribute name="TP_SIGNAL_NAME" x="90.17" y="64.77" size="1.778" layer="97" rot="R90"/>
+</instance>
+<instance part="TP5" gate="G$1" x="88.9" y="60.96" smashed="yes" rot="R90">
+<attribute name="TP_SIGNAL_NAME" x="90.17" y="62.23" size="1.778" layer="97" rot="R90"/>
+</instance>
+<instance part="TP13" gate="G$1" x="88.9" y="58.42" smashed="yes" rot="R90">
+<attribute name="TP_SIGNAL_NAME" x="90.17" y="59.69" size="1.778" layer="97" rot="R90"/>
+</instance>
 </instances>
 <busses>
@@
 <pinref part="U7" gate="G$1" pin="SDA"/>
 <pinref part="R12" gate="G$1" pin="2"/>
-<wire x1="114.3" y1="63.5" x2="81.28" y2="63.5" width="0.1524" layer="91"/>
+<wire x1="114.3" y1="63.5" x2="91.44" y2="63.5" width="0.1524" layer="91"/>
+<wire x1="91.44" y1="63.5" x2="81.28" y2="63.5" width="0.1524" layer="91"/>
 <wire x1="81.28" y1="63.5" x2="66.04" y2="63.5" width="0.1524" layer="91"/>
 <wire x1="81.28" y1="66.04" x2="81.28" y2="63.5" width="0.1524" layer="91"/>
 <junction x="81.28" y="63.5"/>
+<pinref part="TP4" gate="G$1" pin="TP"/>
+<junction x="91.44" y="63.5"/>
 </segment>
 </net>
@@
 <pinref part="U7" gate="G$1" pin="SCL"/>
 <pinref part="R13" gate="G$1" pin="2"/>
-<wire x1="116.84" y1="60.96" x2="78.74" y2="60.96" width="0.1524" layer="91"/>
+<wire x1="116.84" y1="60.96" x2="91.44" y2="60.96" width="0.1524" layer="91"/>
+<wire x1="91.44" y1="60.96" x2="78.74" y2="60.96" width="0.1524" layer="91"/>
 <wire x1="78.74" y1="60.96" x2="66.04" y2="60.96" width="0.1524" layer="91"/>
 <wire x1="78.74" y1="66.04" x2="78.74" y2="60.96" width="0.1524" layer="91"/>
 <junction x="78.74" y="60.96"/>
+<pinref part="TP5" gate="G$1" pin="TP"/>
+<junction x="91.44" y="60.96"/>
 </segment>
 </net>
@@
 <pinref part="U7" gate="G$1" pin="!INT"/>
 <pinref part="R14" gate="G$1" pin="2"/>
-<wire x1="104.14" y1="58.42" x2="73.66" y2="58.42" width="0.1524" layer="91"/>
+<wire x1="104.14" y1="58.42" x2="91.44" y2="58.42" width="0.1524" layer="91"/>
+<wire x1="91.44" y1="58.42" x2="73.66" y2="58.42" width="0.1524" layer="91"/>
 <wire x1="73.66" y1="58.42" x2="66.04" y2="58.42" width="0.1524" layer="91"/>
 <wire x1="73.66" y1="66.04" x2="73.66" y2="58.42" width="0.1524" layer="91"/>
 <junction x="73.66" y="58.42"/>
+<pinref part="TP13" gate="G$1" pin="TP"/>
+<junction x="91.44" y="58.42"/>
 </segment>
 </net>
@@
 <text x="116.84" y="124.46" size="2.54" layer="97">Energy gauge for IM880</text>
 <text x="114.3" y="71.12" size="2.54" layer="97">Energy gauge for GSM module</text>
-<text x="187.96" y="180.34" size="2.54" layer="97">Rsense = 0.05V/Imax = 0.05V/15ma</text>
-<text x="190.5" y="127" size="2.54" layer="97">Rsense = 0.05V/Imax = 0.05V/118ma</text>
+<text x="187.96" y="180.34" size="2.54" layer="97">Rsense = 0.05V/Imax = 0.05V/15mA</text>
+<text x="190.5" y="127" size="2.54" layer="97">Rsense = 0.05V/Imax = 0.05V/118mA</text>
 <text x="190.5" y="73.66" size="2.54" layer="97">Rsense = 0.05V/Imax = 0.05V/3A</text>
 </plain>
