File: modules/audio_spectrum/rev_a/audio_spectrum.brd (EAGLE design)
At the start: 68.1 x 66 mm, 73 parts, among them J1 MODULE_GENERIC, J2 AUDIO-JACK-VERTICAL, J7 TC2030-JLINK-L, P1 4k-200k, P2 4k-200k, Q1 NX3008PBK, Q2 NX3008PBK, U1 SAM4LC8AA, U2 MSGEQ7, U3 MSGEQ7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

Commit message: some final changes and packing up for assembly
Parts:
- removed LED5: LED0603, leds:LED-0603
- added LED2: LED0603, leds:LED-0603
- moved LED3 10.2 mm to (38.1, 5.08)
- renumbered LED7 to LED4, U$1 to U8
Connections:
- net 3V3: now also LED2.A; no longer LED5.A
- net N$23: now also LED2.C; no longer LED3.C
- net N$33: now also LED3.C; no longer LED5.C
Changed lines of the file:
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@@
 <setting verticaltext="up"/>
 </settings>
-<grid distance="0.01" unitdist="inch" unit="inch" style="lines" multiple="1" display="yes" altdistance="0.01" altunitdist="inch" altunit="inch"/>
+<grid distance="0.1" unitdist="inch" unit="inch" style="lines" multiple="1" display="yes" altdistance="0.01" altunitdist="inch" altunit="inch"/>
 <layers>
 <layer number="1" name="Top" color="4" fill="1" visible="yes" active="yes"/>
@@
 <attribute name="NAME" x="30.48" y="57.404" size="0.889" layer="25" font="vector" ratio="12" align="bottom-center"/>
 </element>
-<element name="U$1" library="chips" package="MP23AB02B" value="MP23AB02B" x="28.194" y="8.89" smashed="yes" rot="MR0">
+<element name="U8" library="chips" package="MP23AB02B" value="MP23AB02B" x="28.194" y="8.89" smashed="yes" rot="MR0">
 <attribute name="DIGIKEY" value="497-14947-1-ND" x="28.194" y="8.89" size="1.778" layer="28" font="vector" ratio="12" rot="MR0" display="off"/>
 </element>
@@
 <attribute name="VALUE" x="46.5455" y="5.08" size="1.016" layer="27" font="vector" ratio="12" rot="R90" align="top-center"/>
 </element>
-<element name="LED3" library="leds" package="LED-0603" value="LED0603" x="48.26" y="5.08" smashed="yes">
+<element name="LED2" library="leds" package="LED-0603" value="LED0603" x="48.26" y="5.08" smashed="yes">
 <attribute name="NAME" x="48.9585" y="6.096" size="1.016" layer="25" font="vector" ratio="12" rot="R270" align="bottom-center"/>
 <attribute name="VALUE" x="49.0855" y="5.08" size="1.016" layer="27" font="vector" ratio="12" rot="R90" align="top-center"/>
 </element>
-<element name="LED5" library="leds" package="LED-0603" value="LED0603" x="38.1" y="5.08" smashed="yes">
+<element name="LED3" library="leds" package="LED-0603" value="LED0603" x="38.1" y="5.08" smashed="yes">
 <attribute name="NAME" x="37.4015" y="6.096" size="1.016" layer="25" font="vector" ratio="12" rot="R90" align="bottom-center"/>
 <attribute name="VALUE" x="38.9255" y="5.08" size="1.016" layer="27" font="vector" ratio="12" rot="R90" align="top-center"/>
 </element>
-<element name="LED7" library="leds" package="LED-0603" value="LED0603" x="40.64" y="5.08" smashed="yes">
+<element name="LED4" library="leds" package="LED-0603" value="LED0603" x="40.64" y="5.08" smashed="yes">
 <attribute name="NAME" x="42.4815" y="6.096" size="1.016" layer="25" font="vector" ratio="12" rot="R90" align="bottom-center"/>
 <attribute name="VALUE" x="41.4655" y="5.08" size="1.016" layer="27" font="vector" ratio="12" rot="R90" align="top-center"/>
@@
 <contactref element="R13" pad="2"/>
 <contactref element="C22" pad="1"/>
-<contactref element="U$1" pad="3"/>
+<contactref element="U8" pad="3"/>
 <contactref element="C23" pad="1"/>
 <contactref element="C9" pad="1"/>
@@
 <wire x1="60.127940625" y1="24.634" x2="60.127940625" y2="32.949940625" width="0.508" layer="16"/>
 <wire x1="60.127940625" y1="32.949940625" x2="59.944" y2="33.274" width="0.508" layer="16"/>
+<contactref element="LED2" pad="A"/>
 <contactref element="LED3" pad="A"/>
-<contactref element="LED5" pad="A"/>
-<contactref element="LED7" pad="A"/>
+<contactref element="LED4" pad="A"/>
 <contactref element="LED1" pad="A"/>
 <wire x1="48.26" y1="4.33" x2="45.72" y2="4.33" width="0.508" layer="1"/>
@@
 <contactref element="U5" pad="5"/>
 <contactref element="R10" pad="1"/>
-<contactref element="U$1" pad="2"/>
+<contactref element="U8" pad="2"/>
 <contactref element="C9" pad="2"/>
 <contactref element="C23" pad="2"/>
@@
 <signal name="N$18">
 <contactref element="C25" pad="2"/>
-<contactref element="U$1" pad="1"/>
+<contactref element="U8" pad="1"/>
 <wire x1="28.804" y1="9.815" x2="28.702" y2="9.815" width="0.254" layer="16"/>
 <wire x1="28.702" y1="9.815" x2="28.702" y2="10.414" width="0.254" layer="16"/>
@@
 <signal name="N$25">
 <contactref element="R4" pad="2"/>
-<contactref element="LED7" pad="C"/>
+<contactref element="LED4" pad="C"/>
 <wire x1="40.64" y1="5.83" x2="40.64" y2="7.224" width="0.254" layer="1"/>
 </signal>
@@
 </signal>
 <signal name="N$23">
-<contactref element="LED3" pad="C"/>
+<contactref element="LED2" pad="C"/>
 <contactref element="R2" pad="2"/>
 <wire x1="48.26" y1="5.83" x2="48.26" y2="7.224" width="0.254" layer="1"/>
 </signal>
 <signal name="N$33">
-<contactref element="LED5" pad="C"/>
+<contactref element="LED3" pad="C"/>
 <contactref element="R3" pad="2"/>
 <wire x1="38.1" y1="5.83" x2="38.1" y2="7.224" width="0.254" layer="1"/>
