File: modules/ambient/ambient.sch (KiCad schematic (older format))
At the start: 27 parts, among them P1 CONN_01X03, P2 CONN_01X06, U1 SIGNPOST_MODULE_GENERIC, U2 TPS62086, U3 JLINK-TC, U4 SAM4LC8A, Y1 FH1600015

Commit message: fixes go ambient
Parts:
- removed U1: SIGNPOST_MODULE_GENERIC, signpost:MODULE_GENERIC, symbol SIGNPOST_MODULE_GENERIC
- removed U3: JLINK-TC, lab11-connectors:TC2030-IDC, symbol JLINK-TC
- added P3: SIGNPOST_MODULE_GENERIC, lab11-connectors:SIGNPOST_MODULE_GENERIC, symbol SIGNPOST_MODULE_GENERIC
- added P4: JLINK-TC, lab11-connectors:TC2030-IDC, symbol JLINK-TC
- added R5, R6: GENERIC_R_0402, Resistors_SMD:R_0402, symbol GENERIC_R_0402
- L2: footprint Capacitors_SMD:C_0402 -> Capacitors_SMD:C_0603_HandSoldering
Connections:
- net labels added: USART_RX, USART_TX
- net labels removed: CONN_5, CONN_6
- wire segments 117 -> 121
Changed lines of the file:
@@
 $EndComp
 $Comp
-L GND #PWR15
+L GND #PWR01
 U 1 1 57EB1828
 P 6750 4200
-F 0 "#PWR15" H 6750 3950 50  0001 C CNN
+F 0 "#PWR01" H 6750 3950 50  0001 C CNN
 F 1 "GND" H 6750 4050 50  0000 C CNN
 F 2 "" H 6750 4200 50  0000 C CNN
@@
 F 0 "L2" V 5800 2700 50  0000 C CNN
 F 1 "1.5k Ohm" V 5950 2700 50  0000 C CNN
-F 2 "Capacitors_SMD:C_0402" V 5850 2700 50  0001 C CNN
+F 2 "Capacitors_SMD:C_0603_HandSoldering" V 5850 2700 50  0001 C CNN
 F 3 "" H 5850 2700 50  0000 C CNN
 F 4 "Digikey" V 5850 2700 60  0001 C CNN "Vendor 1"
@@
 $EndComp
 $Comp
-L +3.3V #PWR11
+L +3.3V #PWR02
 U 1 1 57EB32E1
 P 4850 2350
-F 0 "#PWR11" H 4850 2200 50  0001 C CNN
+F 0 "#PWR02" H 4850 2200 50  0001 C CNN
 F 1 "+3.3V" H 4850 2490 50  0000 C CNN
 F 2 "" H 4850 2350 50  0000 C CNN
@@
 $EndComp
 $Comp
-L GND #PWR12
+L GND #PWR03
 U 1 1 57EB425D
 P 5150 3500
-F 0 "#PWR12" H 5150 3250 50  0001 C CNN
+F 0 "#PWR03" H 5150 3250 50  0001 C CNN
 F 1 "GND" H 5150 3350 50  0000 C CNN
 F 2 "" H 5150 3500 50  0000 C CNN
@@
 xout
 $Comp
-L GND #PWR14
+L GND #PWR04
 U 1 1 57EC5AE9
 P 5700 1200
-F 0 "#PWR14" H 5700 950 50  0001 C CNN
+F 0 "#PWR04" H 5700 950 50  0001 C CNN
 F 1 "GND" H 5700 1050 50  0000 C CNN
 F 2 "" H 5700 1200 50  0000 C CNN
@@
 $EndComp
 $Comp
-L +3.3V #PWR16
+L +3.3V #PWR05
 U 1 1 57EC704B
 P 9400 2100
-F 0 "#PWR16" H 9400 1950 50  0001 C CNN
+F 0 "#PWR05" H 9400 1950 50  0001 C CNN
 F 1 "+3.3V" H 9400 2240 50  0000 C CNN
 F 2 "" H 9400 2100 50  0000 C CNN
@@
 $EndComp
 $Comp
-L SIGNPOST_MODULE_GENERIC U1
-U 1 1 57EC99DE
-P 900 6850
-F 0 "U1" H 750 7800 60  0000 C CNN
-F 1 "SIGNPOST_MODULE_GENERIC" V 550 6950 60  0000 C CNN
-F 2 "signpost:MODULE_GENERIC" H 950 8300 60  0001 C CNN
-F 3 "" H 1400 8100 60  0001 C CNN
-F 4 "Digikey" H 900 8200 60  0001 C CNN "Vendor 1"
-F 5 "S9170-ND" H 900 8100 60  0001 C CNN "Vendor 1 Part Number"
-	1    900  6850
-	1    0    0    -1
-$EndComp
-$Comp
-L +5V #PWR4
+L +5V #PWR06
 U 1 1 57EC9DAF
 P 1450 5900
-F 0 "#PWR4" H 1450 5750 50  0001 C CNN
+F 0 "#PWR06" H 1450 5750 50  0001 C CNN
 F 1 "+5V" H 1450 6040 50  0000 C CNN
 F 2 "" H 1450 5900 50  0000 C CNN
@@
 $EndComp
 $Comp
-L +3.3V #PWR5
+L +3.3V #PWR07
 U 1 1 57EC9DF7
 P 1800 5900
-F 0 "#PWR5" H 1800 5750 50  0001 C CNN
+F 0 "#PWR07" H 1800 5750 50  0001 C CNN
 F 1 "+3.3V" H 1800 6040 50  0000 C CNN
 F 2 "" H 1800 5900 50  0000 C CNN
@@
 $EndComp
 $Comp
-L GND #PWR7
+L GND #PWR08
 U 1 1 57EDACD2
 P 3400 4700
-F 0 "#PWR7" H 3400 4450 50  0001 C CNN
+F 0 "#PWR08" H 3400 4450 50  0001 C CNN
 F 1 "GND" H 3400 4550 50  0000 C CNN
 F 2 "" H 3400 4700 50  0000 C CNN
@@
 $EndComp
 $Comp
-L +5V #PWR1
+L +5V #PWR09
 U 1 1 57EDAFE4
 P 1150 4250
-F 0 "#PWR1" H 1150 4100 50  0001 C CNN
+F 0 "#PWR09" H 1150 4100 50  0001 C CNN
 F 1 "+5V" H 1150 4390 50  0000 C CNN
 F 2 "" H 1150 4250 50  0000 C CNN
@@
 $EndComp
 $Comp
-L GND #PWR2
+L GND #PWR010
 U 1 1 57EDB3A5
 P 1150 4750
-F 0 "#PWR2" H 1150 4500 50  0001 C CNN
+F 0 "#PWR010" H 1150 4500 50  0001 C CNN
 F 1 "GND" H 1150 4600 50  0000 C CNN
 F 2 "" H 1150 4750 50  0000 C CNN
@@
 $EndComp
 $Comp
-L +3.3V #PWR6
+L +3.3V #PWR011
 U 1 1 57EDC070
 P 3400 4350
-F 0 "#PWR6" H 3400 4200 50  0001 C CNN
+F 0 "#PWR011" H 3400 4200 50  0001 C CNN
 F 1 "+3.3V" H 3400 4490 50  0000 C CNN
 F 2 "" H 3400 4350 50  0000 C CNN
@@
 SAM4L_SWDIO
 $Comp
-L JLINK-TC U3
-U 1 1 57EE5AAF
-P 4900 5350
-F 0 "U3" H 4650 5550 60  0000 C CNN
-F 1 "JLINK-TC" H 4900 5150 60  0000 C CNN
-F 2 "lab11-connectors:TC2030-IDC" H 4850 5750 60  0001 C CNN
-F 3 "" H 5600 5600 60  0001 C CNN
-	1    4900 5350
-	1    0    0    -1
-$EndComp
-$Comp
-L +3.3V #PWR10
+L +3.3V #PWR012
 U 1 1 57EE5DA7
 P 4300 5250
-F 0 "#PWR10" H 4300 5100 50  0001 C CNN
+F 0 "#PWR012" H 4300 5100 50  0001 C CNN
 F 1 "+3.3V" H 4300 5390 50  0000 C CNN
 F 2 "" H 4300 5250 50  0000 C CNN
@@
 SAM4L_RESET
 $Comp
-L GND #PWR8
+L GND #PWR013
 U 1 1 57EE64A6
 P 3650 5350
-F 0 "#PWR8" H 3650 5100 50  0001 C CNN
+F 0 "#PWR013" H 3650 5100 50  0001 C CNN
 F 1 "GND" H 3650 5200 50  0000 C CNN
 F 2 "" H 3650 5350 50  0000 C CNN
@@
 SDA
 $Comp
-L GND #PWR9
+L GND #PWR014
 U 1 1 57F553C5
 P 3700 3500
-F 0 "#PWR9" H 3700 3250 50  0001 C CNN
+F 0 "#PWR014" H 3700 3250 50  0001 C CNN
 F 1 "GND" H 3700 3350 50  0000 C CNN
 F 2 "" H 3700 3500 50  0000 C CNN
@@
 Text Label 8200 3750 0    60   ~ 0
 LPS_INT1
-Text Label 8200 3650 0    60   ~ 0
-CONN_5
 Wire Wire Line
 	8050 4050 8550 4050
@@
 	8050 3750 8550 3750
 Wire Wire Line
-	8050 3650 8550 3650
-Text Label 8200 3550 0    60   ~ 0
-CONN_6
-Wire Wire Line
-	8050 3550 8550 3550
+	8050 3550 8650 3550
 Text Label 9550 3350 0    60   ~ 0
 TSL_INT
@@
 LPS_INT1
 Text Label 9550 3050 0    60   ~ 0
-CONN_5
+USART_TX
 Text Label 9550 2950 0    60   ~ 0
-CONN_6
+USART_RX
 Wire Wire Line
 	9450 3450 9900 3450
@@
 	9450 2950 9900 2950
 $Comp
-L GND #PWR3
+L GND #PWR015
 U 1 1 57F54934
 P 1400 7600
-F 0 "#PWR3" H 1400 7350 50  0001 C CNN
+F 0 "#PWR015" H 1400 7350 50  0001 C CNN
 F 1 "GND" H 1400 7450 50  0000 C CNN
 F 2 "" H 1400 7600 50  0000 C CNN
@@
 	4850 6850 4950 6850
 $Comp
-L +3.3V #PWR13
+L +3.3V #PWR016
 U 1 1 57F5E465
 P 5350 6100
-F 0 "#PWR13" H 5350 5950 50  0001 C CNN
+F 0 "#PWR016" H 5350 5950 50  0001 C CNN
 F 1 "+3.3V" H 5350 6240 50  0000 C CNN
 F 2 "" H 5350 6100 50  0000 C CNN
@@
 Wire Wire Line
 	8050 2850 8500 2850
+$Comp
+L GENERIC_R_0402 R5
+U 1 1 57F5A076
+P 7000 5850
+F 0 "R5" H 7000 5925 50  0000 C CNN
+F 1 "GENERIC_R_0402" H 7025 6550 50  0001 C CNN
+F 2 "Resistors_SMD:R_0402" H 7000 6400 50  0001 C CNN
+F 3 "" H 7100 6475 50  0001 C CNN
+F 4 "0" H 7000 5775 60  0000 C CNN "Resistance"
+F 5 "Digikey" H 7000 6300 60  0001 C CNN "Vendor 1"
+F 6 "Placeholder" H 7000 6200 60  0001 C CNN "Vendor 1 Part Number"
+	1    7000 5850
+	1    0    0    -1
+$EndComp
+$Comp
+L GENERIC_R_0402 R6
+U 1 1 57F5A392
+P 8250 5850
+F 0 "R6" H 8250 5925 50  0000 C CNN
+F 1 "GENERIC_R_0402" H 8275 6550 50  0001 C CNN
+F 2 "Resistors_SMD:R_0402" H 8250 6400 50  0001 C CNN
+F 3 "" H 8350 6475 50  0001 C CNN
+F 4 "0" H 8250 5775 60  0000 C CNN "Resistance"
+F 5 "Digikey" H 8250 6300 60  0001 C CNN "Vendor 1"
+F 6 "Placeholder" H 8250 6200 60  0001 C CNN "Vendor 1 Part Number"
+	1    8250 5850
+	1    0    0    -1
+$EndComp
+$Comp
+L +3.3V #PWR017
+U 1 1 57F5A5C2
+P 6800 5750
+F 0 "#PWR017" H 6800 5600 50  0001 C CNN
+F 1 "+3.3V" H 6800 5890 50  0000 C CNN
+F 2 "" H 6800 5750 50  0000 C CNN
+F 3 "" H 6800 5750 50  0000 C CNN
+	1    6800 5750
+	1    0    0    -1
+$EndComp
+$Comp
+L +3.3V #PWR018
+U 1 1 57F5A866
+P 8050 5750
+F 0 "#PWR018" H 8050 5600 50  0001 C CNN
+F 1 "+3.3V" H 8050 5890 50  0000 C CNN
+F 2 "" H 8050 5750 50  0000 C CNN
+F 3 "" H 8050 5750 50  0000 C CNN
+	1    8050 5750
+	1    0    0    -1
+$EndComp
+Text GLabel 7250 5850 2    60   Input ~ 0
+SCL
+Text GLabel 8500 5850 2    60   Input ~ 0
+SDA
+Wire Wire Line
+	8500 5850 8450 5850
+Wire Wire Line
+	8050 5750 8050 5850
+Wire Wire Line
+	7250 5850 7200 5850
+Wire Wire Line
+	6800 5850 6800 5750
+Wire Wire Line
+	8050 3450 8650 3450
+Text Label 8200 3450 0    60   ~ 0
+USART_RX
+Text Label 8200 3550 0    60   ~ 0
+USART_TX
+$Comp
+L SIGNPOST_MODULE_GENERIC P3
+U 1 1 57F5F6F0
+P 900 6850
+F 0 "P3" H 750 7800 60  0000 C CNN
+F 1 "SIGNPOST_MODULE_GENERIC" V 550 6950 60  0000 C CNN
+F 2 "lab11-connectors:SIGNPOST_MODULE_GENERIC" H 950 8300 60  0001 C CNN
+F 3 "" H 1400 8100 60  0001 C CNN
+F 4 "Digikey" H 900 8200 60  0001 C CNN "Vendor 1"
+F 5 "S9170-ND" H 900 8100 60  0001 C CNN "Vendor 1 Part Number"
+	1    900  6850
+	1    0    0    -1
+$EndComp
+$Comp
+L JLINK-TC P4
+U 1 1 57F61DBD
+P 4900 5350
+F 0 "P4" H 4650 5550 60  0000 C CNN
+F 1 "JLINK-TC" H 4900 5150 60  0000 C CNN
+F 2 "lab11-connectors:TC2030-IDC" H 4850 5750 60  0001 C CNN
+F 3 "" H 5600 5600 60  0001 C CNN
+	1    4900 5350
+	1    0    0    -1
+$EndComp
 $EndSCHEMATC

Commit message: added holes back in
Parts:
- added H1, H2, H3, H4: SIGNPOST_HOLE, lab11-connectors:SIGNPOST_HOLE, symbol SIGNPOST_HOLE
Changed lines of the file:
@@
+	1    0    0    -1
+$EndComp
+$Comp
+L SIGNPOST_HOLE H1
+U 1 1 57F5C6B7
+P 8500 950
+F 0 "H1" H 8500 950 60  0001 C CNN
+F 1 "SIGNPOST_HOLE" H 8400 1250 60  0001 C CNN
+F 2 "lab11-connectors:SIGNPOST_HOLE" H 8400 850 60  0001 C CNN
+F 3 "" H 8500 950 60  0001 C CNN
+	1    8500 950
+	1    0    0    -1
+$EndComp
+$Comp
+L SIGNPOST_HOLE H2
+U 1 1 57F5C71D
+P 8700 950
+F 0 "H2" H 8700 950 60  0001 C CNN
+F 1 "SIGNPOST_HOLE" H 8600 1250 60  0001 C CNN
+F 2 "lab11-connectors:SIGNPOST_HOLE" H 8600 850 60  0001 C CNN
+F 3 "" H 8700 950 60  0001 C CNN
+	1    8700 950
+	1    0    0    -1
+$EndComp
+$Comp
+L SIGNPOST_HOLE H3
+U 1 1 57F5C783
+P 8950 950
+F 0 "H3" H 8950 950 60  0001 C CNN
+F 1 "SIGNPOST_HOLE" H 8850 1250 60  0001 C CNN
+F 2 "lab11-connectors:SIGNPOST_HOLE" H 8850 850 60  0001 C CNN
+F 3 "" H 8950 950 60  0001 C CNN
+	1    8950 950
+	1    0    0    -1
+$EndComp
+$Comp
+L SIGNPOST_HOLE H4
+U 1 1 57F5C7E9
+P 9250 1000
+F 0 "H4" H 9250 1000 60  0001 C CNN
+F 1 "SIGNPOST_HOLE" H 9150 1300 60  0001 C CNN
+F 2 "lab11-connectors:SIGNPOST_HOLE" H 9150 900 60  0001 C CNN
+F 3 "" H 9250 1000 60  0001 C CNN
+	1    9250 1000
 	1    0    0    -1
 $EndComp
