File: modules/microwave_radar/hardware/rev_a/microwave.sch (EAGLE design)
At the start: 55 parts, among them J1 MODULE_GENERIC, J2 TC2030-JLINK-L, U1 SAM4LC8AA, U2 TLV62130, U3 MSGEQ7, U4 HB100, U5 OP284E_SEPARATE

Commit message: Fabrication files
Parts:
- removed R18: 1k, passives:RESISTOR0402_RES
- added R17: 750k, passives:RESISTOR0402_RES
- R1: value 8.2k -> 1k; DIGIKEY 311-8.20KLRCT-ND -> 1276-3430-1-ND
- R11: DIGIKEY P100KJCT-ND -> 1276-3432-1-ND
- R12: value 200k -> 100k; device passives:RESISTOR0603_RES -> passives:RESISTOR0402_RES; DIGIKEY RHM200KCFCT-ND -> 1276-3432-1-ND
- R13: value 240k -> 100k; DIGIKEY P240KLCT-ND -> P100KJCT-ND
- R14: value 330k -> 200k; device passives:RESISTOR0402_RES -> passives:RESISTOR0603_RES; DIGIKEY 1276-4244-1-ND -> RHM200KCFCT-ND
- R15: value 750k -> 240k; DIGIKEY P750KLCT-ND -> P240KLCT-ND
- R16: value 1k -> 330k; DIGIKEY 1276-3430-1-ND -> 1276-4244-1-ND
- R2: value 10k -> 1k; DIGIKEY 1276-3431-1-ND -> 1276-3430-1-ND
- R3: value 10k -> 8.2k; DIGIKEY 1276-3431-1-ND -> 311-8.20KLRCT-ND
- R4: value 12k -> 10k; DIGIKEY 1276-4122-1-ND -> 1276-3431-1-ND
- R5: value 100k -> 10k; DIGIKEY 1276-3432-1-ND -> 1276-3431-1-ND
- R6: value 100k -> 12k; DIGIKEY 1276-3432-1-ND -> 1276-4122-1-ND
Connections:
- net +3V3: now also R1.1, R10.2, R13.2, R14.1, R17.2, R2.1, R7.2; no longer R11.2, R12.1, R15.2, R16.1, R18.1, R3.2, R6.2
- net AMP_OUT: now also R12.1; no longer R10.1
- net CONTROLLER_SWDCLK: now also R8.1; no longer R6.1
- net CONTROLLER_SWDIO: now also R7.1; no longer R5.1
- net GND: now also R15.1, R6.1, R9.1; no longer R13.1, R4.1, R7.1
- net IF: now also R6.2; no longer R4.2
- net N$1: now also R10.1, R16.2, R9.2; no longer R14.2, R7.2, R8.1
- net N$12: now also R11.2, R4.1; no longer R2.1, R9.2
- net N$14: now also R5.1; no longer R3.1
- net N$15: now also R4.2; no longer R2.2
- net N$17: now also R11.1; no longer R9.1
- net N$18: now also R3.2; no longer R1.2
- net N$19: now also R12.2, R3.1; no longer R1.1, R10.2
- net N$2: now also R14.2; no longer R12.2
- net N$23: now also R13.1; no longer R11.1
- net N$24: now also R15.2, R17.1; no longer R13.2, R15.1
- net N$34: now also R2.2; no longer R18.2
- net N$4: now also R1.2; no longer R16.2
- net N$9: now also R16.1; no longer R14.1
Other:
- moved on the sheet: R10, R13, R15, R4, R5, R9
