File: modules/audio_spectrum/rev_b/audio_spectrum.brd (EAGLE design)
At the start: 68.1 x 66 mm, 92 parts, among them J1 MODULE_GENERIC, J2 AUDIO-JACK-VERTICAL, J7 TC2030-JLINK-L, P1 4k-200k, P2 4k-200k, Q1 NX3008PBK, Q2 NX3008PBK, U1 SAM4LC8AA, U2 MSGEQ7, U3 MSGEQ7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

Commit message: added gnd testpoint
Parts:
- added TP11: TEST_POINT_0.040IN, headers:TESTPOINT_0.040IN
- moved TP12 4.07 mm to (47.8, 64.5)
- moved TP13 3.05 mm to (47.8, 61.7)
- renumbered X2 to X1
Connections:
- net GND: now also TP11.TESTPOINT
Routing:
- net SCL: track 57.4 -> 53.4 mm
- net 5V: track 18.8 -> 17.7 mm
Other:
- board text added: "GND"
Changed lines of the file:
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@@
 <text x="61.214" y="47.752" size="0.889" layer="21" font="vector" ratio="12">Reset
 Button</text>
-<text x="46.736" y="62.23" size="0.889" layer="21" font="vector" ratio="12">SDA</text>
-<text x="50.8" y="62.23" size="0.889" layer="21" font="vector" ratio="12">SCL</text>
+<text x="46.482" y="66.04" size="0.889" layer="21" font="vector" ratio="12">SDA</text>
+<text x="49.53" y="61.214" size="0.889" layer="21" font="vector" ratio="12">SCL</text>
 <text x="20.828" y="66.294" size="0.889" layer="21" font="vector" ratio="12">PPS</text>
 <text x="24.13" y="66.294" size="0.889" layer="21" font="vector" ratio="12">OUT/RX</text>
@@
 <wire x1="42.164" y1="33.274" x2="42.164" y2="35.306" width="0.254" layer="21"/>
 <wire x1="42.164" y1="35.306" x2="40.386" y2="35.306" width="0.254" layer="21"/>
+<text x="50.546" y="66.04" size="0.889" layer="21" font="vector" ratio="12">GND</text>
 </plain>
 <attributes>
@@
 <element name="C1" library="passives" package="0603_CAP" value="8pF" x="50.8" y="33.528" smashed="yes" rot="R90">
 <attribute name="DIGIKEY" value="490-8230-1-ND" x="27.94" y="13.208" size="1.778" layer="27" font="vector" ratio="12" rot="R90" display="off"/>
-<attribute name="NAME" x="52.324" y="33.528" size="0.889" layer="25" font="vector" ratio="12" rot="R90" align="bottom-center"/>
+<attribute name="NAME" x="51.054" y="35.56" size="0.889" layer="25" font="vector" ratio="12" rot="R180" align="bottom-center"/>
 </element>
 <element name="C2" library="passives" package="0603_CAP" value="8pF" x="45.72" y="32.004" smashed="yes" rot="R90">
@@
 <attribute name="NAME" x="45.72" y="34.036" size="0.889" layer="25" font="vector" ratio="12" rot="R180" align="bottom-center"/>
 </element>
-<element name="X2" library="crystals" package="FHXXX" value="16MHz" x="48.26" y="32.004" smashed="yes">
+<element name="X1" library="crystals" package="FHXXX" value="16MHz" x="48.26" y="32.004" smashed="yes">
 <attribute name="DIGIKEY" value="FH1600015CT-ND" x="17.78" y="34.544" size="1.778" layer="27" font="vector" ratio="12" display="off"/>
 <attribute name="NAME" x="47.498" y="33.504" size="0.889" layer="25" font="vector" ratio="12" align="bottom-center"/>
@@
 <attribute name="DIGIKEY" value="SW1020CT-ND" x="63.246" y="45.974" size="0.889" layer="27" font="vector" ratio="12" display="off"/>
 </element>
-<element name="TP12" library="headers" package="TESTPOINT_0.040IN" value="TEST_POINT_0.040IN" x="51.816" y="64.77" smashed="yes">
-<attribute name="DIGIKEY" value="5001K-ND" x="51.816" y="64.77" size="0.889" layer="27" font="vector" ratio="12" display="off"/>
-<attribute name="VALUE" x="51.816" y="62.23" size="1.016" layer="27" font="vector" ratio="12" align="bottom-center"/>
-</element>
-<element name="TP13" library="headers" package="TESTPOINT_0.040IN" value="TEST_POINT_0.040IN" x="47.752" y="64.77" smashed="yes">
-<attribute name="DIGIKEY" value="5001K-ND" x="47.752" y="64.77" size="0.889" layer="27" font="vector" ratio="12" display="off"/>
-<attribute name="VALUE" x="47.752" y="62.23" size="1.016" layer="27" font="vector" ratio="12" align="bottom-center"/>
+<element name="TP12" library="headers" package="TESTPOINT_0.040IN" value="TEST_POINT_0.040IN" x="47.752" y="64.516" smashed="yes">
+<attribute name="DIGIKEY" value="5001K-ND" x="47.752" y="64.516" size="0.889" layer="27" font="vector" ratio="12" display="off"/>
+<attribute name="VALUE" x="47.752" y="61.976" size="1.016" layer="27" font="vector" ratio="12" align="bottom-center"/>
+</element>
+<element name="TP13" library="headers" package="TESTPOINT_0.040IN" value="TEST_POINT_0.040IN" x="47.752" y="61.722" smashed="yes">
+<attribute name="DIGIKEY" value="5001K-ND" x="47.752" y="61.722" size="0.889" layer="27" font="vector" ratio="12" display="off"/>
+<attribute name="VALUE" x="47.752" y="59.182" size="1.016" layer="27" font="vector" ratio="12" align="bottom-center"/>
 </element>
 <element name="TP14" library="headers" package="TESTPOINT_0.040IN" value="TEST_POINT_0.040IN" x="25.654" y="61.976" smashed="yes">
@@
 <attribute name="DIGIKEY" value="5001K-ND" x="21.844" y="64.77" size="0.889" layer="27" font="vector" ratio="12" display="off"/>
 <attribute name="VALUE" x="21.844" y="62.23" size="1.016" layer="27" font="vector" ratio="12" align="bottom-center"/>
+</element>
+<element name="TP11" library="headers" package="TESTPOINT_0.040IN" value="TEST_POINT_0.040IN" x="51.816" y="64.516" smashed="yes">
+<attribute name="DIGIKEY" value="5001K-ND" x="51.816" y="64.516" size="0.889" layer="27" font="vector" ratio="12" display="off"/>
+<attribute name="VALUE" x="51.816" y="61.976" size="1.016" layer="27" font="vector" ratio="12" align="bottom-center"/>
 </element>
 </elements>
@@
 <contactref element="U1" pad="THERMAL"/>
 <contactref element="J7" pad="5"/>
-<contactref element="X2" pad="4"/>
-<contactref element="X2" pad="2"/>
+<contactref element="X1" pad="4"/>
+<contactref element="X1" pad="2"/>
 <contactref element="C1" pad="2"/>
 <contactref element="C2" pad="2"/>
@@
 <via x="39.624" y="31.496" extent="1-16" drill="0.3048"/>
 <via x="43.688" y="14.732" extent="1-16" drill="0.3048"/>
+<contactref element="TP11" pad="TESTPOINT"/>
 </signal>
 <signal name="CONTROLLER_SWDCLK">
@@
 </signal>
 <signal name="CONTROLLER_XIN">
-<contactref element="X2" pad="3"/>
+<contactref element="X1" pad="3"/>
 <contactref element="C1" pad="1"/>
 <contactref element="U1" pad="1"/>
@@
 </signal>
 <signal name="CONTROLLER_XOUT">
-<contactref element="X2" pad="1"/>
+<contactref element="X1" pad="1"/>
 <contactref element="C2" pad="1"/>
 <contactref element="U1" pad="2"/>
@@
 <wire x1="53.098" y1="55.786" x2="52.418" y2="55.786" width="0.254" layer="1"/>
 <wire x1="52.418" y1="55.786" x2="52.418" y2="55.106" width="0.254" layer="1"/>
-<wire x1="44.196" y1="62.23" x2="50.038" y2="62.23" width="0.508" layer="1"/>
-<wire x1="50.038" y1="62.23" x2="51.308" y2="60.96" width="0.508" layer="1"/>
-<wire x1="51.308" y1="60.96" x2="51.308" y2="59.182" width="0.508" layer="1"/>
-<wire x1="51.308" y1="59.182" x2="52.07" y2="58.42" width="0.508" layer="1"/>
-<wire x1="52.07" y1="58.42" x2="53.086" y2="58.42" width="0.508" layer="1"/>
-<wire x1="53.086" y1="58.42" x2="53.086" y2="58.278" width="0.508" layer="1"/>
+<wire x1="44.196" y1="62.23" x2="48.148" y2="58.278" width="0.508" layer="1"/>
+<wire x1="48.148" y1="58.278" x2="53.086" y2="58.278" width="0.508" layer="1"/>
 </signal>
 <signal name="3VSWOUT">
@@
 <wire x1="39.116" y1="62.484" x2="39.878" y2="63.246" width="0.254" layer="16"/>
 <wire x1="39.878" y1="63.246" x2="46.228" y2="63.246" width="0.254" layer="16"/>
-<wire x1="46.228" y1="63.246" x2="47.752" y2="64.77" width="0.254" layer="16"/>
+<wire x1="46.228" y1="63.246" x2="47.752" y2="61.722" width="0.254" layer="16"/>
 </signal>
 <signal name="SCL">
@@
 <wire x1="49.784" y1="51.562" x2="40.386" y2="60.96" width="0.254" layer="1"/>
 <contactref element="TP12" pad="TESTPOINT"/>
-<wire x1="51.816" y1="64.77" x2="50.292" y2="66.294" width="0.254" layer="16"/>
-<wire x1="50.292" y1="66.294" x2="40.64" y2="66.294" width="0.254" layer="16"/>
+<wire x1="47.752" y1="64.516" x2="45.974" y2="66.294" width="0.254" layer="16"/>
+<wire x1="45.974" y1="66.294" x2="40.64" y2="66.294" width="0.254" layer="16"/>
 <wire x1="40.64" y1="66.294" x2="39.116" y2="64.77" width="0.254" layer="16"/>
 </signal>
