File: hardware/power_supply_module/rev_b/power_supply_module.brd (EAGLE design)
At the start: 68.1 x 66 mm, 119 parts, among them J1 MODULE_POWER, U1 TLV62130, U10 LTC2941, U11 LTC2941, U12 LTC2941, U13 LTC2941, U14 LTC2941, U15 LTC2941, U2 TLV62130, U3 TLV62130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

Commit message: rev b to fab
Parts:
- C25: value 22 uH -> 22 uF
- moved U$1 1.27 mm to (11.7, 51.3)
Changed lines of the file:
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@@
 <hole x="13.081" y="3.81" drill="3.2639"/>
 <hole x="54.991" y="3.81" drill="3.2639"/>
-<text x="22.352" y="55.88" size="0.8128" layer="21" font="vector" ratio="12" align="top-left">Signpost
+<text x="24.384" y="55.88" size="0.8128" layer="21" font="vector" ratio="12" align="top-left">Signpost
 Power Module
 Neal Jackson
@@
 <text x="4.445" y="24.765" size="1.016" layer="25" font="vector" ratio="12" rot="R180" align="bottom-center">VBATT-</text>
 <text x="4.445" y="31.115" size="1.016" layer="25" font="vector" ratio="12" align="bottom-center">VBATT+</text>
-<text x="19.9136" y="53.6194" size="3.302" layer="21" font="vector" ratio="12" align="center">B</text>
-<wire x1="17.9578" y1="55.6768" x2="21.082" y2="55.6768" width="0.3048" layer="21"/>
-<wire x1="21.082" y1="55.6768" x2="21.082" y2="51.562" width="0.3048" layer="21"/>
-<wire x1="21.082" y1="51.562" x2="17.9578" y2="51.562" width="0.3048" layer="21"/>
-<wire x1="17.9578" y1="51.562" x2="17.9578" y2="55.6768" width="0.3048" layer="21"/>
+<text x="21.6916" y="53.6194" size="3.302" layer="21" font="vector" ratio="12" align="center">B</text>
+<wire x1="19.7358" y1="55.6768" x2="22.86" y2="55.6768" width="0.3048" layer="21"/>
+<wire x1="22.86" y1="55.6768" x2="22.86" y2="51.562" width="0.3048" layer="21"/>
+<wire x1="22.86" y1="51.562" x2="19.7358" y2="51.562" width="0.3048" layer="21"/>
+<wire x1="19.7358" y1="51.562" x2="19.7358" y2="55.6768" width="0.3048" layer="21"/>
 </plain>
 <attributes>
@@
 <attribute name="NAME" x="27.94" y="11.43" size="1.016" layer="25" font="vector" ratio="12" align="bottom-center"/>
 </element>
-<element name="C25" library="passives" package="0603_CAP" value="22 uH" x="29.21" y="4.445" smashed="yes" rot="R90">
+<element name="C25" library="passives" package="0603_CAP" value="22 uF" x="29.21" y="4.445" smashed="yes" rot="R90">
 <attribute name="NAME" x="30.099" y="4.699" size="1.016" layer="25" font="vector" ratio="12" rot="R270" align="bottom-center"/>
 </element>
@@
 <attribute name="VALUE" x="59.563" y="34.798" size="1.016" layer="27" font="vector" ratio="12" rot="R90" align="bottom-center"/>
 </element>
-<element name="U$1" library="logos" package="UCB_CAL_200MIL" value="" x="10.414" y="51.308"/>
+<element name="U$1" library="logos" package="UCB_CAL_200MIL" value="" x="11.684" y="51.308"/>
 </elements>
 <signals>

Commit message: Use 2kOhm resistors for gauges. Fixes #13
Parts:
- R10, R11, R12, R13, R14, R15, R16, R17, R18, R19, R20, R21, R22, R23, R24, R25, R26, R27, R28, R29, R30, R31, R32, R9: value 10 kΩ -> 2 kΩ
