File: modules/ambient/rev_b/ambient.sch (KiCad schematic (older format))
At the start: 40 parts, among them P1 CONN_01X03, P2 CONN_01X06, P3 SIGNPOST_MODULE_GENERIC, P4 JLINK-TC, P5 CONN_01X06, SW1 BSU-1000P, U2 TPS62086, U4 SAM4LC8A, Y1 FH1600015

Commit message: added pir sensor
Connections:
- net labels added: EKMB_INT
- wire segments 138 -> 141
Changed lines of the file:
@@
 F6 "LPS25HB_INT" I R 4050 2550 60
 F7 "LPS35_INT" I R 4050 2750 60
+F8 "EKMB_INT" I R 4050 2900 60
 $EndSheet
 $Comp
@@
 Text Label 4250 6700 0    60   ~ 0
 SAM4L_RESET
+Wire Wire Line
+	10100 5100 10650 5100
+Text Label 4150 2900 0    60   ~ 0
+EKMB_INT
+Wire Wire Line
+	4050 2900 4600 2900
+Text Label 10200 5100 0    60   ~ 0
+EKMB_INT
+Text Label 8200 2750 0    60   ~ 0
+EKMB_INT
+Wire Wire Line
+	8050 2750 8650 2750
 $EndSCHEMATC
