File: hardware/hail/rev_a/hail.brd (EAGLE design)
At the start: 20.3 x 36.6 mm, 75 parts, among them J1 MICRO_USB_B_HIROSE_ZX62R-B-5P, J2 TC2030-JLINK-NL_NOSILK, J3 TC2030-JLINK-NL_NOSILK, U1 FT231XQ, U2 FXOS8700CQ, U3 ISL29035, U4 MAX8887EZK33+T, U5 NRF51822QF, U6 SAM4LC8BA, U7 SI7021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

Commit message: Renamed to Hail. Added BOM
Routing:
- net PARTICLE_DAC: track 5.10 -> 5.99 mm
Other:
- board text added: "Hail"
- board text removed: "Blew"
