File: hardware/hail/rev_a/hail.sch (EAGLE design)
At the start: 72 parts, among them J1 MICRO_USB_B_HIROSE_ZX62R-B-5P, J2 TC2030-JLINK-NL_NOSILK, J3 TC2030-JLINK-NL_NOSILK, U1 FT231XQ, U2 FXOS8700CQ, U3 ISL29035, U4 MAX8887EZK33+T, U5 NRF51822QF, U6 SAM4LC8BA, U7 SI7021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

Commit message: Renamed to Hail. Added BOM
Parts:
- C1: DIGIKEY (none) -> 490-6212-1-ND
- C10, C11, C12, C13, C14, C15, C16, C17: DIGIKEY (none) -> 490-10777-1-ND
- C23, C24: DIGIKEY (none) -> 490-13252-1-ND
- C6: DIGIKEY (none) -> 490-1303-1-ND
- C7: DIGIKEY (none) -> 490-5419-1-ND
- C8: DIGIKEY (none) -> 490-7763-1-ND
- C9: DIGIKEY (none) -> 445-1264-1-ND
- L1: DIGIKEY (none) -> 490-6840-1-ND
- LED1: DIGIKEY (none) -> 160-1837-6-ND
- R1, R2, R3, R4, R5: DIGIKEY (none) -> 1276-3430-1-ND
- R6, R7, R8: DIGIKEY (none) -> 1276-3431-1-ND
