File: modules/rf_spectrum/rev_a/rf_spectrum.sch (EAGLE design)
At the start: 40 parts, among them J3 MODULE_GENERIC_DEBUGSMT, J4 TC2030-JLINK-L, U1 MWSUB3G, U2 SKY13317, U3 STM32L432KC, U4 TLV62130, X1 ABS05-32.768KHZ-9-T

Commit message: added part numbers
Parts:
- C1, C2: DIGIKEY 490-10777-1-ND -> 490-6243-1-ND; MF (none) -> Murata; MFN (none) -> GRM1555C1H4R3BA01D
- C10, C11: DIGIKEY 490-10777-1-ND -> 490-6328-1-ND; MF (none) -> Murata; MFN (none) -> GRM155R71C104KA88J
- C12: DIGIKEY 490-13252-1-ND -> 490-1320-1-ND; MF (none) -> Murata; MFN (none) -> GRM155R60J105KE19D
- C13: DIGIKEY 490-13252-1-ND -> 490-5915-1-ND; MF (none) -> Murata; MFN (none) -> GRM155R60J475ME47D
- C14: DIGIKEY (none) -> 490-6405-1-ND; MF (none) -> Murata; MFN (none) -> GRM188R60J106ME47J
- C15: DIGIKEY (none) -> 490-7611-1-ND; MF (none) -> Murata; MFN (none) -> GRM188R60J226MEA0D
- C3, C4, C5: DIGIKEY 490-10777-1-ND -> 490-6241-1-ND; MF (none) -> Murata; MFN (none) -> GRM1555C1H470FA01D
- C6: DIGIKEY 490-10777-1-ND -> 490-1293-1-ND; MF (none) -> Murata; MFN (none) -> GRM1555C1H221JA01D
- C7: DIGIKEY (none) -> 490-1503-1-ND; MF (none) -> Murata; MFN (none) -> GRM188R71H332KA01D
- C8: DIGIKEY 490-10777-1-ND -> 490-4516-1-ND; MF (none) -> Murata; MFN (none) -> GRM155R71H103KA88D
- C9: DIGIKEY (none) -> 490-1532-1-ND; MF (none) -> Murata; MFN (none) -> GRM188R71C104KA01D
- D1: DIGIKEY (none) -> 160-1446-1-ND; MF (none) -> Lite-ON; MFN (none) -> LTST-C191KGKT
- D2: DIGIKEY (none) -> 160-1447-1-ND; MF (none) -> Lite-On; MFN (none) -> LTST-C191KRKT
- J1, J2: DIGIKEY (none) -> WM8086-ND; MF (none) -> Molex; MFN (none) -> 0901200764
- R1: DIGIKEY (none) -> 311-0.0JRCT-ND; MF (none) -> Yageo; MFN (none) -> RC0402JR-070RL
- R2, R3: value 10k -> 1k; DIGIKEY (none) -> 311-1.0KJRCT-ND; MF (none) -> Yageo; MFN (none) -> RC0402JR-071KL
- R4: DIGIKEY (none) -> RHM10KCECT-ND; MF (none) -> Rohm; MFN (none) -> MCR01MRTJ103
- R5: DIGIKEY (none) -> 311-100KGRCT-ND; MF (none) -> Yageo; MFN (none) -> RC0603JR-07100KL
- R6: DIGIKEY (none) -> 311-100KLRCT-ND; MF (none) -> Yageo; MFN (none) -> RC0402FR-07100KL
- R7: DIGIKEY (none) -> 311-240KGRCT-ND; MF (none) -> Yageo; MFN (none) -> RC0603JR-07240KL
- R8: DIGIKEY (none) -> 311-750KGRCT-ND; MF (none) -> Yageo; MFN (none) -> 311-750KGRCT-ND
- U3: MF (none) -> STM
- X1: value ABS05-32.768KHZ-9-T -> ABS05-32.768KHZ-T; device crystals:ABS05-32.768KHZ-9-T -> crystals:ABS05-32.768KHZ-T
Connections:
- removed net N$13: D2.ANODE, R4.1
- new net R3: D2.ANODE, R3.1
- new net R4: R4.1
- net DBG_GPIO1: now also R2.2; no longer R3.2
- net DBG_GPIO2: now also R3.2; no longer R4.2
- net GND: no longer R2.1
- net N$11: now also R4.2; no longer R2.2
- net N$12: now also R2.1; no longer R3.1
Other:
- moved on the sheet: R2, R3, R4

Commit message: moved resistor
Parts:
- added R9: 750k, passives:RESISTOR0603_RES
- R7: value 240k -> 100k; device passives:RESISTOR0603_RES -> passives:RESISTOR0402_RES; DIGIKEY 311-240KGRCT-ND -> 311-100KLRCT-ND; MFN RC0603JR-07240KL -> RC0402FR-07100KL
- R8: value 750k -> 240k; DIGIKEY 311-750KGRCT-ND -> 311-240KGRCT-ND; MFN 311-750KGRCT-ND -> RC0603JR-07240KL
Connections:
- net 3V3: now also R7.2, R9.2; no longer R8.2
- net GND: now also R8.1; no longer R7.1
- net N$37: now also R8.2, R9.1; no longer R7.2, R8.1
- net RF_GPIO2: now also R7.1
Other:
- moved on the sheet: R6, R8
Changed lines of the file:
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@@
 <attributes>
 <attribute name="AUTHOR" value="Joshua Adkins"/>
-<attribute name="REV" value="B"/>
-<attribute name="TITLE" value="AUDIO SPECTRUM MODULE"/>
+<attribute name="REV" value="A"/>
+<attribute name="TITLE" value="RF Spectrum Module"/>
 </attributes>
 <variantdefs>
@@
 <part name="GND18" library="umich" deviceset="GND" device=""/>
 <part name="GND21" library="umich" deviceset="GND" device=""/>
-<part name="R8" library="passives" deviceset="RESISTOR" device="0603_RES" value="750k">
+<part name="R9" library="passives" deviceset="RESISTOR" device="0603_RES" value="750k">
 <attribute name="DIGIKEY" value="311-750KGRCT-ND"/>
 <attribute name="MF" value="Yageo"/>
 <attribute name="MFN" value="311-750KGRCT-ND"/>
 </part>
-<part name="R7" library="passives" deviceset="RESISTOR" device="0603_RES" value="240k">
+<part name="R8" library="passives" deviceset="RESISTOR" device="0603_RES" value="240k">
 <attribute name="DIGIKEY" value="311-240KGRCT-ND"/>
 <attribute name="MF" value="Yageo"/>
@@
 <attribute name="MFN" value="0901200764"/>
 </part>
+<part name="R7" library="passives" deviceset="RESISTOR" device="0402_RES" value="100k">
+<attribute name="DIGIKEY" value="311-100KLRCT-ND"/>
+<attribute name="MF" value="Yageo"/>
+<attribute name="MFN" value="RC0402FR-07100KL"/>
+</part>
 </parts>
 <sheets>
@@
 <instances>
 <instance part="FRAME1" gate="G$1" x="0" y="0"/>
-<instance part="FRAME1" gate="G$2" x="147.32" y="0"/>
+<instance part="FRAME1" gate="G$2" x="152.4" y="0"/>
 <instance part="J4" gate="G$1" x="193.04" y="53.34"/>
 <instance part="GND19" gate="1" x="175.26" y="43.18"/>
@@
 <instance part="GND18" gate="1" x="25.4" y="10.16"/>
 <instance part="GND21" gate="1" x="73.66" y="10.16"/>
-<instance part="R8" gate="G$1" x="99.06" y="35.56" rot="R90">
+<instance part="R9" gate="G$1" x="99.06" y="35.56" rot="R90">
 <attribute name="DIGIKEY" x="99.06" y="35.56" size="1.016" layer="96" rot="R90" align="bottom-center" display="off"/>
 <attribute name="MF" x="99.06" y="35.56" size="1.016" layer="96" rot="R90" align="bottom-center" display="off"/>
 <attribute name="MFN" x="99.06" y="35.56" size="1.016" layer="96" rot="R90" align="bottom-center" display="off"/>
 </instance>
-<instance part="R7" gate="G$1" x="99.06" y="22.86" rot="R90">
+<instance part="R8" gate="G$1" x="99.06" y="22.86" rot="R90">
 <attribute name="DIGIKEY" x="99.06" y="22.86" size="1.016" layer="96" rot="R90" align="bottom-center" display="off"/>
 <attribute name="MF" x="99.06" y="22.86" size="1.016" layer="96" rot="R90" align="bottom-center" display="off"/>
@@
 <wire x1="66.04" y1="15.24" x2="73.66" y2="15.24" width="0.1524" layer="91"/>
 <junction x="73.66" y="15.24"/>
-<pinref part="R7" gate="G$1" pin="1"/>
+<pinref part="R8" gate="G$1" pin="1"/>
 <wire x1="73.66" y1="17.78" x2="99.06" y2="17.78" width="0.1524" layer="91"/>
 <junction x="73.66" y="17.78"/>
@@
 <wire x1="91.44" y1="40.64" x2="91.44" y2="38.1" width="0.1524" layer="91"/>
 <junction x="86.36" y="40.64"/>
-<pinref part="R8" gate="G$1" pin="2"/>
+<pinref part="R9" gate="G$1" pin="2"/>
 <wire x1="99.06" y1="38.1" x2="99.06" y2="40.64" width="0.1524" layer="91"/>
 <wire x1="99.06" y1="40.64" x2="91.44" y2="40.64" width="0.1524" layer="91"/>
@@
 <net name="N$37" class="0">
 <segment>
-<pinref part="R7" gate="G$1" pin="2"/>
-<pinref part="R8" gate="G$1" pin="1"/>
+<pinref part="R8" gate="G$1" pin="2"/>
+<pinref part="R9" gate="G$1" pin="1"/>
 <wire x1="99.06" y1="25.4" x2="99.06" y2="30.48" width="0.1524" layer="91"/>
 <pinref part="U4" gate="G$1" pin="FB"/>
@@
 <instances>
 <instance part="FRAME2" gate="G$1" x="0" y="0"/>
-<instance part="FRAME2" gate="G$2" x="147.32" y="0"/>
+<instance part="FRAME2" gate="G$2" x="152.4" y="0"/>
 <instance part="U1" gate="G$1" x="106.68" y="119.38"/>
 <instance part="GND1" gate="1" x="78.74" y="91.44"/>
@@
 <instance part="GND3" gate="1" x="203.2" y="114.3"/>
 <instance part="GND4" gate="1" x="170.18" y="154.94"/>
-<instance part="R6" gate="G$1" x="60.96" y="124.46" rot="R90">
-<attribute name="DIGIKEY" x="60.96" y="124.46" size="1.016" layer="96" rot="R90" align="bottom-center" display="off"/>
-<attribute name="MF" x="60.96" y="124.46" size="1.016" layer="96" rot="R90" align="bottom-center" display="off"/>
-<attribute name="MFN" x="60.96" y="124.46" size="1.016" layer="96" rot="R90" align="bottom-center" display="off"/>
+<instance part="R6" gate="G$1" x="60.96" y="129.54" rot="R90">
+<attribute name="DIGIKEY" x="60.96" y="129.54" size="1.016" layer="96" rot="R90" align="bottom-center" display="off"/>
+<attribute name="MF" x="60.96" y="129.54" size="1.016" layer="96" rot="R90" align="bottom-center" display="off"/>
+<attribute name="MFN" x="60.96" y="129.54" size="1.016" layer="96" rot="R90" align="bottom-center" display="off"/>
 </instance>
 <instance part="A1" gate="G$1" x="170.18" y="167.64"/>
@@
 <attribute name="MFN" x="116.84" y="55.88" size="1.016" layer="96" align="bottom-center" display="off"/>
 </instance>
+<instance part="R7" gate="G$1" x="53.34" y="129.54" rot="R90">
+<attribute name="DIGIKEY" x="53.34" y="129.54" size="1.016" layer="96" rot="R90" align="bottom-center" display="off"/>
+<attribute name="MF" x="53.34" y="129.54" size="1.016" layer="96" rot="R90" align="bottom-center" display="off"/>
+<attribute name="MFN" x="53.34" y="129.54" size="1.016" layer="96" rot="R90" align="bottom-center" display="off"/>
+</instance>
 </instances>
 <busses>
@@
 <pinref part="R6" gate="G$1" pin="2"/>
 <wire x1="76.2" y1="147.32" x2="76.2" y2="152.4" width="0.1524" layer="91"/>
-<wire x1="60.96" y1="127" x2="60.96" y2="147.32" width="0.1524" layer="91"/>
+<wire x1="60.96" y1="132.08" x2="60.96" y2="147.32" width="0.1524" layer="91"/>
 <wire x1="60.96" y1="147.32" x2="76.2" y2="147.32" width="0.1524" layer="91"/>
 <junction x="76.2" y="147.32"/>
+<pinref part="R7" gate="G$1" pin="2"/>
+<wire x1="53.34" y1="132.08" x2="53.34" y2="147.32" width="0.1524" layer="91"/>
+<wire x1="53.34" y1="147.32" x2="60.96" y2="147.32" width="0.1524" layer="91"/>
+<junction x="60.96" y="147.32"/>
 </segment>
 </net>
@@
 <segment>
 <pinref part="U1" gate="G$1" pin="GPIO2"/>
-<wire x1="86.36" y1="119.38" x2="81.28" y2="119.38" width="0.1524" layer="91"/>
-<label x="81.28" y="119.38" size="1.016" layer="95" rot="R180" xref="yes"/>
+<wire x1="86.36" y1="119.38" x2="53.34" y2="119.38" width="0.1524" layer="91"/>
+<label x="50.8" y="119.38" size="1.016" layer="95" rot="R180" xref="yes"/>
+<pinref part="R7" gate="G$1" pin="1"/>
+<wire x1="53.34" y1="119.38" x2="50.8" y2="119.38" width="0.1524" layer="91"/>
+<wire x1="53.34" y1="124.46" x2="53.34" y2="119.38" width="0.1524" layer="91"/>
+<junction x="53.34" y="119.38"/>
 </segment>
 <segment>
@@
 <pinref part="U1" gate="G$1" pin="GPIO3"/>
 <wire x1="86.36" y1="116.84" x2="60.96" y2="116.84" width="0.1524" layer="91"/>
-<label x="55.88" y="116.84" size="1.016" layer="95" rot="R180" xref="yes"/>
+<label x="50.8" y="116.84" size="1.016" layer="95" rot="R180" xref="yes"/>
 <pinref part="R6" gate="G$1" pin="1"/>
-<wire x1="60.96" y1="116.84" x2="55.88" y2="116.84" width="0.1524" layer="91"/>
-<wire x1="60.96" y1="119.38" x2="60.96" y2="116.84" width="0.1524" layer="91"/>
+<wire x1="60.96" y1="116.84" x2="50.8" y2="116.84" width="0.1524" layer="91"/>
+<wire x1="60.96" y1="124.46" x2="60.96" y2="116.84" width="0.1524" layer="91"/>
 <junction x="60.96" y="116.84"/>
 </segment>

Commit message: integrated neal's changes
Parts:
- removed J1: (no value), SparkFun-Connectors:M04PTH
- added JP1: (no value), SparkFun-Connectors:M04PTH
Connections:
- net !RF_RESET: now also JP1.4; no longer J1.4
- net RF_GPIO2: now also JP1.1; no longer J1.1
- net RF_RX: now also JP1.2; no longer J1.2
- net RF_TX: now also JP1.3; no longer J1.3
Changed lines of the file:
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@@
 </part>
 <part name="GND10" library="umich" deviceset="GND" device=""/>
-<part name="J1" library="SparkFun-Connectors" deviceset="M04" device="PTH">
-<attribute name="DIGIKEY" value="WM8086-ND"/>
-<attribute name="MF" value="Molex"/>
-<attribute name="MFN" value="0901200764"/>
-</part>
 <part name="J2" library="SparkFun-Connectors" deviceset="M04" device="PTH">
 <attribute name="DIGIKEY" value="WM8086-ND"/>
@@
 <attribute name="MFN" value="RC0402FR-07100KL"/>
 </part>
+<part name="JP1" library="SparkFun-Connectors" deviceset="M04" device="PTH"/>
 </parts>
 <sheets>
@@
 </instance>
 <instance part="GND10" gate="1" x="134.62" y="142.24"/>
-<instance part="J1" gate="G$1" x="78.74" y="55.88">
-<attribute name="DIGIKEY" x="78.74" y="55.88" size="1.016" layer="96" align="bottom-center" display="off"/>
-<attribute name="MF" x="78.74" y="55.88" size="1.016" layer="96" align="bottom-center" display="off"/>
-<attribute name="MFN" x="78.74" y="55.88" size="1.016" layer="96" align="bottom-center" display="off"/>
-</instance>
 <instance part="J2" gate="G$1" x="116.84" y="55.88">
 <attribute name="DIGIKEY" x="116.84" y="55.88" size="1.016" layer="96" align="bottom-center" display="off"/>
@@
 <attribute name="MFN" x="53.34" y="129.54" size="1.016" layer="96" rot="R90" align="bottom-center" display="off"/>
 </instance>
+<instance part="JP1" gate="G$1" x="76.2" y="55.88"/>
 </instances>
 <busses>
@@
 </segment>
 <segment>
-<pinref part="J1" gate="G$1" pin="3"/>
-<wire x1="83.82" y1="58.42" x2="86.36" y2="58.42" width="0.1524" layer="91"/>
+<wire x1="81.28" y1="58.42" x2="86.36" y2="58.42" width="0.1524" layer="91"/>
 <label x="86.36" y="58.42" size="1.27" layer="95" xref="yes"/>
+<pinref part="JP1" gate="G$1" pin="3"/>
 </segment>
 </net>
@@
 </segment>
 <segment>
-<pinref part="J1" gate="G$1" pin="2"/>
-<wire x1="83.82" y1="55.88" x2="86.36" y2="55.88" width="0.1524" layer="91"/>
+<wire x1="81.28" y1="55.88" x2="86.36" y2="55.88" width="0.1524" layer="91"/>
 <label x="86.36" y="55.88" size="1.27" layer="95" xref="yes"/>
+<pinref part="JP1" gate="G$1" pin="2"/>
 </segment>
 </net>
@@
 </segment>
 <segment>
-<pinref part="J1" gate="G$1" pin="4"/>
-<wire x1="83.82" y1="60.96" x2="86.36" y2="60.96" width="0.1524" layer="91"/>
+<wire x1="81.28" y1="60.96" x2="86.36" y2="60.96" width="0.1524" layer="91"/>
 <label x="86.36" y="60.96" size="1.27" layer="95" xref="yes"/>
+<pinref part="JP1" gate="G$1" pin="4"/>
 </segment>
 </net>
@@
 </segment>
 <segment>
-<pinref part="J1" gate="G$1" pin="1"/>
-<wire x1="83.82" y1="53.34" x2="86.36" y2="53.34" width="0.1524" layer="91"/>
+<wire x1="81.28" y1="53.34" x2="86.36" y2="53.34" width="0.1524" layer="91"/>
 <label x="86.36" y="53.34" size="1.27" layer="95" xref="yes"/>
-</segment>
-</net>
+<pinref part="JP1" gate="G$1" pin="1"/>
+</segment>
+</net>

Commit message: consistent again - got otu sync
Parts:
- removed JP1: (no value), SparkFun-Connectors:M04PTH
- added J1: (no value), SparkFun-Connectors:M04PTH
- R4: DIGIKEY RHM10KCECT-ND -> 311-1.0KJRCT-ND; MF Rohm -> Yageo; MFN MCR01MRTJ103 -> RC0402JR-071KL
Connections:
- removed net R4: R4.1
- net !RF_RESET: now also J1.4; no longer JP1.4
- net GND: now also R4.1
- net RF_GPIO2: now also J1.1; no longer JP1.1
- net RF_RX: now also J1.2; no longer JP1.2
- net RF_TX: now also J1.3; no longer JP1.3
Other:
- moved on the sheet: R4
Changed lines of the file:
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@@
 <attribute name="MFN" value="GRM155R60J105KE19D"/>
-</part>
-<part name="R4" library="passives" deviceset="RESISTOR" device="0402_RES" value="10k">
-<attribute name="DIGIKEY" value="RHM10KCECT-ND"/>
-<attribute name="MF" value="Rohm"/>
-<attribute name="MFN" value="MCR01MRTJ103"/>
 </part>
 <part name="GND6" library="umich" deviceset="GND" device=""/>
@@
 </part>
 <part name="GND7" library="umich" deviceset="GND" device=""/>
-<part name="GND8" library="umich" deviceset="GND" device=""/>
 <part name="R6" library="passives" deviceset="RESISTOR" device="0402_RES" value="100k">
 <attribute name="DIGIKEY" value="311-100KLRCT-ND"/>
@@
 <attribute name="MFN" value="RC0402FR-07100KL"/>
 </part>
-<part name="JP1" library="SparkFun-Connectors" deviceset="M04" device="PTH"/>
+<part name="R4" library="passives" deviceset="RESISTOR" device="0402_RES" value="10k">
+<attribute name="DIGIKEY" value="311-1.0KJRCT-ND"/>
+<attribute name="MF" value="Yageo"/>
+<attribute name="MFN" value="RC0402JR-071KL"/>
+</part>
+<part name="GND8" library="umich" deviceset="GND" device=""/>
+<part name="J1" library="SparkFun-Connectors" deviceset="M04" device="PTH">
+<attribute name="DIGIKEY" value="WM8086-ND"/>
+<attribute name="MF" value="Molex"/>
+<attribute name="MFN" value="0901200764"/>
+</part>
 </parts>
 <sheets>
@@
 <attribute name="MFN" x="139.7" y="149.86" size="1.016" layer="96" align="bottom-center" display="off"/>
 </instance>
-<instance part="R4" gate="G$1" x="226.06" y="132.08" rot="R90">
-<attribute name="DIGIKEY" x="226.06" y="132.08" size="1.016" layer="96" rot="R90" align="bottom-center" display="off"/>
-<attribute name="MF" x="226.06" y="132.08" size="1.016" layer="96" rot="R90" align="bottom-center" display="off"/>
-<attribute name="MFN" x="226.06" y="132.08" size="1.016" layer="96" rot="R90" align="bottom-center" display="off"/>
-</instance>
 <instance part="GND6" gate="1" x="149.86" y="88.9"/>
 <instance part="X1" gate="G$1" x="101.6" y="132.08" rot="R270"/>
@@
 </instance>
 <instance part="GND7" gate="1" x="88.9" y="116.84"/>
-<instance part="GND8" gate="1" x="226.06" y="121.92"/>
 <instance part="D1" gate="G$1" x="127" y="101.6" rot="R270">
 <attribute name="DIGIKEY" x="127" y="101.6" size="1.016" layer="96" rot="R270" align="bottom-center" display="off"/>
@@
 </instance>
 <instance part="GND9" gate="1" x="127" y="91.44"/>
+<instance part="R4" gate="G$1" x="226.06" y="129.54" rot="R90">
+<attribute name="DIGIKEY" x="226.06" y="129.54" size="1.016" layer="96" rot="R90" align="bottom-center" display="off"/>
+<attribute name="MF" x="226.06" y="129.54" size="1.016" layer="96" rot="R90" align="bottom-center" display="off"/>
+<attribute name="MFN" x="226.06" y="129.54" size="1.016" layer="96" rot="R90" align="bottom-center" display="off"/>
+</instance>
+<instance part="GND8" gate="1" x="226.06" y="119.38"/>
 </instances>
 <busses>
@@
 <wire x1="134.62" y1="96.52" x2="134.62" y2="99.06" width="0.1524" layer="91"/>
 <junction x="127" y="96.52"/>
+</segment>
+<segment>
+<pinref part="R4" gate="G$1" pin="1"/>
+<pinref part="GND8" gate="1" pin="GND"/>
+<wire x1="226.06" y1="124.46" x2="226.06" y2="121.92" width="0.1524" layer="91"/>
 </segment>
 </net>
@@
 </segment>
 <segment>
-<pinref part="U3" gate="G$1" pin="PA9"/>
-<wire x1="203.2" y1="109.22" x2="208.28" y2="109.22" width="0.1524" layer="91"/>
-<label x="208.28" y="109.22" size="1.27" layer="95" xref="yes"/>
-</segment>
-<segment>
 <pinref part="U3" gate="G$1" pin="PA7"/>
 <wire x1="203.2" y1="114.3" x2="208.28" y2="114.3" width="0.1524" layer="91"/>
 <label x="208.28" y="114.3" size="1.27" layer="95" xref="yes"/>
+</segment>
+<segment>
+<pinref part="U3" gate="G$1" pin="PA9"/>
+<wire x1="203.2" y1="109.22" x2="208.28" y2="109.22" width="0.1524" layer="91"/>
+<label x="208.28" y="109.22" size="1.016" layer="95" xref="yes"/>
 </segment>
 </net>
@@
 <segment>
 <pinref part="U3" gate="G$1" pin="PH3/BOOT0"/>
+<wire x1="203.2" y1="137.16" x2="226.06" y2="137.16" width="0.1524" layer="91"/>
 <pinref part="R4" gate="G$1" pin="2"/>
-<wire x1="203.2" y1="137.16" x2="226.06" y2="137.16" width="0.1524" layer="91"/>
-<wire x1="226.06" y1="137.16" x2="226.06" y2="134.62" width="0.1524" layer="91"/>
+<wire x1="226.06" y1="132.08" x2="226.06" y2="137.16" width="0.1524" layer="91"/>
 </segment>
 </net>
@@
 <pinref part="R3" gate="G$1" pin="1"/>
 <wire x1="134.62" y1="104.14" x2="134.62" y2="106.68" width="0.1524" layer="91"/>
-</segment>
-</net>
-<net name="R4" class="0">
-<segment>
-<pinref part="R4" gate="G$1" pin="1"/>
-<pinref part="GND8" gate="1" pin="GND"/>
-<wire x1="226.06" y1="127" x2="226.06" y2="124.46" width="0.1524" layer="91"/>
 </segment>
 </net>
@@
 <attribute name="MFN" x="53.34" y="129.54" size="1.016" layer="96" rot="R90" align="bottom-center" display="off"/>
 </instance>
-<instance part="JP1" gate="G$1" x="76.2" y="55.88"/>
+<instance part="J1" gate="G$1" x="78.74" y="55.88">
+<attribute name="DIGIKEY" x="78.74" y="55.88" size="1.016" layer="96" align="bottom-center" display="off"/>
+<attribute name="MF" x="78.74" y="55.88" size="1.016" layer="96" align="bottom-center" display="off"/>
+<attribute name="MFN" x="78.74" y="55.88" size="1.016" layer="96" align="bottom-center" display="off"/>
+</instance>
 </instances>
 <busses>
@@
 </segment>
 <segment>
-<wire x1="81.28" y1="58.42" x2="86.36" y2="58.42" width="0.1524" layer="91"/>
+<wire x1="83.82" y1="58.42" x2="86.36" y2="58.42" width="0.1524" layer="91"/>
 <label x="86.36" y="58.42" size="1.27" layer="95" xref="yes"/>
-<pinref part="JP1" gate="G$1" pin="3"/>
+<pinref part="J1" gate="G$1" pin="3"/>
 </segment>
 </net>
@@
 </segment>
 <segment>
-<wire x1="81.28" y1="55.88" x2="86.36" y2="55.88" width="0.1524" layer="91"/>
+<wire x1="83.82" y1="55.88" x2="86.36" y2="55.88" width="0.1524" layer="91"/>
 <label x="86.36" y="55.88" size="1.27" layer="95" xref="yes"/>
-<pinref part="JP1" gate="G$1" pin="2"/>
+<pinref part="J1" gate="G$1" pin="2"/>
 </segment>
 </net>
@@
 </segment>
 <segment>
-<wire x1="81.28" y1="60.96" x2="86.36" y2="60.96" width="0.1524" layer="91"/>
+<wire x1="83.82" y1="60.96" x2="86.36" y2="60.96" width="0.1524" layer="91"/>
 <label x="86.36" y="60.96" size="1.27" layer="95" xref="yes"/>
-<pinref part="JP1" gate="G$1" pin="4"/>
+<pinref part="J1" gate="G$1" pin="4"/>
 </segment>
 </net>
@@
 </segment>
 <segment>
-<wire x1="81.28" y1="53.34" x2="86.36" y2="53.34" width="0.1524" layer="91"/>
+<wire x1="83.82" y1="53.34" x2="86.36" y2="53.34" width="0.1524" layer="91"/>
 <label x="86.36" y="53.34" size="1.27" layer="95" xref="yes"/>
-<pinref part="JP1" gate="G$1" pin="1"/>
-</segment>
-</net>
+<pinref part="J1" gate="G$1" pin="1"/>
+</segment>
+</net>
