File: hardware/radio_module/rev_b/radio_module.sch (EAGLE design)
At the start: 138 parts, among them J1 MODULE_GENERIC_DEBUGSMT, J10 TC2030-JLINK-NL, J11 U.FL-R-SMT, J12 U.FL-R-SMT, J2 MOLEX_73251-135X, J3 MOLEX_73251-135X, J4 NANO_SIM, J8 TC2030-JLINK-NL, J9 TC2030-JLINK-L, Q1 MOSFET-NCHANNELSMD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

Commit message: fixed up some schematic aesthetics
Changed lines of the file:
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@@
 <attribute name="DIGIKEY" value="490-10777-1-ND"/>
 </part>
-<part name="P+2" library="supply1" library_urn="urn:adsk.eagle:library:371" deviceset="VCC" device=""/>
 <part name="GND46" library="supply1" library_urn="urn:adsk.eagle:library:371" deviceset="GND" device=""/>
 <part name="C14" library="passives" deviceset="CAPACITOR" device="0402_CAP" value="1nF">
@@
 <part name="J10" library="connector" deviceset="TC2030-JLINK" device="-NL"/>
 <part name="GND57" library="supply1" library_urn="urn:adsk.eagle:library:371" deviceset="GND" device=""/>
-<part name="P+4" library="supply1" library_urn="urn:adsk.eagle:library:371" deviceset="VCC" device=""/>
 <part name="X5" library="crystals" deviceset="ABS05-32.768KHZ" device="-9-T"/>
 <part name="C6" library="passives" deviceset="CAPACITOR" device="0402_CAP" value="12pF">
@@
 </part>
 <part name="GND59" library="supply1" library_urn="urn:adsk.eagle:library:371" deviceset="GND" device=""/>
-<part name="P+5" library="supply1" library_urn="urn:adsk.eagle:library:371" deviceset="VCC" device=""/>
 <part name="J5" library="pinhead" library_urn="urn:adsk.eagle:library:325" deviceset="PINHD-2X4" device="">
 <attribute name="DIGIKEY" value="952-2123-ND"/>
@@
 <attribute name="DIGIKEY" value="609-3243-ND"/>
 </part>
+<part name="FRAME6" library="lab11-frames" deviceset="LETTER_L_UMICH" device=""/>
 </parts>
 <sheets>
@@
 <wire x1="0" y1="63.5" x2="66.04" y2="63.5" width="0.1524" layer="97"/>
 <wire x1="66.04" y1="63.5" x2="66.04" y2="0" width="0.1524" layer="97"/>
-<wire x1="66.04" y1="185.42" x2="66.04" y2="71.12" width="0.1524" layer="97"/>
+<wire x1="66.04" y1="190.5" x2="66.04" y2="71.12" width="0.1524" layer="97"/>
 <wire x1="66.04" y1="71.12" x2="0" y2="71.12" width="0.1524" layer="97"/>
 <text x="2.54" y="137.16" size="2.54" layer="97">Level Translator, GSM_INT = 1.8V</text>
@@
 <pinref part="Q4" gate="G$1" pin="D"/>
 <wire x1="190.5" y1="137.16" x2="190.5" y2="149.86" width="0.1524" layer="91"/>
+<label x="152.4" y="137.16" size="1.016" layer="95" rot="R90" xref="yes"/>
 </segment>
 <segment>
@@
 <attribute name="DIGIKEY" x="66.04" y="144.78" size="1.778" layer="96" display="off"/>
 </instance>
-<instance part="P+2" gate="VCC" x="73.66" y="154.94"/>
 <instance part="GND46" gate="1" x="60.96" y="132.08"/>
 <instance part="C14" gate="G$1" x="88.9" y="144.78">
@@
 <instance part="J10" gate="G$1" x="129.54" y="139.7"/>
 <instance part="GND57" gate="1" x="114.3" y="129.54"/>
-<instance part="P+4" gate="VCC" x="114.3" y="149.86"/>
 <instance part="X5" gate="G$1" x="129.54" y="111.76"/>
 <instance part="C6" gate="G$1" x="121.92" y="106.68">
@@
 </instance>
 <instance part="GND59" gate="1" x="40.64" y="30.48"/>
-<instance part="P+5" gate="VCC" x="17.78" y="106.68"/>
 </instances>
 <busses>
@@
 <wire x1="73.66" y1="149.86" x2="66.04" y2="149.86" width="0.1524" layer="91"/>
 <wire x1="66.04" y1="149.86" x2="66.04" y2="147.32" width="0.1524" layer="91"/>
-<pinref part="P+2" gate="VCC" pin="VCC"/>
 <pinref part="C32" gate="G$1" pin="1"/>
 <wire x1="55.88" y1="147.32" x2="55.88" y2="149.86" width="0.1524" layer="91"/>
@@
 <wire x1="73.66" y1="127" x2="73.66" y2="149.86" width="0.1524" layer="91"/>
 <junction x="73.66" y="149.86"/>
+<label x="73.66" y="152.4" size="1.016" layer="95" rot="R90" xref="yes"/>
 </segment>
 <segment>
@@
 <wire x1="116.84" y1="144.78" x2="114.3" y2="144.78" width="0.1524" layer="91"/>
 <wire x1="114.3" y1="144.78" x2="114.3" y2="147.32" width="0.1524" layer="91"/>
-<pinref part="P+4" gate="VCC" pin="VCC"/>
+<label x="114.3" y="147.32" size="1.016" layer="95" rot="R90" xref="yes"/>
 </segment>
 <segment>
 <pinref part="R16" gate="G$1" pin="1"/>
 <wire x1="17.78" y1="101.6" x2="17.78" y2="104.14" width="0.1524" layer="91"/>
-<pinref part="P+5" gate="VCC" pin="VCC"/>
+<label x="17.78" y="104.14" size="1.016" layer="95" rot="R90" xref="yes"/>
 </segment>
 <segment>
@@
 <attribute name="DIGIKEY" x="109.22" y="99.06" size="1.016" layer="96" align="bottom-center" display="off"/>
 </instance>
+<instance part="FRAME6" gate="G$1" x="0" y="0"/>
+<instance part="FRAME6" gate="G$2" x="152.4" y="0"/>
 </instances>
 <busses>

Commit message: switch PPS to tc* pin
Connections:
- net !XDOT_RESET: now also U6.PB04; no longer U6.PA10
- net PPS: now also U6.PA10; no longer U6.PB04
Changed lines of the file:
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@@
 <net name="PPS" class="0">
-<segment>
-<pinref part="U6" gate="U1" pin="PB04"/>
-<label x="121.92" y="119.38" size="1.27" layer="95" rot="R180" xref="yes"/>
-<wire x1="129.54" y1="119.38" x2="121.92" y2="119.38" width="0.1524" layer="91"/>
-</segment>
 <segment>
 <pinref part="J1" gate="G$1" pin="PPS"/>
 <wire x1="25.4" y1="170.18" x2="30.48" y2="170.18" width="0.1524" layer="91"/>
 <label x="30.48" y="170.18" size="1.27" layer="95" xref="yes"/>
+</segment>
+<segment>
+<pinref part="U6" gate="U1" pin="PA10"/>
+<label x="177.8" y="134.62" size="1.27" layer="95" xref="yes"/>
+<wire x1="170.18" y1="134.62" x2="177.8" y2="134.62" width="0.1524" layer="91"/>
 </segment>
 </net>
@@
 <net name="!XDOT_RESET" class="0">
 <segment>
-<pinref part="U6" gate="U1" pin="PA10"/>
-<label x="177.8" y="134.62" size="1.27" layer="95" xref="yes"/>
-<wire x1="170.18" y1="134.62" x2="177.8" y2="134.62" width="0.1524" layer="91"/>
+<pinref part="U6" gate="U1" pin="PB04"/>
+<label x="121.92" y="119.38" size="1.27" layer="95" rot="R180" xref="yes"/>
+<wire x1="129.54" y1="119.38" x2="121.92" y2="119.38" width="0.1524" layer="91"/>
 </segment>
 </net>

Commit message: integrated radio module changes
Other:
- note removed: "Connector for FW upgrade"
Changed lines of the file:
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@@
 <text x="33.02" y="10.16" size="2.54" layer="97">Pull down to
 prevent glitching</text>
-<text x="12.7" y="55.88" size="2.54" layer="97">Network Indicator LED</text>
-<wire x1="0" y1="63.5" x2="66.04" y2="63.5" width="0.1524" layer="97"/>
-<wire x1="66.04" y1="63.5" x2="66.04" y2="0" width="0.1524" layer="97"/>
+<text x="10.16" y="60.96" size="2.54" layer="97">Network Indicator LED</text>
+<wire x1="0" y1="66.04" x2="66.04" y2="66.04" width="0.1524" layer="97"/>
+<wire x1="66.04" y1="66.04" x2="66.04" y2="0" width="0.1524" layer="97"/>
 <wire x1="66.04" y1="190.5" x2="66.04" y2="71.12" width="0.1524" layer="97"/>
 <wire x1="66.04" y1="71.12" x2="0" y2="71.12" width="0.1524" layer="97"/>
 <text x="2.54" y="137.16" size="2.54" layer="97">Level Translator, GSM_INT = 1.8V</text>
 <text x="71.12" y="96.52" size="1.27" layer="97">UART lines for commands</text>
-<text x="71.12" y="71.12" size="1.27" layer="97">Connector for FW upgrade</text>
 <text x="22.86" y="78.74" size="1.27" layer="97" align="bottom-center">I switch labels here to be consistent</text>
 <wire x1="15.24" y1="81.28" x2="15.24" y2="86.36" width="0.254" layer="96"/>
@@
 <attribute name="DIGIKEY" x="109.22" y="132.08" size="1.016" layer="96" rot="R90" align="bottom-center" display="off"/>
 </instance>
-<instance part="C9" gate="G$1" x="198.12" y="66.04">
+<instance part="C9" gate="G$1" x="198.12" y="66.04" smashed="yes">
 <attribute name="DIGIKEY" x="198.12" y="66.04" size="1.016" layer="96" align="bottom-center" display="off"/>
-</instance>
-<instance part="C10" gate="G$1" x="193.04" y="68.58">
+<attribute name="NAME" x="195.58" y="68.58" size="1.778" layer="95" ratio="12" rot="R270" align="bottom-center"/>
+<attribute name="VALUE" x="195.58" y="60.96" size="1.778" layer="96" ratio="12" rot="R270" align="bottom-center"/>
+</instance>
+<instance part="C10" gate="G$1" x="193.04" y="68.58" smashed="yes">
 <attribute name="DIGIKEY" x="193.04" y="68.58" size="1.016" layer="96" align="bottom-center" display="off"/>
-</instance>
-<instance part="C11" gate="G$1" x="187.96" y="71.12">
+<attribute name="NAME" x="190.5" y="71.12" size="1.778" layer="95" ratio="12" rot="R270" align="bottom-center"/>
+<attribute name="VALUE" x="190.5" y="63.5" size="1.778" layer="96" ratio="12" rot="R270" align="bottom-center"/>
+</instance>
+<instance part="C11" gate="G$1" x="187.96" y="71.12" smashed="yes">
 <attribute name="DIGIKEY" x="187.96" y="71.12" size="1.016" layer="96" align="bottom-center" display="off"/>
-</instance>
-<instance part="C12" gate="G$1" x="182.88" y="73.66">
+<attribute name="NAME" x="185.42" y="73.66" size="1.778" layer="95" ratio="12" rot="R270" align="bottom-center"/>
+<attribute name="VALUE" x="185.42" y="66.04" size="1.778" layer="96" ratio="12" rot="R270" align="bottom-center"/>
+</instance>
+<instance part="C12" gate="G$1" x="182.88" y="73.66" smashed="yes">
 <attribute name="DIGIKEY" x="182.88" y="73.66" size="1.016" layer="96" align="bottom-center" display="off"/>
+<attribute name="NAME" x="180.34" y="76.2" size="1.778" layer="95" ratio="12" rot="R270" align="bottom-center"/>
+<attribute name="VALUE" x="180.34" y="68.58" size="1.778" layer="96" ratio="12" rot="R270" align="bottom-center"/>
 </instance>
 <instance part="GND6" gate="1" x="99.06" y="121.92"/>
@@
 <wire x1="88.9" y1="147.32" x2="88.9" y2="149.86" width="0.1524" layer="91"/>
 <pinref part="L1" gate="G$1" pin="1"/>
-<wire x1="35.56" y1="154.94" x2="35.56" y2="160.02" width="0.1524" layer="91"/>
+<wire x1="35.56" y1="154.94" x2="35.56" y2="162.56" width="0.1524" layer="91"/>
 <pinref part="U13" gate="G$1" pin="AVDD"/>
-<wire x1="35.56" y1="160.02" x2="27.94" y2="160.02" width="0.1524" layer="91"/>
-<wire x1="27.94" y1="160.02" x2="78.74" y2="160.02" width="0.1524" layer="91"/>
-<wire x1="78.74" y1="160.02" x2="78.74" y2="149.86" width="0.1524" layer="91"/>
+<wire x1="35.56" y1="162.56" x2="78.74" y2="162.56" width="0.1524" layer="91"/>
+<wire x1="78.74" y1="162.56" x2="78.74" y2="149.86" width="0.1524" layer="91"/>
 <wire x1="78.74" y1="149.86" x2="78.74" y2="127" width="0.1524" layer="91"/>
 <wire x1="88.9" y1="149.86" x2="78.74" y2="149.86" width="0.1524" layer="91"/>
 <junction x="78.74" y="149.86"/>
 <pinref part="C30" gate="G$1" pin="1"/>
-<wire x1="27.94" y1="152.4" x2="27.94" y2="160.02" width="0.1524" layer="91"/>
-<junction x="27.94" y="160.02"/>
+<wire x1="27.94" y1="152.4" x2="27.94" y2="162.56" width="0.1524" layer="91"/>
+<wire x1="27.94" y1="162.56" x2="35.56" y2="162.56" width="0.1524" layer="91"/>
+<junction x="35.56" y="162.56"/>
 </segment>
 </net>
@@
 <wire x1="68.58" y1="134.62" x2="0" y2="134.62" width="0.1524" layer="97"/>
 <text x="12.7" y="177.8" size="1.27" layer="97">To Program the STM32L on the Module</text>
-<text x="111.76" y="129.54" size="1.27" layer="97">DNP</text>
 </plain>
 <instances>

Commit message: fixed a few of the part numbers
Parts:
- C10, C11, C12, C9: DIGIKEY 491-6241-1-ND -> 490-6241-1-ND
- C20: DIGIKEY 491-6241-1-ND -> 490-3254-1-ND; MF (none) -> Murata; MFN (none) -> GRM155R71E473KA88D
- C30: DIGIKEY 1276-1513-1-ND -> 490-1320-1-ND; MF (none) -> Murata; MFN (none) -> GRM155R60J105KE19D
- U6: DIGIKEY (none) -> ATSAM4LC8BA-MU
Changed lines of the file:
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@@
 </part>
 <part name="C9" library="passives" deviceset="CAPACITOR" device="0402_CAP" value="47pF">
-<attribute name="DIGIKEY" value="491-6241-1-ND "/>
+<attribute name="DIGIKEY" value="490-6241-1-ND"/>
 </part>
 <part name="C10" library="passives" deviceset="CAPACITOR" device="0402_CAP" value="47pF">
-<attribute name="DIGIKEY" value="491-6241-1-ND "/>
+<attribute name="DIGIKEY" value="490-6241-1-ND "/>
 </part>
 <part name="C11" library="passives" deviceset="CAPACITOR" device="0402_CAP" value="47pF">
-<attribute name="DIGIKEY" value="491-6241-1-ND "/>
+<attribute name="DIGIKEY" value="490-6241-1-ND "/>
 </part>
 <part name="C12" library="passives" deviceset="CAPACITOR" device="0402_CAP" value="47pF">
-<attribute name="DIGIKEY" value="491-6241-1-ND "/>
+<attribute name="DIGIKEY" value="490-6241-1-ND "/>
 </part>
 <part name="GND6" library="umich" deviceset="GND" device=""/>
@@
 </part>
 <part name="L3" library="passives" deviceset="INDUCTOR" device="IHL" value="2.2uH"/>
-<part name="U6" library="chips" deviceset="SAM4LC8BA" device=""/>
+<part name="U6" library="chips" deviceset="SAM4LC8BA" device="">
+<attribute name="DIGIKEY" value="ATSAM4LC8BA-MU"/>
+</part>
 <part name="GND10" library="umich" deviceset="GND" device=""/>
 <part name="U1" library="signpost" deviceset="LTC2941" device=""/>
@@
 </part>
 <part name="C30" library="passives" deviceset="CAPACITOR" device="0402_CAP" value="1uF">
-<attribute name="DIGIKEY" value="1276-1513-1-ND"/>
+<attribute name="DIGIKEY" value="490-1320-1-ND"/>
+<attribute name="MF" value="Murata"/>
+<attribute name="MFN" value="GRM155R60J105KE19D"/>
 </part>
 <part name="X4" library="crystals" deviceset="TXC-8Y" device="" value="16MHz">
@@
 </part>
 <part name="C20" library="passives" deviceset="CAPACITOR" device="0402_CAP" value="47nF">
-<attribute name="DIGIKEY" value="491-6241-1-ND"/>
+<attribute name="DIGIKEY" value="490-3254-1-ND"/>
+<attribute name="MF" value="Murata"/>
+<attribute name="MFN" value="GRM155R71E473KA88D"/>
 </part>
 <part name="GND51" library="supply1" library_urn="urn:adsk.eagle:library:371" deviceset="GND" device=""/>
@@
 <instance part="C30" gate="G$1" x="27.94" y="149.86">
 <attribute name="DIGIKEY" x="27.94" y="149.86" size="1.778" layer="96" display="off"/>
+<attribute name="MF" x="27.94" y="149.86" size="1.016" layer="96" align="bottom-center" display="off"/>
+<attribute name="MFN" x="27.94" y="149.86" size="1.016" layer="96" align="bottom-center" display="off"/>
 </instance>
 <instance part="X4" gate="G$1" x="157.48" y="111.76">
@@
 <instance part="C20" gate="G$1" x="106.68" y="50.8">
 <attribute name="DIGIKEY" x="106.68" y="50.8" size="1.778" layer="96" display="off"/>
+<attribute name="MF" x="106.68" y="50.8" size="1.016" layer="96" align="bottom-center" display="off"/>
+<attribute name="MFN" x="106.68" y="50.8" size="1.016" layer="96" align="bottom-center" display="off"/>
 </instance>
 <instance part="GND51" gate="1" x="106.68" y="30.48"/>

Commit message: fixed a consistency error
Parts:
- C20: MF Murata -> (none); MFN GRM155R71E473KA88D -> (none)
- C30: MF Murata -> (none); MFN GRM155R60J105KE19D -> (none)
Changed lines of the file:
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@@
 <part name="C30" library="passives" deviceset="CAPACITOR" device="0402_CAP" value="1uF">
 <attribute name="DIGIKEY" value="490-1320-1-ND"/>
-<attribute name="MF" value="Murata"/>
-<attribute name="MFN" value="GRM155R60J105KE19D"/>
 </part>
 <part name="X4" library="crystals" deviceset="TXC-8Y" device="" value="16MHz">
@@
 <part name="C20" library="passives" deviceset="CAPACITOR" device="0402_CAP" value="47nF">
 <attribute name="DIGIKEY" value="490-3254-1-ND"/>
-<attribute name="MF" value="Murata"/>
-<attribute name="MFN" value="GRM155R71E473KA88D"/>
 </part>
 <part name="GND51" library="supply1" library_urn="urn:adsk.eagle:library:371" deviceset="GND" device=""/>
@@
 <instance part="C30" gate="G$1" x="27.94" y="149.86">
 <attribute name="DIGIKEY" x="27.94" y="149.86" size="1.778" layer="96" display="off"/>
-<attribute name="MF" x="27.94" y="149.86" size="1.016" layer="96" align="bottom-center" display="off"/>
-<attribute name="MFN" x="27.94" y="149.86" size="1.016" layer="96" align="bottom-center" display="off"/>
 </instance>
 <instance part="X4" gate="G$1" x="157.48" y="111.76">
@@
 <instance part="C20" gate="G$1" x="106.68" y="50.8">
 <attribute name="DIGIKEY" x="106.68" y="50.8" size="1.778" layer="96" display="off"/>
-<attribute name="MF" x="106.68" y="50.8" size="1.016" layer="96" align="bottom-center" display="off"/>
-<attribute name="MFN" x="106.68" y="50.8" size="1.016" layer="96" align="bottom-center" display="off"/>
 </instance>
 <instance part="GND51" gate="1" x="106.68" y="30.48"/>

Commit message: Saving future me from having wrong packages at assembly
Parts:
- C8: DIGIKEY 490-6241-1-ND -> 712-1342-1-ND
- FB1: DIGIKEY 490-5216-1-ND -> 445-2158-1-ND
- Q1, Q2, Q3: DIGIKEY SI2333DDS-T1-GE3CT-ND -> 2N7002LT1GOSCT-ND
Changed lines of the file:
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@@
 </part>
 <part name="C8" library="passives" deviceset="CAPACITOR" device="0603_CAP" value="33pF">
-<attribute name="DIGIKEY" value="490-6241-1-ND "/>
+<attribute name="DIGIKEY" value="712-1342-1-ND"/>
 </part>
 <part name="FRAME2" library="lab11-frames" deviceset="LETTER_L_UMICH" device=""/>
@@
 </part>
 <part name="FB1" library="passives" deviceset="FERRITE_BEAD" device="0402" value="1.5k">
-<attribute name="DIGIKEY" value="490-5216-1-ND"/>
+<attribute name="DIGIKEY" value="445-2158-1-ND"/>
 </part>
 <part name="L5" library="signpost" deviceset="LHQ3NP" device="" value="22uH"/>
@@
 </part>
 <part name="Q1" library="fets" deviceset="MOSFET-NCHANNEL" device="SMD">
-<attribute name="DIGIKEY" value="SI2333DDS-T1-GE3CT-ND "/>
+<attribute name="DIGIKEY" value="2N7002LT1GOSCT-ND"/>
 </part>
 <part name="Q2" library="fets" deviceset="MOSFET-NCHANNEL" device="SMD">
-<attribute name="DIGIKEY" value="SI2333DDS-T1-GE3CT-ND "/>
+<attribute name="DIGIKEY" value="2N7002LT1GOSCT-ND"/>
 </part>
 <part name="Q3" library="fets" deviceset="MOSFET-NCHANNEL" device="SMD">
-<attribute name="DIGIKEY" value="SI2333DDS-T1-GE3CT-ND "/>
+<attribute name="DIGIKEY" value="2N7002LT1GOSCT-ND"/>
 </part>
 <part name="U11" library="signpost" deviceset="XDOT_MODULE" device=""/>
