File: hardware/backplane/rev_d/backplane.sch (EAGLE design)
At the start: 386 parts, among them J0 BACKPLANE_GENERIC_MODULE, J1 BACKPLANE_GENERIC_MODULE, J2 BACKPLANE_GENERIC_MODULE, J3 BACKPLANE_CONTROLLER_MODULE, J4 BACKPLANE_POWER_MODULE, J5 BACKPLANE_GENERIC_MODULE, J6 BACKPLANE_GENERIC_MODULE, J7 BACKPLANE_GENERIC_MODULE, J8 SCREW-TERMINAL_2_0.100, J9 SCREW-TERMINAL_2_0.100, U1 TUSB2077A, U10 SN74LVC2T45, U11 SN74LVC2T45, U12 SN74LVC2T45, U13 SN74LVC2T45, U14 SN74LVC2T45, U15 SN74LVC2T45, U16 SN74LVC2T45, U17 SN74LVC2T45, U18 SN74LVC2T45, U19 SN74LVC2T45, U2 FXMA2102, U20 TS3USB30E, U21 TS3USB30E, U22 TS3USB30E, U23 TS3USB30E, U24 TS3USB30E, U25 TS3USB30E, U26 MCP23008QFN, U27 MCP23008QFN, U28 MCP23008QFN, U29 MCP23008QFN, U3 FXMA2102, U30 MCP23008QFN, U31 MCP23008QFN, U32 MCP23008QFN, U33 NCP301LSN30, U34 M24C01WMN, U4 FXMA2102, U5 FXMA2102, U6 FXMA2102, U7 FXMA2102, U8 SN74LVC2T45, U9 SN74LVC2T45, Y1 ABMM

Commit message: backplane: hub !BUSPWR -> high
Resolves errata from revC:

USB !BUSPWR is wrong: Currently tied to GND, which states that the hub and
all downstream devices are powered from the upstream port. Should be tied
high, stating that the hub has an "external" power supply. In both modes,
the hub still will perform overcurrent and poweroff protections.

  - Symptom: This limits the hub to 500mA max total draw, as each
    downstream port has a minimum 100mA allotment (USB spec), so the hub
    disables higher ports (cannot use USB in Module 5 or Module 7 slot)
  - Remedy: Cut trace at pin 10 (!BUSPWR) and short pins 10 and 9.
Connections:
- net GND: no longer U1.!BUSPWR
- net VCC_BACKPLANE: now also U1.!BUSPWR
Other:
- note added: "This hub & downstream ports are "externally" powered (not limited to 500mA from host)"
- note removed: "Downstream ports draw VBUS from the "cable""
Changed lines of the file:
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@@
 <?xml version="1.0" encoding="utf-8"?>
 <!DOCTYPE eagle SYSTEM "eagle.dtd">
-<eagle version="8.1.1">
+<eagle version="8.2.2">
 <drawing>
 <settings>
@@
 <part name="GND147" library="umich" deviceset="GND" device=""/>
 <part name="GND148" library="umich" deviceset="GND" device=""/>
+<part name="U$55" library="signpost" deviceset="VCC_BACKPLANE" device=""/>
 </parts>
 <sheets>
@@
 <wire x1="35.56" y1="73.66" x2="35.56" y2="63.5" width="0.1524" layer="98"/>
 <wire x1="35.56" y1="63.5" x2="63.5" y2="63.5" width="0.1524" layer="98"/>
-<text x="88.9" y="167.64" size="1.27" layer="98">Downstream ports draw
-VBUS from the "cable"</text>
+<text x="83.82" y="167.64" size="1.27" layer="98">This hub &amp; downstream ports
+are "externally" powered
+(not limited to 500mA from host)</text>
 <text x="48.26" y="119.38" size="1.27" layer="98">!EXTMEM -&gt; high, no mem
 !GANGED -&gt; high, OVR per port
@@
 <instance part="U$53" gate="G$1" x="17.78" y="124.46"/>
 <instance part="R52" gate="G$1" x="22.86" y="116.84" rot="R90"/>
+<instance part="U$55" gate="G$1" x="111.76" y="172.72"/>
 </instances>
 <busses>
@@
 <net name="GND" class="0">
 <segment>
-<pinref part="U1" gate="G$1" pin="!BUSPWR"/>
-<wire x1="106.68" y1="160.02" x2="109.22" y2="160.02" width="0.1524" layer="91"/>
-<wire x1="109.22" y1="160.02" x2="109.22" y2="172.72" width="0.1524" layer="91"/>
-<wire x1="109.22" y1="172.72" x2="104.14" y2="172.72" width="0.1524" layer="91"/>
-<label x="104.14" y="172.72" size="1.27" layer="95" rot="R180" xref="yes"/>
-</segment>
-<segment>
 <pinref part="U1" gate="G$1" pin="GND"/>
 <pinref part="GND15" gate="1" pin="GND"/>
@@
 <junction x="17.78" y="121.92"/>
 </segment>
+<segment>
+<pinref part="U1" gate="G$1" pin="!BUSPWR"/>
+<wire x1="106.68" y1="160.02" x2="111.76" y2="160.02" width="0.1524" layer="91"/>
+<wire x1="111.76" y1="160.02" x2="111.76" y2="172.72" width="0.1524" layer="91"/>
+<pinref part="U$55" gate="G$1" pin="VCC_BACKPLANE"/>
+</segment>
 </net>
