File: modules/microwave_radar/hardware/rev_b/microwave.sch (EAGLE design)
At the start: 59 parts, among them J1 MODULE_GENERIC_DEBUG, J2 TC2030-JLINK-L, Q1 SI223DDS, Q3 SI223DDS, U1 SAM4LC8AA, U3 MSGEQ7, U4 HB100, U5 OP284E_SEPARATE, U7 TLV62130

Commit message: renumbered resistors
Parts:
- removed R21: 240k, passives:RESISTOR0402_RES
- removed R23: 1k, passives:RESISTOR0402_RES
- removed R24: 100k, passives:RESISTOR0402_RES
- added R1: 1k, passives:RESISTOR0402_RES
- added R15: 200k, passives:RESISTOR0603_RES
- added R17: 330k, passives:RESISTOR0402_RES
- R11, R12: value 1M -> 100k
- R14: value 200k -> 100k; device passives:RESISTOR0603_RES -> passives:RESISTOR0402_RES; DIGIKEY RHM200KCFCT-ND -> (none)
- R16: value 330k -> 240k; DIGIKEY 1276-4244-1-ND -> P240KLCT-ND
- R18: value 100k -> 750k; DIGIKEY 1276-3432-1-ND -> P750KLCT-ND
- R19: value 1k -> 1M; DIGIKEY 1276-3430-1-ND -> 1276-3432-1-ND
- R20: value 750k -> 1M; DIGIKEY P750KLCT-ND -> 1276-3432-1-ND
- R3: value 8.2k -> 1k; DIGIKEY 311-8.20KLRCT-ND -> 1276-3430-1-ND
- R4: value 10k -> 8.2k; DIGIKEY 1276-3431-1-ND -> 311-8.20KLRCT-ND
- R6: value 12k -> 10k; DIGIKEY 1276-4122-1-ND -> 1276-3431-1-ND
- R7: value 100k -> 12k; DIGIKEY 1276-3432-1-ND -> 1276-4122-1-ND
- renumbered R22 to R13
Connections:
- net +3V3: now also R1.1, R14.2, R18.2, R6.2, R9.2; no longer R2.1, R20.2, R24.2, R5.2, R7.2
- net +5V: now also R12.2; no longer R18.2
- net 3V3_GATED: now also R11.2, R15.1; no longer R10.2, R14.1
- net AMP_OUT: now also R20.1; no longer R12.1
- net GND: now also R10.1, R16.1, R7.1; no longer R21.1, R6.1, R9.1
- net IF: now also R7.2; no longer R6.2
- net N$1: now also R10.2, R11.1, R17.2; no longer R10.1, R16.2, R9.2
- net N$12: now also R19.2, R5.1; no longer R11.2, R4.1
- net N$14: now also R6.1; no longer R5.1
- net N$15: now also R5.2; no longer R4.2
- net N$17: now also R19.1; no longer R11.1
- net N$18: now also R4.2; no longer R3.2
- net N$19: now also R20.2, R4.1; no longer R12.2, R3.1
- net N$2: now also R15.2; no longer R14.2
- net N$34: now also R1.2; no longer R2.2
- net N$37: now also R12.1, R2.2; no longer R18.1, R19.2
- net N$38: now also R3.2; no longer R23.2
- net N$44: now also R14.1; no longer R24.1
- net N$45: now also R16.2, R18.1; no longer R20.1, R21.2
- net N$9: now also R17.1; no longer R16.1
- net RADAR_POWER_GATE: now also R2.1, R3.1; no longer R19.1, R23.1
- net SWDCLK: now also R9.1; no longer R8.1
- net SWDIO: now also R8.1; no longer R7.1
Other:
- moved on the sheet: R10, R11, R12, R14, R19, R4, R8

Commit message: silk and renumbering
Parts:
- C15: value 6.8uF -> 100nF; device passives:CAPACITOR0603_CAP -> passives:CAPACITOR0402_CAP; DIGIKEY 445-7484-1-ND -> 490-10777-1-ND
- C17: value 100nF -> 4.7uF; DIGIKEY 490-10777-1-ND -> 1276-1481-1-ND
- C20: value 4.7uF -> 6.8uF; device passives:CAPACITOR0402_CAP -> passives:CAPACITOR0603_CAP; DIGIKEY 1276-1481-1-ND -> 445-7484-1-ND
- J1: value MODULE_GENERIC_DEBUG -> (none); device signpost:MODULE_GENERIC_DEBUG -> umich:JUMPER-2PTH
- J2: value TC2030-JLINK-L -> MODULE_GENERIC_DEBUG; device connector:TC2030-JLINK-L -> signpost:MODULE_GENERIC_DEBUG
- J3: value (none) -> TC2030-JLINK-L; device umich:JUMPER-2PTH -> connector:TC2030-JLINK-L
- renumbered C28 to C21, C29 to C8, C30 to C7, C31 to C22, JP2 to JP1, L5 to L1, LED2 to LED1, Q3 to Q2
Connections:
- net !RESET: now also J2.DBG_!RESET, J3.!RESET; no longer J1.DBG_!RESET, J2.!RESET
- net +3V3: now also J1.1, J2.VCCIO, J3.VCC; no longer J1.VCCIO, J2.VCC, J3.1
- net +5V: now also J2.5V; no longer J1.5V
- net ADVREFP: now also J1.2; no longer J3.2
- net DBG_GPIO1: now also J2.DBG_GPIO1; no longer J1.DBG_GPIO1
- net DBG_GPIO2: now also J2.DBG_GPIO2; no longer J1.DBG_GPIO2
- net DBG_RX: now also J2.DBG_RX; no longer J1.DBG_RX
- net DBG_TX: now also J2.DBG_TX; no longer J1.DBG_TX
- net GND: now also C18.1, C20.1, J3.GND; no longer C17.1, C19.1, J1.GND
- net I2C_CLK: now also J2.SCL; no longer J1.SCL
- net I2C_DATA: now also J2.SDA; no longer J1.SDA
- net IF: now also C17.1; no longer C18.1
- net MOD_IN: now also J2.MOD_IN; no longer J1.MOD_IN
- net MOD_OUT: now also J2.MOD_OUT; no longer J1.MOD_OUT
- net N$15: now also C18.2; no longer C19.2
- net N$17: now also C19.1; no longer C20.1
- net N$18: now also C19.2; no longer C20.2
- net N$28: now also J2.USB_VBUS; no longer J1.USB_VBUS
- net N$36: now also C20.2; no longer C16.2
- net N$5: now also C16.2; no longer C17.2
- net N$9: now also C17.2; no longer C18.2
- net PPS: now also J2.PPS; no longer J1.PPS
- net SWDCLK: now also J2.DBG_SWDCLK, J3.SWDCLK; no longer J1.DBG_SWDCLK, J2.SWDCLK
- net SWDIO: now also J2.DBG_SWDIO, J3.SWDIO; no longer J1.DBG_SWDIO, J2.SWDIO
- net USB+: now also J2.USB_D+; no longer J1.USB_D+
- net USB-: now also J2.USB_D-; no longer J1.USB_D-
Other:
- moved on the sheet: C15, C17, C18, C19

Commit message: fixed supply parts
Connections:
- net +3V3 renamed 3V3
- net +5V renamed 5V
Changed lines of the file:
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@@
 <part name="GND6" library="umich" deviceset="GND" device=""/>
 <part name="J2" library="signpost" deviceset="MODULE_GENERIC_DEBUG" device=""/>
-<part name="+3V2" library="supply1" deviceset="+3V3" device=""/>
-<part name="P+1" library="supply1" deviceset="+5V" device=""/>
-<part name="P+2" library="supply1" deviceset="+5V" device=""/>
-<part name="+3V4" library="supply1" deviceset="+3V3" device=""/>
-<part name="+3V5" library="supply1" deviceset="+3V3" device=""/>
-<part name="+3V6" library="supply1" deviceset="+3V3" device=""/>
-<part name="+3V7" library="supply1" deviceset="+3V3" device=""/>
-<part name="+3V8" library="supply1" deviceset="+3V3" device=""/>
-<part name="P+3" library="supply1" deviceset="+5V" device=""/>
 <part name="SUPPLY1" library="supply1" deviceset="GND" device=""/>
 <part name="J1" library="umich" deviceset="JUMPER-2" device="PTH"/>
-<part name="+3V9" library="supply1" deviceset="+3V3" device=""/>
 <part name="U3" library="chips" deviceset="MSGEQ7" device=""/>
 <part name="GND8" library="supply1" deviceset="GND" device=""/>
@@
 <part name="JP1" library="pinhead" deviceset="PINHD-1X8" device=""/>
 <part name="LED1" library="leds" deviceset="LED" device="0603"/>
-<part name="+3V13" library="supply1" deviceset="+3V3" device=""/>
 <part name="Q1" library="fets" deviceset="SI223DDS" device=""/>
 <part name="R12" library="passives" deviceset="RESISTOR" device="0402_RES" value="100k">
@@
 <attribute name="DIGIKEY" value="1276-3430-1-ND"/>
 </part>
-<part name="+3V14" library="supply1" deviceset="+3V3" device=""/>
 <part name="Q2" library="fets" deviceset="SI223DDS" device=""/>
 <part name="R13" library="passives" deviceset="RESISTOR" device="0402_RES" value="100k">
@@
 </instance>
 <instance part="J2" gate="G$1" x="22.86" y="142.24"/>
-<instance part="+3V4" gate="G$1" x="60.96" y="124.46"/>
-<instance part="+3V5" gate="G$1" x="160.02" y="60.96"/>
-<instance part="+3V6" gate="G$1" x="195.58" y="71.12"/>
-<instance part="+3V7" gate="G$1" x="203.2" y="139.7"/>
-<instance part="+3V8" gate="G$1" x="48.26" y="165.1"/>
-<instance part="P+3" gate="1" x="40.64" y="170.18"/>
 <instance part="SUPPLY1" gate="1" x="45.72" y="91.44"/>
 <instance part="J1" gate="A" x="81.28" y="162.56"/>
-<instance part="+3V9" gate="G$1" x="76.2" y="170.18"/>
 <instance part="R1" gate="G$1" x="198.12" y="109.22" rot="R270">
 <attribute name="DIGIKEY" x="198.12" y="109.22" size="1.778" layer="96" rot="R270" display="off"/>
 </instance>
 <instance part="LED1" gate="G$1" x="198.12" y="101.6" rot="R270"/>
-<instance part="+3V13" gate="G$1" x="198.12" y="119.38"/>
 </instances>
 <busses>
@@
 </segment>
 </net>
-<net name="+3V3" class="0">
+<net name="3V3" class="0">
 <segment>
 <pinref part="J2" gate="G$1" pin="VCCIO"/>
 <wire x1="33.02" y1="160.02" x2="48.26" y2="160.02" width="0.1524" layer="91"/>
-<pinref part="+3V8" gate="G$1" pin="+3V3"/>
 <wire x1="48.26" y1="160.02" x2="48.26" y2="162.56" width="0.1524" layer="91"/>
+<label x="48.26" y="162.56" size="1.016" layer="95" rot="R90" xref="yes"/>
 </segment>
 <segment>
@@
 <wire x1="81.28" y1="160.02" x2="81.28" y2="157.48" width="0.1524" layer="91"/>
 <wire x1="81.28" y1="157.48" x2="76.2" y2="157.48" width="0.1524" layer="91"/>
-<pinref part="+3V9" gate="G$1" pin="+3V3"/>
 <wire x1="76.2" y1="157.48" x2="76.2" y2="167.64" width="0.1524" layer="91"/>
+<label x="76.2" y="167.64" size="1.016" layer="95" rot="R90" xref="yes"/>
 </segment>
 <segment>
@@
 <wire x1="114.3" y1="116.84" x2="91.44" y2="116.84" width="0.1524" layer="91"/>
 <junction x="114.3" y="116.84"/>
-<pinref part="+3V4" gate="G$1" pin="+3V3"/>
 <wire x1="91.44" y1="116.84" x2="81.28" y2="116.84" width="0.1524" layer="91"/>
 <wire x1="81.28" y1="116.84" x2="73.66" y2="116.84" width="0.1524" layer="91"/>
@@
 <wire x1="91.44" y1="116.84" x2="91.44" y2="111.76" width="0.1524" layer="91"/>
 <junction x="91.44" y="116.84"/>
+<label x="60.96" y="121.92" size="1.016" layer="95" rot="R90" xref="yes"/>
 </segment>
 <segment>
 <pinref part="R6" gate="G$1" pin="2"/>
 <wire x1="200.66" y1="132.08" x2="203.2" y2="132.08" width="0.1524" layer="91"/>
-<pinref part="+3V7" gate="G$1" pin="+3V3"/>
 <wire x1="203.2" y1="132.08" x2="203.2" y2="137.16" width="0.1524" layer="91"/>
-</segment>
-<segment>
-<pinref part="+3V5" gate="G$1" pin="+3V3"/>
+<label x="203.2" y="137.16" size="1.016" layer="95" rot="R90" xref="yes"/>
+</segment>
+<segment>
 <wire x1="160.02" y1="58.42" x2="160.02" y2="45.72" width="0.1524" layer="91"/>
 <pinref part="J3" gate="G$1" pin="VCC"/>
 <wire x1="160.02" y1="45.72" x2="165.1" y2="45.72" width="0.1524" layer="91"/>
+<label x="160.02" y="58.42" size="1.016" layer="95" rot="R90" xref="yes"/>
 </segment>
 <segment>
 <pinref part="R8" gate="G$1" pin="2"/>
-<pinref part="+3V6" gate="G$1" pin="+3V3"/>
 <wire x1="195.58" y1="58.42" x2="195.58" y2="63.5" width="0.1524" layer="91"/>
 <wire x1="195.58" y1="63.5" x2="195.58" y2="68.58" width="0.1524" layer="91"/>
@@
 <pinref part="R9" gate="G$1" pin="2"/>
 <wire x1="203.2" y1="63.5" x2="203.2" y2="58.42" width="0.1524" layer="91"/>
+<label x="195.58" y="68.58" size="1.016" layer="95" rot="R90" xref="yes"/>
 </segment>
 <segment>
 <pinref part="R1" gate="G$1" pin="1"/>
-<pinref part="+3V13" gate="G$1" pin="+3V3"/>
 <wire x1="198.12" y1="116.84" x2="198.12" y2="114.3" width="0.1524" layer="91"/>
+<label x="198.12" y="116.84" size="1.016" layer="95" rot="R90" xref="yes"/>
 </segment>
 </net>
@@
 </segment>
 </net>
-<net name="+5V" class="0">
+<net name="5V" class="0">
 <segment>
 <pinref part="J2" gate="G$1" pin="5V"/>
 <wire x1="33.02" y1="162.56" x2="40.64" y2="162.56" width="0.1524" layer="91"/>
-<pinref part="P+3" gate="1" pin="+5V"/>
 <wire x1="40.64" y1="162.56" x2="40.64" y2="167.64" width="0.1524" layer="91"/>
+<label x="40.64" y="167.64" size="1.016" layer="95" rot="R90" xref="yes"/>
 </segment>
 </net>
@@
 </instance>
 <instance part="GND6" gate="1" x="106.68" y="86.36"/>
-<instance part="P+2" gate="1" x="185.42" y="142.24"/>
 <instance part="GND7" gate="1" x="60.96" y="91.44"/>
 <instance part="U4" gate="G1" x="109.22" y="114.3">
@@
 </segment>
 </net>
-<net name="+5V" class="0">
+<net name="5V" class="0">
 <segment>
 <pinref part="Q1" gate="G$1" pin="S"/>
-<pinref part="P+2" gate="1" pin="+5V"/>
 <wire x1="185.42" y1="129.54" x2="185.42" y2="137.16" width="0.1524" layer="91"/>
 <pinref part="R12" gate="G$1" pin="2"/>
@@
 <wire x1="175.26" y1="137.16" x2="185.42" y2="137.16" width="0.1524" layer="91"/>
 <junction x="185.42" y="137.16"/>
+<label x="185.42" y="139.7" size="1.016" layer="95" rot="R180" xref="yes"/>
 </segment>
 </net>
@@
 <instance part="FRAME4" gate="G$1" x="-20.32" y="-10.16"/>
 <instance part="FRAME4" gate="G$2" x="127" y="-10.16"/>
-<instance part="+3V2" gate="G$1" x="99.06" y="165.1"/>
-<instance part="P+1" gate="1" x="2.54" y="167.64"/>
 <instance part="U3" gate="G$1" x="96.52" y="66.04"/>
 <instance part="GND8" gate="1" x="93.98" y="25.4"/>
@@
 </instance>
 <instance part="JP1" gate="A" x="193.04" y="101.6"/>
-<instance part="+3V14" gate="G$1" x="165.1" y="165.1"/>
 <instance part="Q2" gate="G$1" x="165.1" y="152.4" rot="MR180"/>
 <instance part="R13" gate="G$1" x="152.4" y="157.48" rot="R90">
@@
 </busses>
 <nets>
-<net name="+5V" class="0">
+<net name="5V" class="0">
 <segment>
 <pinref part="JP1" gate="A" pin="1"/>
@@
 <wire x1="17.78" y1="142.24" x2="22.86" y2="142.24" width="0.1524" layer="91"/>
 <junction x="2.54" y="152.4"/>
-<pinref part="P+1" gate="1" pin="+5V"/>
 <wire x1="2.54" y1="152.4" x2="2.54" y2="165.1" width="0.1524" layer="91"/>
+<label x="2.54" y="165.1" size="1.016" layer="95" rot="R90" xref="yes"/>
 </segment>
 </net>
@@
 </segment>
 </net>
-<net name="+3V3" class="0">
+<net name="3V3" class="0">
 <segment>
 <pinref part="JP1" gate="A" pin="4"/>
@@
 <segment>
 <pinref part="Q2" gate="G$1" pin="S"/>
-<pinref part="+3V14" gate="G$1" pin="+3V3"/>
 <wire x1="165.1" y1="157.48" x2="165.1" y2="160.02" width="0.1524" layer="91"/>
 <pinref part="R13" gate="G$1" pin="2"/>
@@
 <wire x1="152.4" y1="160.02" x2="165.1" y2="160.02" width="0.1524" layer="91"/>
 <junction x="165.1" y="160.02"/>
+<label x="165.1" y="162.56" size="1.016" layer="95" rot="R90" xref="yes"/>
 </segment>
 <segment>
@@
 <junction x="86.36" y="152.4"/>
 <junction x="99.06" y="152.4"/>
-<pinref part="+3V2" gate="G$1" pin="+3V3"/>
 <wire x1="99.06" y1="152.4" x2="99.06" y2="162.56" width="0.1524" layer="91"/>
-</segment>
-</net>
+<label x="99.06" y="162.56" size="1.016" layer="95" rot="R90" xref="yes"/>
+</segment>
+</net>

Commit message: updated discontinued part
Parts:
- R15: DIGIKEY RHM200KCFCT-ND -> 311-200KGRCT-ND
Changed lines of the file:
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@@
 </part>
 <part name="R15" library="passives" deviceset="RESISTOR" device="0603_RES" value="200k">
-<attribute name="DIGIKEY" value="RHM200KCFCT-ND"/>
+<attribute name="DIGIKEY" value="311-200KGRCT-ND"/>
 </part>
 <part name="C16" library="passives" deviceset="CAPACITOR" device="0402_CAP" value="100nF">
