File: hardware/power_supply_module/rev_f/power_supply_module.sch (EAGLE design)
At the start: 172 parts, among them J1 MODULE_POWER, J3 TC2030-FTDI-I2C, Q1 MOSFET-NCHANNELSMD, U1 TLV62130, U10 LTC2943, U11 LTC2943, U12 LTC2943, U13 LTC2943, U14 LTC2943, U15 LTC2943, U16 LT3652, U17 LM234, U18 MAX17205, U19 ESDR0502N, U2 TLV62130, U20 AP22814, U21 AP22814, U22 AP22814, U23 AP22814, U24 AP22814, U25 PCA9544AQFN-N20, U26 LTC2943, U27 MAX6746, U28 3.3V, U29 M24C01WMN, U3 TLV62130, U30 SN74AUP1T14DCKR, U4 TLV62130, U5 TLV62130, U6 PCA9544AQFN-N20, U7 PCA9544AQFN-N20, U8 LTC2941, U9 LTC2943

Commit message: Ran the script, generate gerbers
Parts:
- added !RESET: TEST_POINT_0.040IN, headers:TEST_POINT_0.040IN
Connections:
- removed net ENABLE: U1.EN, U2.EN, U27.!RESET, U3.EN, U30.A, U4.EN, U5.EN
- new net !RESET: !RESET.TESTPOINT, U1.EN, U2.EN, U27.!RESET, U3.EN, U30.A, U4.EN, U5.EN
Changed lines of the file:
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@@
 </part>
 <part name="U$48" library="signpost" deviceset="VCC_BACKPLANE" device=""/>
+<part name="!RESET" library="headers" deviceset="TEST_POINT_0.040IN" device=""/>
 </parts>
 <sheets>
@@
 </segment>
 </net>
-<net name="ENABLE" class="0">
+<net name="!RESET" class="0">
 <segment>
 <pinref part="U5" gate="G$1" pin="EN"/>
@@
 </segment>
 </net>
-<net name="ENABLE" class="0">
-<segment>
-<wire x1="139.7" y1="50.8" x2="180.34" y2="50.8" width="0.1524" layer="91"/>
-<pinref part="U27" gate="G$1" pin="!RESET"/>
-<wire x1="180.34" y1="63.5" x2="180.34" y2="50.8" width="0.1524" layer="91"/>
-<wire x1="180.34" y1="63.5" x2="182.88" y2="63.5" width="0.1524" layer="91"/>
-<label x="182.88" y="63.5" size="1.27" layer="95" xref="yes"/>
-<pinref part="U30" gate="G$1" pin="A"/>
-<wire x1="200.66" y1="50.8" x2="180.34" y2="50.8" width="0.1524" layer="91"/>
-<junction x="180.34" y="50.8"/>
-</segment>
-</net>
 <net name="N$77" class="0">
 <segment>
@@
 </segment>
 </net>
+<net name="!RESET" class="0">
+<segment>
+<wire x1="139.7" y1="50.8" x2="180.34" y2="50.8" width="0.1524" layer="91"/>
+<pinref part="U27" gate="G$1" pin="!RESET"/>
+<wire x1="180.34" y1="63.5" x2="180.34" y2="50.8" width="0.1524" layer="91"/>
+<wire x1="180.34" y1="63.5" x2="182.88" y2="63.5" width="0.1524" layer="91"/>
+<label x="182.88" y="63.5" size="1.27" layer="95" xref="yes"/>
+<pinref part="U30" gate="G$1" pin="A"/>
+<wire x1="200.66" y1="50.8" x2="180.34" y2="50.8" width="0.1524" layer="91"/>
+<junction x="180.34" y="50.8"/>
+</segment>
+</net>
 </nets>
 </sheet>
@@
 <instance part="FAULT" gate="G$1" x="116.84" y="111.76"/>
 <instance part="CHRG" gate="G$1" x="116.84" y="109.22"/>
+<instance part="!RESET" gate="G$1" x="116.84" y="106.68"/>
 </instances>
 <busses>
@@
 </segment>
 </net>
+<net name="!RESET" class="0">
+<segment>
+<pinref part="!RESET" gate="G$1" pin="TESTPOINT"/>
+<wire x1="119.38" y1="106.68" x2="121.92" y2="106.68" width="0.1524" layer="91"/>
+<label x="121.92" y="106.68" size="1.27" layer="95" xref="yes"/>
+</segment>
+</net>

Commit message: Fix up component names
Change gnd symbol to SUPPLY, test points to TP, and switches to S. Works
better with eagle bom script
Parts:
- D2: value (none) -> DIODE_ZENERSOT323
- D3: value DIODE_SCHOTTKYSOD323 -> None
- renumbered !RESET to TP8, 3V3 to TP1, 5V_1 to TP2, 5V_2 to TP3, 5V_3 to TP4, 5V_4 to TP5, CHRG to TP7, FAULT to TP6, RESET to S2

Commit message: add manufacturer pns
Parts:
- C1, C10, C11, C12, C13, C14, C15, C16, C17, C18, C19, C2, C20, C21, C22, C23, C3, C4, C5, C6, C7, C8, C9: DESCRIPTION (none) -> CAP CER 0.1UF 25V X5R 0402; DIGIKEY 490-5920-1-ND -> 490-5920-1-ND; MANUFACTURER (none) -> Murata; MPN (none) -> GRM155R61E104KA87D
- C24, C25, C26: DESCRIPTION (none) -> CAP CER 0.47UF 6.3V X5R 0402; MANUFACTURER (none) -> Murata; MPN (none) -> GRM155R60J474KE19D
- C27: DESCRIPTION (none) -> CAP CER 0.82UF 6.3V X6S 0402; MANUFACTURER (none) -> Murata; MPN (none) -> GRM155C80J824KE15D
- C28: DESCRIPTION (none) -> CAP CER 1UF 10V X5R 0603; MANUFACTURER (none) -> Murata; MPN (none) -> GRM188R61A105KA61D
- C29, C30, C31, C32, C33: DESCRIPTION (none) -> CAP CER 3300PF 50V 10% X7R 0402; DIGIKEY 490-3248-1-ND -> 490-3248-1-ND; MANUFACTURER (none) -> Murata; MPN (none) -> GRM155R71H332KA01D
- C34, C35, C36, C37, C38, C39, C40: DESCRIPTION (none) -> CAP CER 10UF 25V 10% X5R 0805; DIGIKEY 490-5523-1-ND -> 490-5523-1-ND; MANUFACTURER (none) -> Murata; MPN (none) -> GRM21BR61E106KA73L
- C41, C42, C43, C44, C45, C46, C47, C48, C49, C50: DESCRIPTION (none) -> CAP CER 22UF 6.3V X5R 0603; DIGIKEY 1276-1193-1-ND -> 1276-1193-1-ND; MANUFACTURER (none) -> Samsung; MPN (none) -> CL10A226MQ8NRNC
- D1: DESCRIPTION (none) -> DIODE SCHOTTKY 40V 1.75A SOT23F; MANUFACTURER (none) -> Central Semiconductor; MPN (none) -> CMPSH1-4 TR
- D2: DESCRIPTION (none) -> DIODE ZENER 3.6V 400MW SOD323; MANUFACTURER (none) -> NXP Semiconductors; MPN (none) -> PDZ3.6B,115
- D3: value None -> DIODE_SCHOTTKYSOD323; DESCRIPTION (none) -> DIODE SCHOTTKY 40V 200MA SOD323; MANUFACTURER (none) -> Central Semiconductor; MPN (none) -> CMDSH2-4L TR
- H1, H2, H3, H4: device holes:MOUNT-PAD-ROUND3.0 -> holes:MOUNT-PAD-ROUND3
- L6: DESCRIPTION (none) -> FIXED IND 6.8UH 5.5A 46.8 MOHM; MANUFACTURER (none) -> Vishay Dale; MPN (none) -> IHLP2525CZER6R8M11
- Q1: DESCRIPTION (none) -> MOSFET N-CH 60V 0.115A SOT-23; MANUFACTURER (none) -> ON Semiconductor; MPN (none) -> 2N7002LT1G
- R1: DESCRIPTION (none) -> RES SMD 0.01 OHM 1% 1/2W 0805; MANUFACTURER (none) -> Vishay Dale; MPN (none) -> WSLP0805R0100FEB
- R10, R11: DESCRIPTION (none) -> RES SMD 0.05 OHM 1% 1/2W 0805; MANUFACTURER (none) -> Vishay Dale; MPN (none) -> WSLP0805R0500FEB
- R12, R13, R66: DESCRIPTION (none) -> RES SMD 1K OHM 5% 1/10W 0402; MANUFACTURER (none) -> Panasonic; MPN (none) -> ERJ-2GEJ102X
- R15, R16: DESCRIPTION (none) -> RES SMD 1M OHM 1% 1/10W 0402; MANUFACTURER (none) -> Panasonic; MPN (none) -> ERJ-2RKF1004X
- R17, R18, R19, R20, R21, R22, R23, R24, R25, R26, R27, R28, R29, R30, R31, R32, R33, R34, R35, R36, R37, R38, R39, R40, R41, R42, R43: DESCRIPTION (none) -> RES SMD 2K OHM 1% 1/10W 0402; MANUFACTURER (none) -> Panasonic; MPN (none) -> ERJ-2RKF2001X
- R2, R3, R4, R5, R6, R7, R8, R9: DESCRIPTION (none) -> RES SMD 0.017 OHM 1% 1/2W 0805; MANUFACTURER (none) -> Vishay Dale; MPN (none) -> WSLP0805R0170FEB
- R44: DESCRIPTION (none) -> RES SMD 23.2K OHM 0.1% 1/8W 0805; MANUFACTURER (none) -> Panasonic; MPN (none) -> ERA6AEB2322V
- R45, R46, R47, R48, R49: DESCRIPTION (none) -> RES SMD 100K OHM 5% 1/10W 0402; DIGIKEY P100KJCT-ND -> P100KJCT-ND; MANUFACTURER (none) -> Panasonic; MPN (none) -> ERJ-2GEJ104X
- R50, R51, R52, R53: DESCRIPTION (none) -> RES SMD 130K OHM 1% 1/10W 0402; DIGIKEY P130KLCT-ND -> P130KLCT-ND; MANUFACTURER (none) -> Panasonic; MPN (none) -> ERJ-2RKF1303X
- R54, R55, R70: DESCRIPTION (none) -> RES SMD 150 OHM 1% 1/10W 0402; MANUFACTURER (none) -> Panasonic; MPN (none) -> ERJ-2RKF1500X
- R56: DESCRIPTION (none) -> RES SMD 240K OHM 1% 1/10W 0402; MANUFACTURER (none) -> Panasonic; MPN (none) -> ERJ-2RKF2403X
- R57: DESCRIPTION (none) -> RES SMD 301K OHM 0.1% 1/8W 0805; MANUFACTURER (none) -> Panasonic; MPN (none) -> ERA-6AEB3013V
- R58: DESCRIPTION (none) -> RES SMD 340K OHM 0.1% 1/8W 0805; MANUFACTURER (none) -> Panasonic; MPN (none) -> ERA-6AEB3403V
- R59, R60, R61, R62: DESCRIPTION (none) -> RES SMD 680K OHM 1% 1/10W 0402; DIGIKEY P680KLCT-ND -> P680KLCT-ND; MANUFACTURER (none) -> Panasonic; MPN (none) -> ERJ-2RKF6803X
- R63: DESCRIPTION (none) -> RES SMD 750K OHM 5% 1/10W 0402; MANUFACTURER (none) -> Panasonic; MPN (none) -> ERJ-2GEJ754X
- R64: DESCRIPTION (none) -> RES SMD 953K OHM 0.1% 1/8W 0805; MANUFACTURER (none) -> Panasonic; MPN (none) -> ERA-6AEB9533V
- U28: DESCRIPTION (none) -> IC REG LDO 3.3V 50MA SOT23-3; MANUFACTURER (none) -> Diodes Inc.; MPN (none) -> ZMR330FTA
