File: hardware/controller/rev_d/controller.sch (EAGLE design)
At the start: 107 parts, among them J1 DM3AT-SF-PEJM5, J10 SOLDERJUMPERTRACE, J11 SOLDERJUMPERTRACE, J12 SOLDERJUMPERTRACE, J14 TC2030-JLINK-L, J15 TC2030-JLINK-L, J16 U.FL-R-SMT, J2 MICRO_USB_B_HIROSE_ZX62R-B-5P, J3 MICRO_USB_B_HIROSE_ZX62R-B-5P, J4 MODULE_CONTROLLER, J9 SOLDERJUMPERTRACE, Q1 DMN32D2LDF, SW1 B3U-1000P, SW2 B3U-1000P, SW3 B3U-1000P, SW4 B3U-1000P, SW5 SIP3240X, SW6 SIP3240X, SW7 SIP3240X, U1 FM25CLXXB-DG, U10 TXS0108EVQFN20, U2 FTDI234XD, U3 NCP301LSN30, U4 NCP301LSN30, U5 RXM-GPS-RM-T, U6 SAM4LC8BA, U7 SAM4LC8BA, U8 SN74LVC1G125DBVR, U9 TS3USB30E, X1 16MHz, X2 16MHz

Commit message: Rev D of the controller
 * Connected PPS to Storage Master
 * Output enable pulldown on logic level converter
 * Moved caps to VDDCORE, not VDDOUT (both SAM4Ls)
 * Added debug pins for Storage Master MOD IN/OUT
 * Connected ADVREFP to VDDANA (both SAM4Ls)
Parts:
- added J17: (no value), pinhead:PINHD-1X2
Connections:
- net MODSTORAGE_IN: now also J17.1
- net MODSTORAGE_OUT: now also J17.2
- net N$29: now also U6.ADVREFP
- net N$32: now also U7.ADVREFP
- net N$44: no longer C17.1, C26.1
- net N$45: no longer C12.1, C25.1
- net N$46: now also C12.1, C25.1
- net N$59: now also C17.1, C26.1
Other:
- moved on the sheet: C12, C17, C25, C26

Commit message: Changed isolator voltage source
Left side of the isolator is now connected to VCC_CONTROLLER, which is
the source of _almost_ all of its I/O lines. The except is the indicator
LED, which is powered from VCC_LINUX_3V3. In that case though, there's a
diode preventing current from flowing from Controller to Linux domain if
Linux is disabled.
Connections:
- net VCC_CONTROLLER: now also C21.2, U10.VCCB
- net VCC_LINUX_3V3: no longer C21.2, U10.VCCB
Changed lines of the file:
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@@
 <part name="U$14" library="signpost" deviceset="VCC_LINUX_1V8" device=""/>
 <part name="GND22" library="umich" deviceset="GND" device=""/>
-<part name="U$15" library="signpost" deviceset="VCC_LINUX_3V3" device=""/>
 <part name="GND23" library="umich" deviceset="GND" device=""/>
 <part name="J14" library="connector" deviceset="TC2030-JLINK" device="-L"/>
@@
 <part name="GND42" library="umich" deviceset="GND" device=""/>
 <part name="J17" library="pinhead" library_urn="urn:adsk.eagle:library:325" deviceset="PINHD-1X2" device=""/>
+<part name="U$32" library="signpost" deviceset="VCC_CONTROLLER" device=""/>
 </parts>
 <sheets>
@@
 <instance part="U$14" gate="G$1" x="93.98" y="111.76"/>
 <instance part="GND22" gate="1" x="58.42" y="55.88" rot="MR0"/>
-<instance part="U$15" gate="G$1" x="58.42" y="111.76"/>
 <instance part="GND23" gate="1" x="30.48" y="35.56" rot="MR0"/>
 <instance part="VR1" gate="G$1" x="111.76" y="144.78"/>
@@
 </instance>
 <instance part="GND42" gate="1" x="93.98" y="55.88" rot="MR0"/>
+<instance part="U$32" gate="G$1" x="58.42" y="111.76"/>
 </instances>
 <busses>
@@
 <pinref part="U$13" gate="G$1" pin="VCC_LINUX_3V3"/>
 <wire x1="10.16" y1="53.34" x2="10.16" y2="55.88" width="0.1524" layer="91"/>
-</segment>
-<segment>
-<pinref part="U10" gate="G$1" pin="VCCB"/>
-<pinref part="U$15" gate="G$1" pin="VCC_LINUX_3V3"/>
-<wire x1="60.96" y1="91.44" x2="58.42" y2="91.44" width="0.1524" layer="91"/>
-<wire x1="58.42" y1="91.44" x2="58.42" y2="109.22" width="0.1524" layer="91"/>
-<wire x1="58.42" y1="109.22" x2="58.42" y2="111.76" width="0.1524" layer="91"/>
-<pinref part="C21" gate="G$1" pin="2"/>
-<wire x1="53.34" y1="106.68" x2="53.34" y2="109.22" width="0.1524" layer="91"/>
-<wire x1="53.34" y1="109.22" x2="58.42" y2="109.22" width="0.1524" layer="91"/>
-<junction x="58.42" y="109.22"/>
 </segment>
 <segment>
@@
 </segment>
 </net>
+<net name="VCC_CONTROLLER" class="0">
+<segment>
+<pinref part="U10" gate="G$1" pin="VCCB"/>
+<wire x1="60.96" y1="91.44" x2="58.42" y2="91.44" width="0.1524" layer="91"/>
+<wire x1="58.42" y1="91.44" x2="58.42" y2="109.22" width="0.1524" layer="91"/>
+<pinref part="C21" gate="G$1" pin="2"/>
+<wire x1="53.34" y1="106.68" x2="53.34" y2="109.22" width="0.1524" layer="91"/>
+<wire x1="53.34" y1="109.22" x2="58.42" y2="109.22" width="0.1524" layer="91"/>
+<pinref part="U$32" gate="G$1" pin="VCC_CONTROLLER"/>
+<wire x1="58.42" y1="109.22" x2="58.42" y2="111.76" width="0.1524" layer="91"/>
+<junction x="58.42" y="109.22"/>
+</segment>
+</net>
