File: modules/microwave_radar/hardware/rev_b/macrofab_compliant/microwave.brd (EAGLE design)
At the start: 68.1 x 66 mm, 63 parts, among them J3 TC2030-JLINK-L, J6 SIGNPOST_MODULE_HEADER, J7 SIGNPOST_DEBUG_HEADER, Q1 SI223DDS, Q2 SI223DDS, U1 SAM4LC8AA, U3 MSGEQ7, U4 HB100, U5 OP284E_SEPARATE, U7 TLV62130, X1 FH1600015

Commit message: updated files for macrofab
Parts:
- removed J1: (no value), umich:1X02
- removed Q1, Q2: SI223DDS, fets:SOT23-3
- removed R20, R21: 1M, passives:0402_RES
- added C24: 22uF, passives:0603_CAP
- added C25: 100uF, passives:1210_CAP
- added S1, S2: SIP3240X, signpost:TDFN4
- C20: value 6.8uF -> 4.7uF; device passives:0603_CAP -> passives:0402_CAP
- C21: value 10uF -> 4.7uF; device passives:0805_CAP -> passives:0402_CAP
- C22: value 22uF -> 6.8uF
- C23: value 100uF -> 10uF; device passives:1210_CAP -> passives:0805_CAP
- R1: value 0 -> DNP - 0
- R14: value 100k -> 200k; device passives:0402_RES -> passives:0603-RES
- R15: value 100k -> 240k
- R16: value 200k -> 330k; device passives:0603-RES -> passives:0402_RES
- R17: value 240k -> 750k
- R18: value 330k -> 1M
- R19: value 750k -> 1M
- R3: value 1k -> 8.2k
- R4: value 1k -> 10k
- R5: value 8.2k -> 10k
- R6: value 10k -> 12k
- R7: value 10k -> 100k
- R8: value 12k -> 100k
- moved R11 45.8 mm to (62.5, 29.2)
- moved R12 37.5 mm to (61.0, 29.2), turned to 270 degrees
- moved R19 37.2 mm to (33.0, 14.0), turned to 180 degrees
- moved R15 34.5 mm to (34.3, 51.1)
- moved R16 33.3 mm to (25.4, 22.9), turned to 90 degrees
- moved R3 32.2 mm to (27.4, 21.3), turned to 180 degrees
- moved R10 27.9 mm to (35.6, 49.7), turned to 0 degrees
- moved C20 24.4 mm to (23.6, 54.1), turned to 180 degrees
- moved C23 20.9 mm to (29.2, 46.2), turned to 90 degrees
- moved R14 18.2 mm to (56.9, 11.9), turned to 0 degrees
- moved R4 16.0 mm to (24.1, 15.2)
- moved C21 15.9 mm to (21.7, 32.3), turned to 270 degrees
- moved R13 14.3 mm to (23.4, 57.1)
- moved R5 14.0 mm to (31.2, 34.8)
- moved R8 13.7 mm to (27.9, 22.9)
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Connections:
- removed net ADVREFP: J1.2, U1.18
- removed net N$21: U1.16
- removed net N$26: U1.32
- removed net N$27: U1.35
- removed net N$28: J6.13
- removed net N$29: U1.37
- removed net N$32: U1.41
- removed net N$33: U1.42
- removed net N$37: Q1.1, R11.1, R3.2
- removed net N$38: Q2.1, R12.1, R4.2
- removed net N$5: C16.2, Q1.3, U4.5V_1, U4.5V_2
- new net 5V_GATED: C16.2, S1.1, U4.5V_1, U4.5V_2
- net 3V3: now also C21.1, C24.2, R10.2, R11.2, R17.2, R5.2, S2.3; no longer C22.2, J1.1, Q2.2, R13.2, R14.2, R15.2, R19.2, R7.2
- net 3V3_GATED: now also C10.2, R14.1, R8.2, S2.1; no longer C9.2, Q2.3, R10.2, R16.1
- net 5V: now also C20.1, C23.P$1, S1.3; no longer C21.P$1, Q1.2
- net AMP_OUT: now also R19.1; no longer R21.1
- net GND: now also C10.1, C20.2, C21.2, C23.P$2, C24.1, C25.1, C9.2, R13.1, R15.1, R6.1, R7.1, S1.2, S1.PAD, S2.2, S2.PAD; no longer C10.2, C20.1, C21.P$2, C23.1, C9.1, R11.2, R17.1, R8.1
- net IF: now also R6.2; no longer R8.2
- net N$1: now also C25.2, R16.2, R7.2, R8.1; no longer C23.2, R10.1, R18.2, R9.2
- net N$12: now also R18.2, R4.1; no longer R20.2, R6.1
- net N$14: now also R5.1; no longer R7.1
- net N$15: now also R4.2; no longer R6.2
- net N$17: now also R18.1; no longer R20.1
- net N$18: now also R3.2; no longer R5.2
- net N$19: now also R19.2, R3.1; no longer R21.2, R5.1
- net N$2: now also R14.2; no longer R16.2
- net N$36: now also C22.2; no longer C20.2
- net N$44: now also R10.1; no longer R13.1
- net N$45: now also R15.2, R17.1; no longer R17.2, R19.1
- net N$7: now also C9.1; no longer C10.1
- net N$9: now also R16.1; no longer R18.1
- net RADAR_POWER_GATE: now also R13.2, R9.2, S1.4, S2.4; no longer R3.1, R4.1
- net SWDCLK: now also R12.1; no longer R15.1
- net SWDIO: now also R11.1; no longer R14.1
Routing:
- net ADVREFP: track 27.9 -> 0.00 mm, vias 1 -> 0
- net N$5: track 12.8 -> 0.00 mm
- net 3V3: track 214.0 -> 201.7 mm
- net RADAR_POWER_GATE: track 45.7 -> 56.3 mm, vias 5 -> 6
- net 5V_GATED: track 0.00 -> 8.78 mm
- net 5V: track 63.1 -> 68.7 mm
- net N$38: track 3.05 -> 0.00 mm
- net N$37: track 2.90 -> 0.00 mm
- net GND: track 17.1 -> 18.7 mm
- net 3V3_GATED: track 55.6 -> 57.2 mm
- added copper zone on layer 1, net 3V3_GATED
- added copper zone on layer 1, net 5V_GATED
Other:
- board text removed: "AREF=3V3"
