File: modules/microwave_radar/hardware/rev_b/macrofab_compliant/microwave.sch (EAGLE design)
At the start: 61 parts, among them J3 TC2030-JLINK-L, J6 SIGNPOST_MODULE_HEADER, J7 SIGNPOST_DEBUG_HEADER, Q1 SI223DDS, Q2 SI223DDS, U1 SAM4LC8AA, U3 MSGEQ7, U4 HB100, U5 OP284E_SEPARATE, U7 TLV62130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

Commit message: updated files for macrofab
Parts:
- removed J1: (no value), umich:JUMPER-2PTH
- removed Q1, Q2: SI223DDS, fets:SI223DDS
- removed R20, R21: 1M, passives:RESISTOR0402_RES
- added C24: 22uF, passives:CAPACITOR0603_CAP
- added C25: 100uF, passives:CAPACITOR1210_CAP
- added S1, S2: SIP3240X, signpost:SIP3240X
- C20: value 6.8uF -> 4.7uF; device passives:CAPACITOR0603_CAP -> passives:CAPACITOR0402_CAP; DESCRIPTION CAP CER 6.8UF 10V X5R 0603 -> CAP CER 4.7UF 6.3V X5R 0402; DIGIKEY 445-7484-1-ND -> 1276-1481-1-ND; MANUFACTURER TDK -> Samsung; MPN C1608X5R1A685K080AC -> CL05A475KQ5NRNC
- C21: value 10uF -> 4.7uF; device passives:CAPACITOR0805_CAP -> passives:CAPACITOR0402_CAP; DESCRIPTION CAP CER 10UF 10V X5R 0805 -> CAP CER 4.7UF 6.3V X5R 0402; DIGIKEY 399-4925-1-ND -> 1276-1481-1-ND; MANUFACTURER KEMET -> Samsung; MPN C0805C106K8PACTU -> CL05A475KQ5NRNC
- C22: value 22uF -> 6.8uF; DESCRIPTION CAP CER 22UF 6.3V X5R 0603 -> CAP CER 6.8UF 10V X5R 0603; DIGIKEY 311-1815-1-ND -> 445-7484-1-ND; MANUFACTURER Yageo -> TDK; MPN CC0603MRX5R5BB226 -> C1608X5R1A685K080AC
- C23: value 100uF -> 10uF; device passives:CAPACITOR1210_CAP -> passives:CAPACITOR0805_CAP; DESCRIPTION CAP CER 100UF 6.3V 20% X5R 1210 -> CAP CER 10UF 10V X5R 0805; DIGIKEY 490-3390-1-ND -> 399-4925-1-ND; MANUFACTURER Murata -> KEMET; MPN GRM32ER60J107ME20L -> C0805C106K8PACTU
- R1: value 0 -> DNP - 0
- R14: value 100k -> 200k; device passives:RESISTOR0402_RES -> passives:RESISTOR0603_RES; DESCRIPTION RES SMD 100K OHM 1% 1/16W 0402 -> RES SMD 200K OHM 5% 1/10W 0603; DIGIKEY 1276-3432-1-ND -> 311-200KGRCT-ND; MANUFACTURER Samsung -> Yageo; MPN RC1005F104CS -> RC0603JR-07200KL
- R15: value 100k -> 240k; DESCRIPTION RES SMD 100K OHM 1% 1/16W 0402 -> RES SMD 240K OHM 1% 1/10W 0402; DIGIKEY 1276-3432-1-ND -> P240KLCT-ND; MANUFACTURER Samsung -> Panasonic; MPN RC1005F104CS -> ERJ-2RKF2403X
- R16: value 200k -> 330k; device passives:RESISTOR0603_RES -> passives:RESISTOR0402_RES; DESCRIPTION RES SMD 200K OHM 5% 1/10W 0603 -> RES SMD 330K OHM 1% 1/16W 0402; DIGIKEY 311-200KGRCT-ND -> 1276-4244-1-ND; MANUFACTURER Yageo -> Samsung; MPN RC0603JR-07200KL -> RC1005F334CS
- R17: value 240k -> 750k; DESCRIPTION RES SMD 240K OHM 1% 1/10W 0402 -> RES SMD 750K OHM 1% 1/10W 0402; DIGIKEY P240KLCT-ND -> P750KLCT-ND; MPN ERJ-2RKF2403X -> ERJ-2RKF7503X
- R18: value 330k -> 1M; DESCRIPTION RES SMD 330K OHM 1% 1/16W 0402 -> RES SMD 100K OHM 1% 1/16W 0402; DIGIKEY 1276-4244-1-ND -> 1276-3432-1-ND; MPN RC1005F334CS -> RC1005F104CS
- R19: value 750k -> 1M; DESCRIPTION RES SMD 750K OHM 1% 1/10W 0402 -> RES SMD 100K OHM 1% 1/16W 0402; DIGIKEY P750KLCT-ND -> 1276-3432-1-ND; MANUFACTURER Panasonic -> Samsung; MPN ERJ-2RKF7503X -> RC1005F104CS
- R3: value 1k -> 8.2k; DESCRIPTION RES SMD 1K OHM 1% 1/16W 0402 -> RES SMD 8.2K OHM 1% 1/16W 0402; DIGIKEY 1276-3430-1-ND -> 311-8.20KLRCT-ND; MANUFACTURER Samsung -> Yageo; MPN RC1005F102CS -> RC0402FR-078K2L
- R4: value 1k -> 10k; DESCRIPTION RES SMD 1K OHM 1% 1/16W 0402 -> RES SMD 10K OHM 1% 1/16W 0402; DIGIKEY 1276-3430-1-ND -> 1276-3431-1-ND; MPN RC1005F102CS -> RC1005F103CS
- R5: value 8.2k -> 10k; DESCRIPTION RES SMD 8.2K OHM 1% 1/16W 0402 -> RES SMD 10K OHM 1% 1/16W 0402; DIGIKEY 311-8.20KLRCT-ND -> 1276-3431-1-ND; MANUFACTURER Yageo -> Samsung; MPN RC0402FR-078K2L -> RC1005F103CS
- R6: value 10k -> 12k; DESCRIPTION RES SMD 10K OHM 1% 1/16W 0402 -> RES SMD 12K OHM 1% 1/16W 0402; DIGIKEY 1276-3431-1-ND -> 1276-4122-1-ND; MPN RC1005F103CS -> RC1005F123CS
- R7: value 10k -> 100k; DESCRIPTION RES SMD 10K OHM 1% 1/16W 0402 -> RES SMD 100K OHM 1% 1/16W 0402; DIGIKEY 1276-3431-1-ND -> 1276-3432-1-ND; MPN RC1005F103CS -> RC1005F104CS
- R8: value 12k -> 100k; DESCRIPTION RES SMD 12K OHM 1% 1/16W 0402 -> RES SMD 100K OHM 1% 1/16W 0402; DIGIKEY 1276-4122-1-ND -> 1276-3432-1-ND; MPN RC1005F123CS -> RC1005F104CS
Connections:
- removed net ADVREFP: J1.2, U1.ADVREFP
- removed net N$21: U1.PA07
- removed net N$26: U1.PA13
- removed net N$27: U1.PA16
- removed net N$28: J6.USB_VBUS
- removed net N$29: U1.PA18
- removed net N$32: U1.PA21
- removed net N$33: U1.PA22
- removed net N$37: Q1.G, R11.1, R3.2
- removed net N$38: Q2.G, R12.1, R4.2
- removed net N$5: C16.2, Q1.D, U4.5V_1, U4.5V_2
- new net 5V_GATED: C16.2, S1.VLOAD, U4.5V_1, U4.5V_2
- net 3V3: now also C21.1, C24.2, R10.2, R11.2, R17.2, R5.2, S2.VSUPP; no longer C22.2, J1.1, Q2.S, R13.2, R14.2, R15.2, R19.2, R7.2
- net 3V3_GATED: now also C10.2, R14.1, R8.2, S2.VLOAD; no longer C9.2, Q2.D, R10.2, R16.1
- net 5V: now also C20.1, C23.1, S1.VSUPP; no longer C21.1, Q1.S
- net AMP_OUT: now also R19.1; no longer R21.1
- net GND: now also C10.1, C20.2, C23.2, C24.1, C25.1, C9.2, R13.1, R15.1, R6.1, R7.1, S1.GND, S2.GND; no longer C10.2, C20.1, C23.1, C9.1, R11.2, R17.1, R8.1
- net IF: now also R6.2; no longer R8.2
- net N$1: now also C25.2, R16.2, R7.2, R8.1; no longer C23.2, R10.1, R18.2, R9.2
- net N$12: now also R18.2, R4.1; no longer R20.2, R6.1
- net N$14: now also R5.1; no longer R7.1
- net N$15: now also R4.2; no longer R6.2
- net N$17: now also R18.1; no longer R20.1
- net N$18: now also R3.2; no longer R5.2
- net N$19: now also R19.2, R3.1; no longer R21.2, R5.1
- net N$2: now also R14.2; no longer R16.2
- net N$36: now also C22.2; no longer C20.2
- net N$44: now also R10.1; no longer R13.1
- net N$45: now also R15.2, R17.1; no longer R17.2, R19.1
- net N$7: now also C9.1; no longer C10.1
- net N$9: now also R16.1; no longer R18.1
- net RADAR_POWER_GATE: now also R13.2, R9.2, S1.EN, S2.EN; no longer R3.1, R4.1
- net SWDCLK: now also R12.1; no longer R15.1
- net SWDIO: now also R11.1; no longer R14.1
Other:
- moved on the sheet: C10, C21, C9, R17, R18, R3, R6, R8
