File: modules/audio_spectrum/rev_e/audio_spectrum.brd (EAGLE design)
At the start: 68.1 x 66 mm, 112 parts, among them J1 AUDIO-JACK-VERTICAL, J2 SIGNPOST_DEBUG_HEADER, J3 SIGNPOST_MODULE_HEADER, J4 TC2030-JLINK-L, P1 4k-200k, P2 4k-200k, Q1 NX3008PBK, Q2 NX3008PBK, U1 AT45DB641EUDFN, U10 TLV62130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

Commit message: changed data, added advref
Connections:
- net N$32: now also U9.24
Routing:
- net N$32: track 5.24 -> 6.60 mm
Other:
- board text added: "9/2017"
- board text removed: "7/2017"
Changed lines of the file:
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@@
 <setting verticaltext="up"/>
 </settings>
-<grid distance="100" unitdist="mil" unit="mil" style="lines" multiple="1" display="yes" altdistance="10" altunitdist="mil" altunit="mil"/>
+<grid distance="5" unitdist="mil" unit="mil" style="lines" multiple="1" display="yes" altdistance="10" altunitdist="mil" altunit="mil"/>
 <layers>
-<layer number="1" name="Top" color="4" fill="1" visible="no" active="yes"/>
-<layer number="2" name="Route2" color="1" fill="3" visible="no" active="yes"/>
+<layer number="1" name="Top" color="4" fill="1" visible="yes" active="yes"/>
+<layer number="2" name="Route2" color="1" fill="3" visible="yes" active="yes"/>
 <layer number="3" name="Route3" color="4" fill="3" visible="no" active="no"/>
 <layer number="4" name="Route4" color="1" fill="4" visible="no" active="no"/>
@@
 <layer number="13" name="Route13" color="4" fill="5" visible="no" active="no"/>
 <layer number="14" name="Route14" color="1" fill="6" visible="no" active="no"/>
-<layer number="15" name="Route15" color="4" fill="6" visible="no" active="yes"/>
-<layer number="16" name="Bottom" color="1" fill="1" visible="no" active="yes"/>
-<layer number="17" name="Pads" color="2" fill="1" visible="no" active="yes"/>
-<layer number="18" name="Vias" color="2" fill="1" visible="no" active="yes"/>
-<layer number="19" name="Unrouted" color="6" fill="1" visible="no" active="yes"/>
-<layer number="20" name="Dimension" color="15" fill="1" visible="no" active="yes"/>
+<layer number="15" name="Route15" color="4" fill="6" visible="yes" active="yes"/>
+<layer number="16" name="Bottom" color="1" fill="1" visible="yes" active="yes"/>
+<layer number="17" name="Pads" color="2" fill="1" visible="yes" active="yes"/>
+<layer number="18" name="Vias" color="2" fill="1" visible="yes" active="yes"/>
+<layer number="19" name="Unrouted" color="6" fill="1" visible="yes" active="yes"/>
+<layer number="20" name="Dimension" color="15" fill="1" visible="yes" active="yes"/>
 <layer number="21" name="tPlace" color="7" fill="1" visible="yes" active="yes"/>
 <layer number="22" name="bPlace" color="7" fill="1" visible="yes" active="yes"/>
-<layer number="23" name="tOrigins" color="15" fill="1" visible="no" active="yes"/>
-<layer number="24" name="bOrigins" color="15" fill="1" visible="no" active="yes"/>
+<layer number="23" name="tOrigins" color="15" fill="1" visible="yes" active="yes"/>
+<layer number="24" name="bOrigins" color="15" fill="1" visible="yes" active="yes"/>
 <layer number="25" name="tNames" color="7" fill="1" visible="yes" active="yes"/>
 <layer number="26" name="bNames" color="7" fill="1" visible="yes" active="yes"/>
@@
 <text x="50.9016" y="42.7736" size="0.762" layer="25" font="vector" ratio="12" align="bottom-center">Samuel Rohrer
 Joshua Adkins</text>
-<text x="49.7078" y="45.0088" size="0.889" layer="25" font="vector" ratio="12" align="bottom-center">7/2017</text>
+<text x="49.7078" y="45.0088" size="0.889" layer="25" font="vector" ratio="12" align="bottom-center">9/2017</text>
 <text x="32.4358" y="41.8592" size="0.889" layer="21" font="vector" ratio="12" align="bottom-center">RESET</text>
 <text x="32.4358" y="39.0906" size="0.889" layer="21" font="vector" ratio="12" align="bottom-center">POWER</text>
@@
 <attribute name="DIGIKEY" value="RHM1.5KCGCT-ND" x="18.3388" y="10.4648" size="1.778" layer="27" rot="R270" display="off"/>
 <attribute name="MANUFACTURER" value="Rohm" x="18.3388" y="10.4648" size="1.778" layer="27" rot="R270" display="off"/>
-<attribute name="MPN" value="MCR03ERTJ152
-" x="18.3388" y="10.4648" size="1.778" layer="27" rot="R270" display="off"/>
+<attribute name="MPN" value="MCR03ERTJ152 " x="18.3388" y="10.4648" size="1.778" layer="27" rot="R270" display="off"/>
 <attribute name="NAME" x="17.5514" y="11.557" size="0.889" layer="25" font="vector" ratio="12" align="bottom-center"/>
 </element>
@@
 <attribute name="DIGIKEY" value="RHM1.5KCGCT-ND" x="27.0256" y="54.5592" size="1.778" layer="27" rot="R270" display="off"/>
 <attribute name="MANUFACTURER" value="Rohm" x="27.0256" y="54.5592" size="1.778" layer="27" rot="R270" display="off"/>
-<attribute name="MPN" value="MCR03ERTJ152
-" x="27.0256" y="54.5592" size="1.778" layer="27" rot="R270" display="off"/>
+<attribute name="MPN" value="MCR03ERTJ152 " x="27.0256" y="54.5592" size="1.778" layer="27" rot="R270" display="off"/>
 <attribute name="NAME" x="27.0764" y="52.578" size="0.889" layer="25" font="vector" ratio="12" align="bottom-center"/>
 </element>
@@
 <contactref element="FB1" pad="1"/>
 <contactref element="U9" pad="25"/>
-<wire x1="53.3868" y1="24.6088" x2="53.3868" y2="23.0742" width="0.254" layer="1"/>
+<wire x1="53.3868" y1="23.456809375" x2="53.3868" y2="24.6088" width="0.254" layer="1"/>
+<wire x1="53.3868" y1="23.456809375" x2="53.3868" y2="23.0742" width="0.254" layer="1"/>
 <wire x1="53.3868" y1="23.0742" x2="52.8828" y2="22.5702" width="0.254" layer="1"/>
 <wire x1="50.4952" y1="21.10866875" x2="51.95673125" y2="22.5702" width="0.254" layer="1"/>
 <wire x1="51.95673125" y1="22.5702" x2="52.8828" y2="22.5702" width="0.254" layer="1"/>
+<contactref element="U9" pad="24"/>
+<wire x1="52.8868" y1="24.6088" x2="52.8868" y2="23.956809375" width="0.254" layer="1"/>
+<wire x1="52.8868" y1="23.956809375" x2="53.3868" y2="23.456809375" width="0.254" layer="1"/>
 </signal>
 <signal name="N$44">

Commit message: added final audio files
Parts:
- R1: value 0 -> DNP - 0
Routing:
- removed copper zone on layer 15, net 3V3
- removed copper zone on layer 2, net GND
Changed lines of the file:
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@@
 <setting verticaltext="up"/>
 </settings>
-<grid distance="5" unitdist="mil" unit="mil" style="lines" multiple="1" display="yes" altdistance="10" altunitdist="mil" altunit="mil"/>
+<grid distance="100" unitdist="mil" unit="mil" style="lines" multiple="1" display="yes" altdistance="10" altunitdist="mil" altunit="mil"/>
 <layers>
 <layer number="1" name="Top" color="4" fill="1" visible="yes" active="yes"/>
@@
 <layer number="27" name="tValues" color="7" fill="1" visible="no" active="yes"/>
 <layer number="28" name="bValues" color="7" fill="1" visible="no" active="yes"/>
-<layer number="29" name="tStop" color="7" fill="3" visible="yes" active="yes"/>
-<layer number="30" name="bStop" color="7" fill="6" visible="yes" active="yes"/>
+<layer number="29" name="tStop" color="7" fill="3" visible="no" active="yes"/>
+<layer number="30" name="bStop" color="7" fill="6" visible="no" active="yes"/>
 <layer number="31" name="tCream" color="7" fill="4" visible="no" active="yes"/>
 <layer number="32" name="bCream" color="7" fill="5" visible="no" active="yes"/>
@@
 &lt;p&gt;
 &lt;i&gt;Attention: Upon running the design check and making modifications, please remember to save any changes before closing the application and sending in your board file to Sunstone Circuits for conversion.&lt;i&gt;</description>
-<param name="layerSetup" value="(1+2*15+16)"/>
+<param name="layerSetup" value="(1*16)"/>
 <param name="mtCopper" value="0.0178mm 0.0356mm 0.0356mm 0.0356mm 0.0356mm 0.0356mm 0.0356mm 0.0356mm 0.0356mm 0.0356mm 0.0356mm 0.0356mm 0.0356mm 0.0356mm 0.0356mm 0.0178mm"/>
 <param name="mtIsolate" value="12mil 28mil 0.2007mm 0.1499mm 0.2007mm 0.1499mm 0.2007mm 0.1499mm 0.2007mm 0.1499mm 0.2007mm 0.1499mm 0.2007mm 0.1499mm 12mil"/>
@@
 <attribute name="NAME" x="28.1686" y="21.2344" size="0.889" layer="25" font="vector" ratio="12" rot="R270" align="bottom-center"/>
 </element>
-<element name="R1" library="passives" package="0603-RES" value="0" x="42.164" y="37.084" smashed="yes">
+<element name="R1" library="passives" package="0603-RES" value="DNP - 0" x="42.164" y="37.084" smashed="yes">
 <attribute name="DIGIKEY" value="1276-3431-1-ND" x="42.164" y="37.084" size="1.778" layer="27" font="vector" ratio="12" display="off"/>
 <attribute name="MANUFACTURER" value="Samsung" x="42.164" y="37.084" size="1.778" layer="27" display="off"/>
@@
 <wire x1="33.6804" y1="55.2704" x2="34.29" y2="54.6608" width="0.254" layer="1"/>
 <wire x1="34.29" y1="54.6608" x2="34.29" y2="53.9543" width="0.254" layer="1"/>
-<polygon width="0.254" layer="2" isolate="0.1524" rank="2">
-<vertex x="2.032" y="75.692"/>
-<vertex x="79.502" y="75.692"/>
-<vertex x="79.502" y="-3.302"/>
-<vertex x="2.032" y="-3.302"/>
-</polygon>
 <via x="57.531" y="6.3246" extent="1-16" drill="2.9464" diameter="6.35"/>
 <via x="15.621" y="6.3246" extent="1-16" drill="2.9464" diameter="6.35"/>
@@
 <wire x1="24.3332" y1="38.2524" x2="32.893" y2="38.2524" width="0.508" layer="16"/>
 <wire x1="40.8432" y1="38.1762" x2="42.8244" y2="40.132" width="0.508" layer="16"/>
-<polygon width="0.254" layer="15" isolate="0.1524" rank="2">
-<vertex x="1.524" y="76.2"/>
-<vertex x="80.518" y="76.2"/>
-<vertex x="80.518" y="-4.064"/>
-<vertex x="1.524" y="-4.064"/>
-</polygon>
 <wire x1="69.4944" y1="27.686" x2="69.4944" y2="32.8676" width="0.254" layer="1"/>
 <wire x1="69.4944" y1="32.8676" x2="68.072" y2="34.29" width="0.254" layer="1"/>
