File: modules/rf_spectrum/rev_b/macrofab_compliant/rf_spectrum.sch (EAGLE design)
At the start: 45 parts, among them J3 SIGNPOST_DEBUG_HEADERSMT, J4 SIGNPOST_MODULE_HEADER, J5 TC2030-JLINK-L, Q1 SI223DDS, U1 MWSUB3G, U2 SKY13317, U3 STM32L432KC, U4 TLV62130, X1 ABS05-32.768KHZ-T

Commit message: updated rf spectrum with fixed attribute
Parts:
- R4: DIGIKEY 311-100KLRCT-ND -> 311-1.0KJRCT-ND; MPN RC0402FR-07100KL -> RC0402JR-071KL
Changed lines of the file:
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@@
 </part>
 <part name="R4" library="passives" deviceset="RESISTOR" device="0402_RES" value="1k">
-<attribute name="DIGIKEY" value="311-100KLRCT-ND"/>
+<attribute name="DIGIKEY" value="311-1.0KJRCT-ND"/>
 <attribute name="MANUFACTURER" value="Yageo"/>
-<attribute name="MPN" value="RC0402FR-07100KL"/>
+<attribute name="MPN" value="RC0402JR-071KL"/>
 </part>
 <part name="J4" library="signpost" deviceset="SIGNPOST_MODULE_HEADER" device=""/>
